Commit message: Add position controller to swerve module

File: src/rover/description/ros2_control.xacro (robot description, xacro)
@@ -1,7 +1,15 @@
 <?xml version="1.0"?>
 <robot xmlns:xacro="http://www.ros.org/wiki/xacro">
-    <xacro:macro name="swerve_module_ros2control_iface" params="name">
+    <xacro:macro name="ros2control_swerve_module_iface" params="name">
         <joint name="db_${name}_fork_tyre_joint">
             <command_interface name="velocity">
+                <param name="min">-2</param>
+                <param name="max">2</param>
+            </command_interface>
+            <state_interface name="position"/>
+            <state_interface name="velocity"/>
+        </joint>
+        <joint name="db_${name}_smount_fork_joint">
+            <command_interface name="position">
                 <param name="min">-2</param>
                 <param name="max">2</param>
@@ -16,8 +24,8 @@
         </hardware>
         <!-- Drivebase drive motors -->
-        <xacro:swerve_module_ros2control_iface name="fl"/>
-        <xacro:swerve_module_ros2control_iface name="fr"/>
-        <xacro:swerve_module_ros2control_iface name="bl"/>
-        <xacro:swerve_module_ros2control_iface name="br"/>
+        <xacro:ros2control_swerve_module_iface name="fl"/>
+        <xacro:ros2control_swerve_module_iface name="fr"/>
+        <xacro:ros2control_swerve_module_iface name="bl"/>
+        <xacro:ros2control_swerve_module_iface name="br"/>
         <!-- TODO: Drivebase turn motors -->
     </ros2_control>

Commit message: Fixes

File: src/rover/description/ros2_control.xacro (robot description, xacro)
@@ -19,4 +19,9 @@
         </joint>
     </xacro:macro>
+    <xacro:macro name="ros2control_drivebase_suspension_pivot" params="side">
+        <joint name="${side}db_pivot_joint">
+            <state_interface name="position"/>
+        </joint>
+    </xacro:macro>
     <ros2_control name="RobotSystem" type="system">
         <hardware>
@@ -28,4 +33,6 @@
         <xacro:ros2control_swerve_module_iface name="bl"/>
         <xacro:ros2control_swerve_module_iface name="br"/>
+        <xacro:ros2control_drivebase_suspension_pivot side="l"/>
+        <xacro:ros2control_drivebase_suspension_pivot side="r"/>
         <!-- TODO: Drivebase turn motors -->
     </ros2_control>
