Commit message: [Description] Comment ROS2Control xacro includes, remove castor wheel, create a JointStatePublisher and add pkg info

File: src/rover/description/robot.urdf.xacro (robot description, xacro)
@@ -4,9 +4,9 @@
     <xacro:arg name="sim_mode" default="false"/>
     <xacro:include filename="robot_core.xacro" />
-    <xacro:if value="$(arg use_ros2_control)">
+    <!-- <xacro:if value="$(arg use_ros2_control)">
         <xacro:include filename="ros2_control.xacro" />
     </xacro:if>
     <xacro:unless value="$(arg use_ros2_control)">
         <xacro:include filename="gazebo_control.xacro" />
-    </xacro:unless>
+    </xacro:unless> -->
 </robot>

File: src/rover/description/robot_core.xacro (robot description, xacro)
@@ -34,12 +34,4 @@
     <link name="base_link">
     </link>
-    <!-- BASE_FOOTPRINT LINK -->
-    <joint name="base_footprint_joint" type="fixed">
-        <parent link="base_link"/>
-        <child link="base_footprint"/>
-        <origin xyz="0 0 0" rpy="0 0 0"/>
-    </joint>
-    <link name="base_footprint">
-    </link>
     <!-- CHASSIS LINK -->
     <joint name="chassis_joint" type="fixed">
@@ -71,5 +63,5 @@
     <!-- LEFT WHEEL LINK -->
     <joint name="left_wheel_joint" type="continuous">
-        <parent link="base_link"/>
+        <parent link="chassis"/>
         <child link="left_wheel"/>
         <origin xyz="0 ${wheel_offset_y} 0" rpy="-${pi/2} 0 0" />
@@ -97,5 +89,5 @@
     <!-- RIGHT WHEEL LINK -->
     <joint name="right_wheel_joint" type="continuous">
-        <parent link="base_link"/>
+        <parent link="chassis"/>
         <child link="right_wheel"/>
         <origin xyz="0 ${-wheel_offset_y} 0" rpy="${pi/2} 0 0" />
@@ -121,30 +113,3 @@
         <material>Gazebo/Blue</material>
     </gazebo>
-    <!-- CASTER WHEEL LINK -->
-    <joint name="caster_wheel_joint" type="fixed">
-        <parent link="chassis"/>
-        <child link="caster_wheel"/>
-        <origin xyz="${caster_wheel_offset_x} 0 ${caster_wheel_offset_z}"/>
-    </joint>
-    <link name="caster_wheel">
-        <visual>
-            <geometry>
-                <sphere radius="${caster_wheel_radius}"/>
-            </geometry>
-            <material name="white"/>
-        </visual>
-        <collision>
-            <geometry>
-                <sphere radius="${caster_wheel_radius}"/>
-            </geometry>
-        </collision>
-        <xacro:inertial_sphere mass="${caster_wheel_mass}" radius="${caster_wheel_radius}">
-            <origin xyz="0 0 0" rpy="0 0 0"/>
-        </xacro:inertial_sphere>
-    </link>
-    <gazebo reference="caster_wheel">
-        <material>Gazebo/White</material>
-        <mu1 value="0.001"/>
-        <mu2 value="0.001"/>
-    </gazebo>
 </robot>

Commit message: Fix simulation

File: src/rover/description/robot.urdf.xacro (robot description, xacro)
@@ -5,4 +5,3 @@
     <xacro:include filename="robot_core.xacro" />
     <xacro:include filename="ros2_control.xacro" />
-    <xacro:include filename="gazebo_control.xacro" />
 </robot>

File: src/rover/description/robot_core.xacro (robot description, xacro)
@@ -81,5 +81,5 @@
         <axis xyz="0 0 1"/>
         <limit lower="${-pi/6}" upper="${pi/6}" effort="0.0" velocity="0.0"/>
-        <mimic joint="ldb_pivot_joint" multiplier="-1"/>
+        <!-- TODO: <mimic joint="ldb_pivot_joint" multiplier="-1"/> -->
     </joint>
     <link name="rdb_pivot">

File: src/rover/description/ros2_control.xacro (robot description, xacro)
@@ -1,28 +1,28 @@
 <?xml version="1.0"?>
 <robot xmlns:xacro="http://www.ros.org/wiki/xacro">
-    <ros2_control name="GazeboSimSystem" type="system">
-        <hardware>
-            <plugin>gz_ros2_control/GazeboSimSystem</plugin>
-        </hardware>
-        <joint name="left_wheel_joint">
+    <xacro:macro name="swerve_module_ros2control_iface" params="name">
+        <joint name="db_${name}_fork_tyre_joint">
             <command_interface name="velocity">
-                <param name="min">-10</param>
-                <param name="max">10</param>
+                <param name="min">-2</param>
+                <param name="max">2</param>
             </command_interface>
             <state_interface name="position"/>
             <state_interface name="velocity"/>
         </joint>
-        <joint name="right_wheel_joint">
-            <command_interface name="velocity">
-                <param name="min">-10</param>
-                <param name="max">10</param>
-            </command_interface>
-            <state_interface name="position"/>
-            <state_interface name="velocity"/>
-        </joint>
+    </xacro:macro>
+    <ros2_control name="RobotSystem" type="system">
+        <hardware>
+            <plugin>gz_ros2_control/GazeboSimSystem</plugin>
+        </hardware>
+        <!-- Drivebase drive motors -->
+        <xacro:swerve_module_ros2control_iface name="fl"/>
+        <xacro:swerve_module_ros2control_iface name="fr"/>
+        <xacro:swerve_module_ros2control_iface name="bl"/>
+        <xacro:swerve_module_ros2control_iface name="br"/>
+        <!-- TODO: Drivebase turn motors -->
     </ros2_control>
     <gazebo>
-        <plugin name="gazebo_ros2_control" filename="libgazebo_ros2_control.so">
-            <parameters>$(find OWR-502)/src/rover/description/diff_drive_controller.yaml</parameters>
+        <plugin filename="gz_ros2_control-system" name="gz_ros2_control::GazeboSimROS2ControlPlugin">
+            <parameters>$(find rover)/config/drivebase/diff_drive_controller.yaml</parameters>
         </plugin>
     </gazebo>

Commit message: Fix xacro file

File: src/rover/description/robot.urdf.xacro (robot description, xacro)
@@ -7,3 +7,10 @@
     <xacro:include filename="drivebase/drivebase.xacro" />
     <xacro:include filename="utils/gazebo_plugins.xacro" />
+    <joint name="test_motor" type="continuous">
+        <parent link="chassis"/>
+        <child link="dumb"/>
+        <origin xyz="0 0 0" rpy="${-pi/2} 0 0" />
+        <axis xyz="0 0 1"/>
+    </joint>
+    <link name="dumb"/>
 </robot>
