Commit message: [Drivebase] Fix azipod azimuth axis, add joint limits for diff bar pivot

File: src/rover/description/drivebase/db_helpers.xacro (robot description, xacro)
@@ -19,4 +19,5 @@
             <child link="${prefix}_wheel_fork"/>
             <origin xyz="0 0 ${-0.213/2 - 0.03/2}" rpy="0 0 0" />
+            <axis xyz="0 0 1"/>
         </joint>
         <!-- This is the actual wheel -->

File: src/rover/description/robot_core.xacro (robot description, xacro)
@@ -51,10 +51,11 @@
     </gazebo>
     <!-- LEFT SIDE STUFF -->
-    <!-- TODO: Make it a revolute joint and add constraints -->
-    <joint name="ldb_pivot_joint" type="continuous">
+    <!-- TODO: Fix effort and velocity limits -->
+    <joint name="ldb_pivot_joint" type="revolute">
         <parent link="chassis"/>
         <child link="ldb_pivot"/>
         <origin xyz="0 ${chassis_width/2 + 0.014 + diff_bar_bearing_seat_width} 0" rpy="-${pi/2} 0 0" />
         <axis xyz="0 0 1"/>
+        <limit lower="${-pi/6}" upper="${pi/6}" effort="0.0" velocity="0.0"/>
     </joint>
     <link name="ldb_pivot">
@@ -70,5 +71,5 @@
     <xacro:db_module_corner prefix="db_bl" isrear="-1" parent="ldb_pivot"/>
     <!-- RIGHT SIDE STUFF -->
-    <!-- TODO: Make it a revolute joint and add constraints -->
+    <!-- TODO: Fix effort and velocity limits -->
     <joint name="rdb_pivot_joint" type="continuous">
         <parent link="chassis"/>
@@ -76,4 +77,6 @@
         <origin xyz="0 -${chassis_width/2 + 0.014 + diff_bar_bearing_seat_width} 0" rpy="-${pi/2} 0 0" />
         <axis xyz="0 0 1"/>
+        <limit lower="${-pi/6}" upper="${pi/6}" effort="0.0" velocity="0.0"/>
+        <mimic joint="ldb_pivot_joint" multiplier="-1"/>
     </joint>
     <link name="rdb_pivot">

Commit message: [Drivebase] Add steering joint limits

File: src/rover/description/drivebase/db_helpers.xacro (robot description, xacro)
@@ -14,10 +14,12 @@
             <origin xyz="${isrear*diff_bar_length/2} ${0.05} ${(0.0425 + 0.02975)*flip_x}" rpy="${pi/2} 0 ${isrear*(pi/-6)}" />
         </joint>
-        <!-- This is the steering joint, TODO: add limits -->
-        <joint name="${prefix}_smount_fork_joint" type="continuous">
+        <!-- This is the steering joint -->
+        <!-- TODO: Fix effort and velocity limits, and get actual lower/upper -->
+        <joint name="${prefix}_smount_fork_joint" type="revolute">
             <parent link="${prefix}_smount"/>
             <child link="${prefix}_wheel_fork"/>
             <origin xyz="0 0 ${-0.213/2 - 0.03/2}" rpy="0 0 0" />
             <axis xyz="0 0 1"/>
+            <limit lower="${-pi/2}" upper="${pi/2}" effort="0.0" velocity="0.0"/>
         </joint>
         <!-- This is the actual wheel -->

Commit message: Added collision to wheels, inertia to frame parts

File: src/rover/description/drivebase/db_helpers.xacro (robot description, xacro)
@@ -38,4 +38,7 @@
                 <material name="orange"/>
             </visual>
+            <xacro:inertial_box mass="2" x="${diff_bar_length}" y="${diff_bar_bearing_seat_width}" z="${diff_bar_bearing_seat_width}">
+                <origin xyz="0 0 0" rpy="0 0 0"/>
+            </xacro:inertial_box>
         </link>
         <!-- Steering mount -->
@@ -65,4 +68,12 @@
                 <material name="black"/>
             </visual>
+            <collision>
+                <geometry>
+                    <sphere radius="${0.125}"/>
+                </geometry>
+            </collision>
+            <xacro:inertial_sphere mass="2.5" radius="${0.125}" >
+                <origin xyz="0 0 0" rpy="0 0 0"/>
+            </xacro:inertial_sphere>
         </link>
     </xacro:macro>

File: src/rover/description/robot_core.xacro (robot description, xacro)
@@ -46,4 +46,7 @@
             <material name="orange"/>
         </visual>
+        <xacro:inertial_box mass="15" x="${chassis_length}" y="${chassis_width}" z="${chassis_height}">
+            <origin xyz="0 0 0" rpy="0 0 0"/>
+        </xacro:inertial_box>
     </link>
     <gazebo reference="chassis">

Commit message: added arbitrary inertia to wheel fork to stop gazebo complaints

File: src/rover/description/drivebase/db_helpers.xacro (robot description, xacro)
@@ -59,4 +59,7 @@
                 <material name="blue"/>
             </visual>
+            <xacro:inertial_box mass="1" x="0.066" y="0.170" z="0.213">
+                <origin xyz="0 0 0" rpy="0 0 0"/>
+            </xacro:inertial_box>
         </link>
         <!-- Wheel -->

Commit message: Add one correct and one bogus velocity and effort limit

File: src/rover/description/drivebase/db_helpers.xacro (robot description, xacro)
@@ -15,5 +15,4 @@
         </joint>
         <!-- This is the steering joint -->
-        <!-- TODO: Fix effort and velocity limits, and get actual lower/upper -->
         <joint name="${prefix}_smount_fork_joint" type="revolute">
             <parent link="${prefix}_smount"/>
@@ -21,5 +20,5 @@
             <origin xyz="0 0 ${-0.213/2 - 0.03/2}" rpy="0 0 0" />
             <axis xyz="0 0 1"/>
-            <limit lower="${-pi/2}" upper="${pi/2}" effort="0.0" velocity="0.0"/>
+            <limit lower="${-pi/2}" upper="${pi/2}" effort="40.0" velocity="12.8"/>
         </joint>
         <!-- This is the actual wheel -->

File: src/rover/description/robot_core.xacro (robot description, xacro)
@@ -54,5 +54,5 @@
     </gazebo>
     <!-- LEFT SIDE STUFF -->
-    <!-- TODO: Fix effort and velocity limits -->
+    <!-- TODO: Fix effort and velocity limits. Current values are arbitrary. -->
     <joint name="ldb_pivot_joint" type="revolute">
         <parent link="chassis"/>
@@ -60,5 +60,5 @@
         <origin xyz="0 ${chassis_width/2 + 0.014 + diff_bar_bearing_seat_width} 0" rpy="-${pi/2} 0 0" />
         <axis xyz="0 0 1"/>
-        <limit lower="${-pi/6}" upper="${pi/6}" effort="0.0" velocity="0.0"/>
+        <limit lower="${-pi/6}" upper="${pi/6}" effort="80.0" velocity="10.0"/>
     </joint>
     <link name="ldb_pivot">
