Commit message: Refactor rover URDF description files

File: src/rover/description/drivebase/drivebase.xacro (robot description, xacro)
@@ -1,9 +1,6 @@
 <?xml version="1.0"?>
 <robot xmlns:xacro="http://www.ros.org/wiki/xacro" >
-    <xacro:include filename="inertial_macros.xacro"/>
-    <xacro:property name="chassis_length" value="0.600"/>
-    <xacro:property name="chassis_width" value="0.450"/>
-    <xacro:property name="chassis_height" value="0.100"/>
-    <xacro:property name="chassis_mass" value="10.0"/>
+    <xacro:include filename="db_helpers.xacro" />
+    <xacro:include filename="ros2_control.xacro"/>
     <xacro:property name="diff_bar_bearing_seat_width" value="0.04"/>
     <xacro:property name="diff_bar_length" value="0.600"/>
@@ -14,43 +11,4 @@
     <xacro:property name="wheel_offset_y" value="0.3"/>
     <xacro:property name="wheel_offset_z" value="0.01"/>
-    <material name="white">
-        <color rgba="1 1 1 1" />
-    </material>
-    <material name="orange">
-        <color rgba="1 0.3 0.1 1"/>
-    </material>
-    <material name="blue">
-        <color rgba="0.2 0.2 1 1"/>
-    </material>
-    <material name="black">
-        <color rgba="0 0 0 1"/>
-    </material>
-    <material name="red">
-        <color rgba="1 0 0 1"/>
-    </material>
-    <!-- BASE LINK -->
-    <link name="base_link">
-    </link>
-    <!-- CHASSIS LINK -->
-    <joint name="chassis_joint" type="fixed">
-        <parent link="base_link"/>
-        <child link="chassis"/>
-        <origin xyz="0 0 0"/>
-    </joint>
-    <link name="chassis">
-        <visual>
-            <origin xyz="0 0 0"/>
-            <geometry>
-                <box size="${chassis_length} ${chassis_width} ${chassis_height}"/>
-            </geometry>
-            <material name="orange"/>
-        </visual>
-        <xacro:inertial_box mass="15" x="${chassis_length}" y="${chassis_width}" z="${chassis_height}">
-            <origin xyz="0 0 0" rpy="0 0 0"/>
-        </xacro:inertial_box>
-    </link>
-    <gazebo reference="chassis">
-        <material>Gazebo/Orange</material>
-    </gazebo>
     <!-- LEFT SIDE STUFF -->
     <!-- TODO: Fix effort and velocity limits. Current values are arbitrary. -->
@@ -70,5 +28,4 @@
         </visual>
     </link>
-    <xacro:include filename="drivebase/db_helpers.xacro" />
     <xacro:db_module_corner prefix="db_fl" isrear="1" parent="ldb_pivot"/>
     <xacro:db_module_corner prefix="db_bl" isrear="-1" parent="ldb_pivot"/>

File: src/rover/description/drivebase/ros2_control.xacro (robot description, xacro)
@@ -24,4 +24,5 @@
         </joint>
     </xacro:macro>
+    <!-- FIXME: Gate this behind is_simulation -->
     <ros2_control name="RobotSystem" type="system">
         <hardware>
@@ -37,4 +38,5 @@
         <!-- TODO: Drivebase turn motors -->
     </ros2_control>
+    <!-- FIXME: Gate this behind is_simulation -->
     <gazebo>
         <plugin filename="gz_ros2_control-system" name="gz_ros2_control::GazeboSimROS2ControlPlugin">

File: src/rover/description/robot.urdf.xacro (robot description, xacro)
@@ -1,7 +1,8 @@
 <?xml version="1.0"?>
 <robot xmlns:xacro="http://www.ros.org/wiki/xacro"  name="robot">
-    <xacro:arg name="use_ros2_control" default="true"/>
-    <xacro:arg name="sim_mode" default="false"/>
-    <xacro:include filename="robot_core.xacro" />
-    <xacro:include filename="ros2_control.xacro" />
+    <xacro:arg name="is_simulation" default="true"/>
+    <xacro:include filename="utils/inertial_macros.xacro" />
+    <xacro:include filename="utils/materials.xacro" />
+    <xacro:include filename="chassis/chassis.xacro" />
+    <xacro:include filename="drivebase/drivebase.xacro" />
 </robot>
