Commit message: It is no longer unemployed.
xian zia ta bu shi wu yong de ren

File: src/rover/description/drivebase/ros2_control.xacro (robot description, xacro)
@@ -28,7 +28,7 @@
     <ros2_control name="test_motor" type="actuator">
         <hardware>
-            <plugin>bg431esc1_actuator/Bg431esc1Actuator</plugin>
+            <plugin>bg431esc1_actuator::Bg431esc1Actuator</plugin>
+            <param name="device_index">1</param>
         </hardware>
-        <param name="device_index">1</param>
         <joint name="test">
             <command_interface name="position"/>

File: src/rover/description/robot.urdf.xacro (robot description, xacro)
@@ -1,11 +1,10 @@
 <?xml version="1.0"?>
-<robot xmlns:xacro="http://www.ros.org/wiki/xacro"  name="robot">
-    <xacro:arg name="is_simulation" default="true"/>
+<robot xmlns:xacro="http://www.ros.org/wiki/xacro" name="robot">
     <xacro:include filename="utils/inertial_macros.xacro" />
     <xacro:include filename="utils/materials.xacro" />
     <xacro:include filename="chassis/chassis.xacro" />
     <xacro:include filename="drivebase/drivebase.xacro" />
-    <xacro:include filename="utils/gazebo_plugins.xacro" />
-    <joint name="test_motor" type="continuous">
+    <!--<xacro:include filename="utils/gazebo_plugins.xacro" />-->
+    <joint name="test" type="continuous">
         <parent link="chassis"/>
         <child link="dumb"/>

Commit message: Restor rover stuf

File: src/rover/description/drivebase/ros2_control.xacro (robot description, xacro)
@@ -6,6 +6,4 @@
                 <param name="min">-2</param>
                 <param name="max">2</param>
-                <param name="can_id">1</param>
-                <param name="control_mode">3</param>
             </command_interface>
             <state_interface name="position"/>
@@ -26,33 +24,10 @@
         </joint>
     </xacro:macro>
-    <ros2_control name="test_motor" type="actuator">
-        <hardware>
-            <plugin>bg431esc1_actuator::Bg431esc1Actuator</plugin>
-            <param name="device_index">1</param>
-            <param name="ratio">1</param>
-            <param name="use_auxilary">false</param>
-        </hardware>
-        <joint name="test">
-            <command_interface name="position"/>
-            <command_interface name="velocity"/>
-            <command_interface name="torque"/>
-            <state_interface name="position"/>
-            <state_interface name="velocity"/>
-            <state_interface name="primary_position"/>
-            <state_interface name="primary_velocity"/>
-            <state_interface name="auxilary_position"/>
-            <state_interface name="auxilary_velocity"/>
-            <state_interface name="applied_voltage"/>
-            <state_interface name="stator_current"/>
-            <state_interface name="supply_current"/>
-            <state_interface name="bus_voltage"/>
-            <state_interface name="driver_temperature"/>
-        </joint>
-    </ros2_control>
-<!--
+    <!-- FIXME: Gate this behind is_simulation -->
     <ros2_control name="RobotSystem" type="system">
         <hardware>
             <plugin>gz_ros2_control/GazeboSimSystem</plugin>
         </hardware>
+        <!-- Drivebase drive motors -->
         <xacro:ros2control_swerve_module_iface name="fl"/>
         <xacro:ros2control_swerve_module_iface name="fr"/>
@@ -61,9 +36,12 @@
         <xacro:ros2control_drivebase_suspension_pivot side="l"/>
         <xacro:ros2control_drivebase_suspension_pivot side="r"/>
+        <!-- TODO: Drivebase turn motors -->
     </ros2_control>
+    <!-- FIXME: Gate this behind is_simulation -->
     <gazebo>
         <plugin filename="gz_ros2_control-system" name="gz_ros2_control::GazeboSimROS2ControlPlugin">
+            <!-- FIXME: reenable? <parameters>$(find rover)/config/drivebase/diff_drive_controller.yaml</parameters> -->
             <parameters>$(find rover)/config/drivebase/swerve_drive_controller.yaml</parameters>
         </plugin>
-    </gazebo> -->
+    </gazebo>
 </robot>

File: src/rover/description/robot.urdf.xacro (robot description, xacro)
@@ -1,15 +1,9 @@
 <?xml version="1.0"?>
-<robot xmlns:xacro="http://www.ros.org/wiki/xacro" name="robot">
+<robot xmlns:xacro="http://www.ros.org/wiki/xacro"  name="robot">
+    <xacro:arg name="is_simulation" default="true"/>
     <xacro:include filename="utils/inertial_macros.xacro" />
     <xacro:include filename="utils/materials.xacro" />
     <xacro:include filename="chassis/chassis.xacro" />
     <xacro:include filename="drivebase/drivebase.xacro" />
-    <!--<xacro:include filename="utils/gazebo_plugins.xacro" />-->
-    <joint name="test" type="continuous">
-        <parent link="chassis"/>
-        <child link="dumb"/>
-        <origin xyz="0 0 0" rpy="${-pi/2} 0 0" />
-        <axis xyz="0 0 1"/>
-    </joint>
-    <link name="dumb"/>
+    <xacro:include filename="utils/gazebo_plugins.xacro" />
 </robot>

Commit message: Add switch for simulation to xacro

File: src/rover/description/drivebase/ros2_control.xacro (robot description, xacro)
@@ -1,47 +1,58 @@
 <?xml version="1.0"?>
 <robot xmlns:xacro="http://www.ros.org/wiki/xacro">
-    <xacro:macro name="ros2control_swerve_module_iface" params="name">
-        <joint name="db_${name}_fork_tyre_joint">
-            <command_interface name="velocity">
-                <param name="min">-2</param>
-                <param name="max">2</param>
-            </command_interface>
-            <state_interface name="position"/>
-            <state_interface name="velocity"/>
-        </joint>
-        <joint name="db_${name}_smount_fork_joint">
-            <command_interface name="position">
-                <param name="min">-2</param>
-                <param name="max">2</param>
-            </command_interface>
-            <state_interface name="position"/>
-            <state_interface name="velocity"/>
-        </joint>
-    </xacro:macro>
-    <xacro:macro name="ros2control_drivebase_suspension_pivot" params="side">
-        <joint name="${side}db_pivot_joint">
-            <state_interface name="position"/>
-        </joint>
-    </xacro:macro>
-    <!-- FIXME: Gate this behind is_simulation -->
+    <xacro:if value="$(arg is_simulation)">
+        <xacro:macro name="ros2control_swerve_module_iface" params="name drive_id turn_id">
+            <joint name="db_${name}_fork_tyre_joint">
+                <command_interface name="velocity">
+                    <param name="min">-2</param>
+                    <param name="max">2</param>
+                </command_interface>
+                <state_interface name="position"/>
+                <state_interface name="velocity"/>
+            </joint>
+            <joint name="db_${name}_smount_fork_joint">
+                <command_interface name="position">
+                    <param name="min">-2</param>
+                    <param name="max">2</param>
+                </command_interface>
+                <state_interface name="position"/>
+                <state_interface name="velocity"/>
+            </joint>
+        </xacro:macro>
+        <xacro:macro name="ros2control_drivebase_suspension_pivot" params="side">
+            <joint name="${side}db_pivot_joint">
+                <state_interface name="position"/>
+            </joint>
+        </xacro:macro>
+    </xacro:if>
+    <xacro:unless value="$(arg is_simulation)">
+        <xacro:macro name="ros2control_swerve_module_iface" params="name drive_id turn_id">
+            <!-- TODO: set ratios correctly -->
+            <xacro:bg431_motor name="db_${name}_fork_tyre_joint" device_index="${drive_id}" ratio="1" use_auxilary="false"/>
+            <xacro:bg431_motor name="db_${name}_smount_fork_joint" device_index="${turn_id}" ratio="1" use_auxilary="true"/>
+        </xacro:macro>
+        <xacro:macro name="ros2control_drivebase_suspension_pivot" params="side"/>
+    </xacro:unless>
     <ros2_control name="RobotSystem" type="system">
-        <hardware>
-            <plugin>gz_ros2_control/GazeboSimSystem</plugin>
-        </hardware>
+        <xacro:if value="$(arg is_simulation)">
+            <hardware>
+                <plugin>gz_ros2_control/GazeboSimSystem</plugin>
+            </hardware>
+        </xacro:if>
         <!-- Drivebase drive motors -->
-        <xacro:ros2control_swerve_module_iface name="fl"/>
-        <xacro:ros2control_swerve_module_iface name="fr"/>
-        <xacro:ros2control_swerve_module_iface name="bl"/>
-        <xacro:ros2control_swerve_module_iface name="br"/>
+        <xacro:ros2control_swerve_module_iface name="fl" drive_id="1" turn_id="2"/>
+        <xacro:ros2control_swerve_module_iface name="fr" drive_id="3" turn_id="4"/>
+        <xacro:ros2control_swerve_module_iface name="bl" drive_id="5" turn_id="6"/>
+        <xacro:ros2control_swerve_module_iface name="br" drive_id="7" turn_id="8"/>
         <xacro:ros2control_drivebase_suspension_pivot side="l"/>
         <xacro:ros2control_drivebase_suspension_pivot side="r"/>
         <!-- TODO: Drivebase turn motors -->
     </ros2_control>
-    <!-- FIXME: Gate this behind is_simulation -->
-    <gazebo>
-        <plugin filename="gz_ros2_control-system" name="gz_ros2_control::GazeboSimROS2ControlPlugin">
-            <!-- FIXME: reenable? <parameters>$(find rover)/config/drivebase/diff_drive_controller.yaml</parameters> -->
-            <parameters>$(find rover)/config/drivebase/swerve_drive_controller.yaml</parameters>
-        </plugin>
-    </gazebo>
+    <xacro:if value="$(arg is_simulation)">
+        <gazebo>
+            <plugin filename="gz_ros2_control-system" name="gz_ros2_control::GazeboSimROS2ControlPlugin">
+                <parameters>$(find rover)/config/drivebase/swerve_drive_controller.yaml</parameters>
+            </plugin>
+        </gazebo>
+    </xacro:if>
 </robot>

File: src/rover/description/robot.urdf.xacro (robot description, xacro)
@@ -2,8 +2,13 @@
 <robot xmlns:xacro="http://www.ros.org/wiki/xacro"  name="robot">
     <xacro:arg name="is_simulation" default="true"/>
+    <xacro:unless value="$(arg is_simulation)">
+        <xacro:include filename="utils/bg431_motor.xacro"/>
+    </xacro:unless>
     <xacro:include filename="utils/inertial_macros.xacro" />
     <xacro:include filename="utils/materials.xacro" />
     <xacro:include filename="chassis/chassis.xacro" />
     <xacro:include filename="drivebase/drivebase.xacro" />
-    <xacro:include filename="utils/gazebo_plugins.xacro" />
+    <xacro:if value="$(arg is_simulation)">
+        <xacro:include filename="utils/gazebo_plugins.xacro" />
+    </xacro:if>
 </robot>
