File: src/can_converter/Can_converter_v1/Can_converter_v1.kicad_sch (KiCad schematic)
At the start: 10 parts, among them J1 SM02B-PASS, X1 629722000214_pasteInHole

Commit message: Create second version from scratch with rearranged components
Parts:
- X1: footprint Socket_GCT:USB4105_pasteInHole -> Connector_USB:USB_C_Receptacle_GCT_USB4105-xx-A_16P_TopMnt_Horizontal
Changed lines of the file:
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@@
 			)
 		)
-		(property "Footprint" "Socket_GCT:USB4105_pasteInHole"
+		(property "Footprint" "Connector_USB:USB_C_Receptacle_GCT_USB4105-xx-A_16P_TopMnt_Horizontal"
 			(at 33.02 55.88 0)
 			(effects
