File: src/can_converter/Can_converter_v1/PSU.kicad_sch (KiCad schematic)
At the start: 5 parts

Commit message: Create second version from scratch with rearranged components
Parts:
- PS1: footprint SOT94P279X130-5N -> Package_TO_SOT_SMD:SOT-23-5_HandSoldering
Changed lines of the file:
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@@
 			)
 		)
-		(property "Footprint" "SOT94P279X130-5N"
+		(property "Footprint" "Package_TO_SOT_SMD:SOT-23-5_HandSoldering"
 			(at 152.4 209.22 0)
 			(effects
