File: src/computing_power_hub_elec/_autosave-connectors.kicad_sch (KiCad schematic)
At the start: 49 parts, among them J105 BM03B-PASS, J106 BM03B-PASS, J107 BM03B-PASS, J108 BM03B-PASS, J310 XT30M, J320 RJ45, J321 RJ45, J330 S2P-VH, J340 S2P-VH, Q301 BC846S,115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

Commit message: Is sisyphus happy?
Connections:
- net ETH_{IBM}: now also R322.1, TR101.18 (CT); no longer R321.1, TR101.21 (CT)
- net ETH_{ICM}: now also R321.1, TR101.21 (CT); no longer R322.1, TR101.18 (CT)
- net ETH_{IAT}: now reaches C320.2, R320.2
- net ETH_{ICT}: now reaches C321.2, R321.2
- net ETH_{IBT}: now reaches C322.2, R322.2
- net ETH_{IDT}: now reaches C323.2, R323.2
Changed lines of the file:
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@@
+		)
+	)
+	(label "ETH_{ICT}"
+		(at 128.27 72.39 0)
+		(effects
+			(font
+				(size 0.381 0.381)
+			)
+			(justify left bottom)
 		)
 	)
@@
 		)
 	)
+	(label "ETH_{IAT}"
+		(at 124.46 72.39 0)
+		(effects
+			(font
+				(size 0.381 0.381)
+			)
+			(justify left bottom)
+		)
+	)
 	(label "ETH_{ICM}"
-		(at 142.24 57.15 90)
+		(at 142.24 46.99 90)
+		(effects
+			(font
+				(size 0.381 0.381)
+			)
+			(justify left bottom)
+		)
+	)
+	(label "ETH_{IBT}"
+		(at 132.08 72.39 0)
 		(effects
 			(font
@@
 		)
 	)
-	(label "ETH_{IBM}"
-		(at 142.24 46.99 90)
+	(label "ETH_{IDT}"
+		(at 135.89 72.39 0)
 		(effects
 			(font
+				(size 0.381 0.381)
+			)
+			(justify left bottom)
+		)
+	)
+	(label "ETH_{IBM}"
+		(at 142.24 57.15 90)
+		(effects
+			(font
