File: src/computing_power_hub_elec/computing-power-hub.kicad_pcb (KiCad board)
At the start: 6 copper layers, 70 x 45 mm, 188 parts, among them J101 IDC_6P, J105 BM03B-PASS, J106 BM03B-PASS, J107 BM03B-PASS, J108 BM03B-PASS, J109 SM02B-PASS, J310 XT30M, J320 BM08B-PASS, J321 BM08B-PASS, J330 S2P-VH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

Commit message: I remember
Parts:
- removed C119: 2u2, Capacitor_SMD:C_0603_1608Metric
- removed C127, C128: 220n, Capacitor_SMD:C_0402_1005Metric
- removed H101, H102: M2.5, Bluesat:M2.5_Edge
- removed H103: M2.5, Bluesat:M2.5_Internal
- D101, D102, D105: footprint LED_SMD:LED_WS2812B-2020_PLCC4_2.0x2.0mm -> Bluesat:WS2812B-2020
- moved C126 79.5 mm to (34.6, 25.9)
- moved TH103 72.2 mm to (51.4, 5.88), turned to 90 degrees
- moved R115 71.5 mm to (34.6, 27.0), turned to 0 degrees
- moved C116 69.8 mm to (50.1, 5.88), turned to -90 degrees
- moved R121 51.1 mm to (18.9, 34.1), turned to 0 degrees
- moved R122 49.4 mm to (18.9, 31.9), turned to 0 degrees
- moved TH102 45.1 mm to (23.8, 16.5), turned to -90 degrees
- moved R120 41.8 mm to (18.9, 33.0), turned to 0 degrees
- moved C115 40.6 mm to (22.0, 14.4), turned to -90 degrees
- moved R123 40.4 mm to (18.9, 35.2), turned to 0 degrees
- moved TH101 38.6 mm to (12.0, 27.5), turned to 90 degrees
- moved C114 34.4 mm to (13.1, 27.5), turned to -90 degrees
- moved C117 21.8 mm to (7.38, 12.5), turned to 0 degrees
- moved TH104 18.6 mm to (7.38, 11.4)
- moved Y101 8.67 mm to (32.1, 40.6), turned to -90 degrees
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Routing:
- net /TEMP2: track 0.00 -> 74.3 mm, vias 0 -> 4
- net +5V: track 17.5 -> 66.6 mm, vias 7 -> 20
- net GND: track 9.79 -> 58.8 mm, vias 93 -> 146
- net /Regulators/EN_{24V}: track 6.82 -> 52.7 mm, vias 1 -> 3
- net /Connectors/ARGB_{3}: track 0.00 -> 45.2 mm, vias 1 -> 2
- net /TEMP3: track 0.00 -> 44.1 mm, vias 0 -> 2
- net /Regulators/VS_{24V}: track 1.25 -> 44.6 mm, vias 1 -> 3
- net /Regulators/EN_{19V}: track 8.52 -> 45.3 mm, vias 2 -> 4
- net /Connectors/IS_{24V}: track 6.62 -> 43.1 mm, vias 0 -> 3
- net /Regulators/VS_{19V}: track 0.07 -> 35.9 mm, vias 0 -> 3
- net /Connectors/IS_{19V}: track 0.00 -> 35.0 mm, vias 0 -> 3
- net /Connectors/IS_{5VB}: track 0.88 -> 34.2 mm, vias 10 -> 11
- net /DBG.SWO: track 0.00 -> 31.8 mm, vias 0 -> 4
- net /Connectors/NEN_{5VA}: track 0.00 -> 30.8 mm, vias 0 -> 2
- net /TEMP1: track 0.00 -> 29.4 mm, vias 0 -> 3
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- added copper zone on B.Cu, net VDD
- added copper zone on B.Cu, net VDDA
Other:
- outline, holes or cut-outs redrawn
- board text removed: "${REFERENCE}"

Commit message: Fucking
Other:
- board text added: "19V-8A"
- board text added: "24V-POE"
- board text added: "A- A+ B- B+ C- C+ D- D+"
- board text added: "IN"
- board text added: "RGB +5V GND"
- board text added: "帕瓦电板 Compute Power Hub Rev. 2p0"
Changed lines of the file:
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@@
 			(primitives
 				(gr_rect
-					(start -2.415 -1.68)
-					(end -1.755 -2.13)
+					(start -2.415 -2.13)
+					(end -1.755 -1.68)
 					(width 0)
 					(fill yes)
 				)
 				(gr_rect
-					(start -2.415 -0.41)
-					(end -1.755 -0.86)
+					(start -2.415 -0.86)
+					(end -1.755 -0.41)
 					(width 0)
 					(fill yes)
 				)
 				(gr_rect
-					(start -2.415 0.86)
-					(end -1.755 0.41)
+					(start -2.415 0.41)
+					(end -1.755 0.86)
 					(width 0)
 					(fill yes)
 				)
 				(gr_rect
-					(start -2.415 2.13)
-					(end -1.755 1.68)
+					(start -2.415 1.68)
+					(end -1.755 2.13)
 					(width 0)
 					(fill yes)
@@
 			(primitives
 				(gr_rect
-					(start -2.415 -1.68)
-					(end -1.755 -2.13)
+					(start -2.415 -2.13)
+					(end -1.755 -1.68)
 					(width 0)
 					(fill yes)
 				)
 				(gr_rect
-					(start -2.415 -0.41)
-					(end -1.755 -0.86)
+					(start -2.415 -0.86)
+					(end -1.755 -0.41)
 					(width 0)
 					(fill yes)
 				)
 				(gr_rect
-					(start -2.415 0.86)
-					(end -1.755 0.41)
+					(start -2.415 0.41)
+					(end -1.755 0.86)
 					(width 0)
 					(fill yes)
 				)
 				(gr_rect
-					(start -2.415 2.13)
-					(end -1.755 1.68)
+					(start -2.415 1.68)
+					(end -1.755 2.13)
 					(width 0)
 					(fill yes)
@@
 	)
 	(gr_rect
+		(start 35.875 19.375)
+		(end 45.875 21.375)
+		(stroke
+			(width 0)
+			(type solid)
+		)
+		(fill yes)
+		(layer "F.SilkS")
+	)
+	(gr_rect
 		(start 1.5 1.5)
 		(end 68.5 43.5)
@@
 		(layer "Edge.Cuts")
 	)
+	(gr_text "24V-POE"
+		(at 49.25 12 0)
+		(layer "F.SilkS" knockout)
+		(effects
+			(font
+				(size 1.2 1.2)
+				(thickness 0.2)
+				(bold yes)
+			)
+			(justify left)
+		)
+	)
+	(gr_text "19V-8A"
+		(at 49.25 2.75 0)
+		(layer "F.SilkS" knockout)
+		(effects
+			(font
+				(size 1.2 1.2)
+				(thickness 0.2)
+				(bold yes)
+			)
+			(justify left)
+		)
+	)
+	(gr_text "IN"
+		(at 48.125 23.625 0)
+		(layer "F.SilkS" knockout)
+		(effects
+			(font
+				(size 1.2 1.2)
+				(thickness 0.2)
+				(bold yes)
+			)
+			(justify left)
+		)
+	)
+	(gr_text "RGB\n+5V\nGND"
+		(at 34.25 38.375 0)
+		(layer "F.SilkS")
+		(effects
+			(font
+				(size 0.8 0.8)
+				(thickness 0.1)
+			)
+			(justify right)
+		)
+	)
+	(gr_text "帕瓦电板\nCompute Power Hub\nRev. 2p0"
+		(at 35.75 15.5 0)
+		(layer "F.SilkS")
+		(effects
+			(font
+				(size 0.8 0.8)
+				(thickness 0.1)
+			)
+			(justify left top)
+		)
+	)
+	(gr_text "A-\nA+\nB-\nB+\nC-\nC+\nD-\nD+"
+		(at 47.75 30.625 90)
+		(layer "F.SilkS")
+		(effects
+			(font
+				(size 0.8 0.8)
+				(thickness 0.1)
+			)
+			(justify left bottom)
+		)
+	)
 	(segment
