File: src/computing_power_hub_elec/connectors.kicad_sch (KiCad schematic)
At the start: 49 parts, among them J105 BM03B-PASS, J106 BM03B-PASS, J107 BM03B-PASS, J108 BM03B-PASS, J310 XT30M, J320 RJ45, J321 RJ45, J330 S2P-VH, J340 S2P-VH, Q301 BC846S,115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

Commit message: Baa
Parts:
- removed C340: 220n, Capacitor_SMD:C_0402_1005Metric, symbol Bluesat:C_CompactV
- removed J340: S2P-VH, symbol Connector:Conn_01x02_Pin
- removed Q301: BC846S,115, Package_TO_SOT_SMD:SOT-363_SC-70-6, symbol Transistor_BJT:Q_Dual_NPN_NPN_E1B1C2E2B2C1
- removed Q340, Q350: SSM3K333R, Package_TO_SOT_SMD:SOT-23, symbol Transistor_FET:Q_NMOS_GSD
- removed R340: 10k, Resistor_SMD:R_0402_1005Metric, symbol Bluesat:R_CompactV
- removed R341: 100k, Resistor_SMD:R_0402_1005Metric, symbol Bluesat:R_CompactV
- removed R342: 20m, Diode_SMD:D_2512_6332Metric, symbol Bluesat:R_CompactV
Connections:
- net IS_{5V}: no longer J105.1 (Pin_1), J106.1 (Pin_1), J107.1 (Pin_1), J108.1 (Pin_1)
- net PO_{5}: no longer J105.2 (Pin_2), J106.2 (Pin_2), J107.2 (Pin_2), J108.2 (Pin_2), R352.1, R353.1, R354.1, R355.1
Other:
- note added: "4. 5V ARGB"
- note removed: "4. 12V Output"
- note removed: "5. 5V ARGB"
- moved on the sheet: C301, C302, C303, C304, C305, C306, C307, C350, J105, J106, J107, J108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

Commit message: tmp
Parts:
- added Q301: IRFH7440TRPBF, Package_TO_SOT_SMD:SOT-23, symbol Transistor_FET:Q_NMOS_GSD
- added Q302: BC846S, symbol Transistor_BJT:Q_Dual_NPN_NPN_E1B1C2E2B2C1
- C310: value 68u -> 270u
- R352, R353, R354, R355: value 10k -> 1k
Connections:
- net +5V: now also Q301.3 (D)
- net ARGB_{0}: now also R352.1; no longer R352.2
- net ARGB_{1}: now also R353.1; no longer R353.2
- net ARGB_{2}: now also R354.1; no longer R354.2
- net ARGB_{3}: now also R355.1; no longer R355.2
- net GND: now also Q302.1 (E1)
- net IS_{5V}: now also J105.1 (Pin_1), J106.1 (Pin_1), J107.1 (Pin_1), J108.1 (Pin_1)
- net PO_{5}: now also J105.2 (Pin_2), J106.2 (Pin_2), J107.2 (Pin_2), J108.2 (Pin_2), R352.2, R353.2, R354.2, R355.2, Q301.2 (S)
- net QG_{5}: now also Q301.1 (G), Q302.6 (C1)
- net VDD: no longer names the net of R350.1
- net VDD: now also Q302.2 (B1)
- no-connect marks 0 -> 3
Other:
- moved on the sheet: C350, J105, J106, J107, J108, R350, R351, R352, R353, R354, R355, R356

Commit message: Temp
Parts:
- removed D310: 30V, Diode_SMD:D_SMF, symbol Device:D_TVS_Small
- added D310: 30V, Diode_SMD:D_SMF, symbol Device:D_Zener_Small
- J105, J106, J107, J108: footprint (none) -> Bluesat:BM03B-PASS
- J320, J321: footprint (none) -> Bluesat:FG RJ-064-1
- J330: footprint (none) -> Bluesat:S2P-VH
- Q301: footprint Package_TO_SOT_SMD:SOT-23 -> Bluesat:PQFN_5x6mm_E_DGS; symbol Transistor_FET:Q_NMOS_GSD -> Transistor_FET:Q_NMOS_DGS
- Q302: footprint (none) -> Bluesat:SOT-363
- R330, R356: footprint Diode_SMD:D_2512_6332Metric -> Resistor_SMD:R_2512_6332Metric
- TR101: footprint Transformer_SMD:Transformer_Ethernet_YDS_30F-51NL_SO-24_7.1x15.1mm -> Bluesat:Transformer_Ethernet
Connections:
- net +5V: now also Q301.1 (D); no longer Q301.3 (D)
- net GND: now also D310.2 (A)
- net PO_{5}: now also Q301.3 (S); no longer Q301.2 (S)
- net QG_{5}: now also Q301.2 (G); no longer Q301.1 (G)
- net VBUS: now also D310.1 (K)
Changed lines of the file:
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@@
 			)
 		)
-		(property "Footprint" "Transformer_SMD:Transformer_Ethernet_YDS_30F-51NL_SO-24_7.1x15.1mm"
+		(property "Footprint" "Bluesat:Transformer_Ethernet"
 			(at 160.02 44.45 0)
 			(effects
@@
 			)
 		)
-		(property "Footprint" ""
+		(property "Footprint" "Bluesat:FG RJ-064-1"
 			(at 185.42 51.435 90)
 			(effects
@@
 	)
 	(symbol
+		(lib_id "Device:D_Zener_Small")
+		(at 46.99 38.1 270)
+		(unit 1)
+		(exclude_from_sim no)
+		(in_bom yes)
+		(on_board yes)
+		(dnp no)
+		(property "Reference" "D310"
+			(at 48.26 37.338 90)
+			(effects
+				(font
+					(size 1.016 1.016)
+				)
+				(justify left)
+			)
+		)
+		(property "Value" "30V"
+			(at 48.26 38.862 90)
+			(effects
+				(font
+					(size 1.016 1.016)
+				)
+				(justify left)
+			)
+		)
+		(property "Footprint" "Diode_SMD:D_SMF"
+			(at 46.99 38.1 90)
+			(effects
+				(font
+					(size 1.27 1.27)
+				)
+				(hide yes)
+			)
+		)
+		(property "Datasheet" "~"
+			(at 46.99 38.1 90)
+			(effects
+				(font
+					(size 1.27 1.27)
+				)
+				(hide yes)
+			)
+		)
+		(property "Description" "Zener diode, small symbol"
+			(at 46.99 38.1 0)
+			(effects
+				(font
+					(size 1.27 1.27)
+				)
+				(hide yes)
+			)
+		)
+		(pin "2"
+		)
+		(pin "1"
+		)
+		(instances
+			(project ""
+				(path "/294cc751-7444-4d80-b629-85aa96521600/fcae8f75-3f79-40cf-823d-66a8972288db"
+					(reference "D310")
+					(unit 1)
+				)
+			)
+		)
+	)
+	(symbol
 		(lib_id "Bluesat:C_CompactV")
 		(at 234.95 152.4 0)
@@
 			)
 		)
-		(property "Footprint" ""
+		(property "Footprint" "Bluesat:BM03B-PASS"
 			(at 86.36 96.52 0)
 			(effects
@@
 			)
 		)
-		(property "Footprint" ""
+		(property "Footprint" "Bluesat:FG RJ-064-1"
 			(at 102.87 51.435 90)
 			(effects
@@
 			)
 		)
-		(property "Footprint" ""
+		(property "Footprint" "Bluesat:SOT-363"
 			(at 50.8 104.14 0)
 			(effects
@@
 			)
 		)
-		(property "Footprint" "Diode_SMD:D_2512_6332Metric"
+		(property "Footprint" "Resistor_SMD:R_2512_6332Metric"
 			(at 66.04 115.57 0)
 			(effects
@@
 			)
 		)
-		(property "Footprint" ""
+		(property "Footprint" "Bluesat:BM03B-PASS"
 			(at 181.61 96.52 0)
 			(effects
@@
 			)
 		)
-		(property "Footprint" "Diode_SMD:D_2512_6332Metric"
+		(property "Footprint" "Resistor_SMD:R_2512_6332Metric"
 			(at 40.64 74.93 0)
 			(effects
@@
 			)
 		)
-		(property "Footprint" ""
+		(property "Footprint" "Bluesat:BM03B-PASS"
 			(at 149.86 96.52 0)
 			(effects
@@
 	)
 	(symbol
-		(lib_id "Transistor_FET:Q_NMOS_GSD")
+		(lib_id "Transistor_FET:Q_NMOS_DGS")
 		(at 58.42 100.33 0)
 		(unit 1)
@@
 			)
 		)
-		(property "Footprint" "Package_TO_SOT_SMD:SOT-23"
+		(property "Footprint" "Bluesat:PQFN_5x6mm_E_DGS"
 			(at 63.5 97.79 0)
 			(effects
@@
 			)
 		)
-		(property "Description" "N-MOSFET transistor, gate/source/drain"
+		(property "Description" "N-MOSFET transistor, drain/gate/source"
 			(at 58.42 100.33 0)
 			(effects
@@
 	)
 	(symbol
-		(lib_id "Device:D_TVS_Small")
-		(at 46.99 38.1 90)
-		(unit 1)
-		(exclude_from_sim no)
-		(in_bom yes)
-		(on_board yes)
-		(dnp no)
-		(property "Reference" "D310"
-			(at 48.26 37.465 90)
-			(effects
-				(font
-					(size 1.016 1.016)
-				)
-				(justify right)
-			)
-		)
-		(property "Value" "30V"
-			(at 48.26 38.735 90)
-			(effects
-				(font
-					(size 1.016 1.016)
-				)
-				(justify right)
-			)
-		)
-		(property "Footprint" "Diode_SMD:D_SMF"
-			(at 46.99 38.1 0)
-			(effects
-				(font
-					(size 1.27 1.27)
-				)
-				(hide yes)
-			)
-		)
-		(property "Datasheet" "~"
-			(at 46.99 38.1 0)
-			(effects
-				(font
-					(size 1.27 1.27)
-				)
-				(hide yes)
-			)
-		)
-		(property "Description" "Bidirectional transient-voltage-suppression diode, small symbol"
-			(at 46.99 38.1 0)
-			(effects
-				(font
-					(size 1.27 1.27)
-				)
-				(hide yes)
-			)
-		)
-		(pin "1"
-		)
-		(pin "2"
-		)
-		(instances
-			(project "computing-power-hub"
-				(path "/294cc751-7444-4d80-b629-85aa96521600/fcae8f75-3f79-40cf-823d-66a8972288db"
-					(reference "D310")
-					(unit 1)
-				)
-			)
-		)
-	)
-	(symbol
 		(lib_id "power:GND")
 		(at 48.26 111.76 0)
@@
 			)
 		)
-		(property "Footprint" ""
+		(property "Footprint" "Bluesat:BM03B-PASS"
 			(at 118.11 96.52 0)
 			(effects
@@
 			)
 		)
-		(property "Footprint" ""
+		(property "Footprint" "Bluesat:SOT-363"
 			(at 66.04 137.16 0)
 			(effects
@@
 			)
 		)
-		(property "Footprint" ""
+		(property "Footprint" "Bluesat:S2P-VH"
 			(at 46.99 69.85 0)
 			(effects

Commit message: Grovel human! For this is ~~the Compute~~ Power ~~Module~~.
Parts:
- removed C305: 4u7, Capacitor_SMD:C_1206_3216Metric, symbol Bluesat:C_CompactV
- removed J320, J321: RJ45, Bluesat:FG RJ-064-1, symbol Connector:RJ45
- added C308: 220n, Capacitor_SMD:C_0402_1005Metric, symbol Bluesat:C_CompactV
- added J320, J321: BM08B-PASS, Bluesat:BM08B-PASS, symbol Connector:Conn_01x08_Pin
- added Q303: SSM3K333R, Package_TO_SOT_SMD:TSOT-23, symbol Transistor_FET:Q_NMOS_DGS
- added R301: 50m, Resistor_SMD:R_1206_3216Metric, symbol Bluesat:R_CompactV
- added R302: 10k, Resistor_SMD:R_0402_1005Metric, symbol Bluesat:R_CompactV
- added R303: 100k, Resistor_SMD:R_0402_1005Metric, symbol Bluesat:R_CompactV
- Q301: value IRFH7440TRPBF -> SSM3K333R; footprint Bluesat:PQFN_5x6mm_E_DGS -> Package_TO_SOT_SMD:TSOT-23
- R356: value 20m -> 50m; footprint Resistor_SMD:R_2512_6332Metric -> Resistor_SMD:R_1206_3216Metric
Connections:
- net +12V: now also R351.1, R303.1
- net +24V: now also TR101.7 (CT); no longer R351.1, TR101.4 (CT)
- net +5V: now also Q303.1 (D); no longer C301.2, C302.2, C303.2, C304.2
- net ETH_{IA+}: now also J320.1 (Pin_1)
- net ETH_{IA-}: now also J320.2 (Pin_2)
- net ETH_{IB+}: now also TR101.19 (MX2-), J320.4 (Pin_4); no longer TR101.17 (MX3+)
- net ETH_{IB-}: now also TR101.20 (MX2+), J320.3 (Pin_3); no longer TR101.16 (MX3-)
- net ETH_{IC+}: now also TR101.16 (MX3-), J320.6 (Pin_6); no longer TR101.20 (MX2+)
- net ETH_{IC-}: now also TR101.17 (MX3+), J320.5 (Pin_5); no longer TR101.19 (MX2-)
- net ETH_{ID+}: now also TR101.13 (MX4-), J320.8 (Pin_8); no longer TR101.14 (MX4+)
- net ETH_{ID-}: now also TR101.14 (MX4+), J320.7 (Pin_7); no longer TR101.13 (MX4-)
- net ETH_{OA+}: now also TR101.3 (TD1-), J321.2 (Pin_2); no longer TR101.2 (TD1+)
- net ETH_{OA-}: now also TR101.2 (TD1+), J321.1 (Pin_1); no longer TR101.3 (TD1-)
- net ETH_{OB+}: now also TR101.6 (TD2-), J321.4 (Pin_4); no longer TR101.8 (TD3+)
- net ETH_{OB-}: now also TR101.5 (TD2+), J321.3 (Pin_3); no longer TR101.9 (TD3-)
- net ETH_{OC+}: now also TR101.9 (TD3-), J321.6 (Pin_6); no longer TR101.5 (TD2+)
- net ETH_{OC-}: now also TR101.8 (TD3+), J321.5 (Pin_5); no longer TR101.6 (TD2-)
- net ETH_{OD+}: now also TR101.12 (TD4-), J321.8 (Pin_8); no longer TR101.11 (TD4+)
- net ETH_{OD-}: now also TR101.11 (TD4+), J321.7 (Pin_7); no longer TR101.12 (TD4-)
- net GND: now also Q302.4 (E2), C308.1, R301.2; no longer C301.1, C302.1, C303.1, C304.1, C306.1, C307.1
- net IS_{19V}: now also C306.1
- net IS_{24V}: now also C307.1, TR101.4 (CT); no longer TR101.7 (CT)
- net QG_{5B}: now reaches Q302.3 (C2)
- net QG_{5B}: now also Q303.2 (G), R303.2
- net at Q302.5 (B2): now also R302.1
- net IS_{5V} renamed IS_{5VA}
- net IS_{5VA}: now also C301.2, C302.2; no longer J107.1 (Pin_1), J108.1 (Pin_1)
- net NEN_{5V} renamed NEN_{5VA}
- net PO_{5} renamed PO_{5A}
- net PO_{5A}: now also C301.1, C302.1; no longer J107.2 (Pin_2), J108.2 (Pin_2), R354.2, R355.2
- net QG_{5} renamed QG_{5A}
- new net IS_{5VB}: C303.2, C304.2, C308.2, J107.1 (Pin_1), J108.1 (Pin_1), R301.1
- new net NEN_{5VB}: R302.2
- new net PO_{5B}: C303.1, C304.1, J107.2 (Pin_2), J108.2 (Pin_2), Q303.3 (S), R354.2, R355.2
- no-connect marks 3 -> 0
Other:
- moved on the sheet: C301, C302, C303, C304, C306, C307, C320, C321, C322, C323, C324, J107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

Commit message: Fix MPM/CPM Medium NMOS symbol, DGS -> GSD
Parts:
- Q301, Q303: symbol Transistor_FET:Q_NMOS_DGS -> Transistor_FET:Q_NMOS_GSD
Connections:
- net +5V: now also Q301.3 (D), Q303.3 (D); no longer Q301.1 (D), Q303.1 (D)
- net PO_{5A}: now also Q301.2 (S); no longer Q301.3 (S)
- net PO_{5B}: now also Q303.2 (S); no longer Q303.3 (S)
- net QG_{5A}: now also Q301.1 (G); no longer Q301.2 (G)
- net QG_{5B}: now also Q303.1 (G); no longer Q303.2 (G)
Changed lines of the file:
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@@
 	)
 	(symbol
-		(lib_id "Transistor_FET:Q_NMOS_DGS")
+		(lib_id "Transistor_FET:Q_NMOS_GSD")
 		(at 58.42 100.33 0)
 		(unit 1)
@@
 			)
 		)
-		(property "Description" "N-MOSFET transistor, drain/gate/source"
+		(property "Description" "N-MOSFET transistor, gate/source/drain"
 			(at 58.42 100.33 0)
 			(effects
@@
 	)
 	(symbol
-		(lib_id "Transistor_FET:Q_NMOS_DGS")
+		(lib_id "Transistor_FET:Q_NMOS_GSD")
 		(at 149.86 100.33 0)
 		(unit 1)
@@
 			)
 		)
-		(property "Description" "N-MOSFET transistor, drain/gate/source"
+		(property "Description" "N-MOSFET transistor, gate/source/drain"
 			(at 149.86 100.33 0)
 			(effects

Commit message: aaa
Parts:
- C310: footprint Capacitor_SMD:CP_Elec_6.3x7.7 -> Capacitor_SMD:CP_Elec_10x10
- J330: footprint Bluesat:S2P-VH -> Bluesat:B2P-VH
Connections:
- net ETH_{IA+}: now also J320.8 (Pin_8); no longer J320.1 (Pin_1)
- net ETH_{IA-}: now also J320.7 (Pin_7); no longer J320.2 (Pin_2)
- net ETH_{IB+}: now also J320.5 (Pin_5); no longer J320.4 (Pin_4)
- net ETH_{IB-}: now also J320.6 (Pin_6); no longer J320.3 (Pin_3)
- net ETH_{IC+}: now also J320.3 (Pin_3); no longer J320.6 (Pin_6)
- net ETH_{IC-}: now also J320.4 (Pin_4); no longer J320.5 (Pin_5)
- net ETH_{ID+}: now also J320.1 (Pin_1); no longer J320.8 (Pin_8)
- net ETH_{ID-}: now also J320.2 (Pin_2); no longer J320.7 (Pin_7)
- net ETH_{OA+}: now also J321.7 (Pin_7); no longer J321.2 (Pin_2)
- net ETH_{OA-}: now also J321.8 (Pin_8); no longer J321.1 (Pin_1)
- net ETH_{OB+}: now also J321.5 (Pin_5); no longer J321.4 (Pin_4)
- net ETH_{OB-}: now also J321.6 (Pin_6); no longer J321.3 (Pin_3)
- net ETH_{OC+}: now also J321.3 (Pin_3); no longer J321.6 (Pin_6)
- net ETH_{OC-}: now also J321.4 (Pin_4); no longer J321.5 (Pin_5)
- net ETH_{OD+}: now also J321.1 (Pin_1); no longer J321.8 (Pin_8)
- net ETH_{OD-}: now also J321.2 (Pin_2); no longer J321.7 (Pin_7)
Other:
- moved on the sheet: J321
Changed lines of the file:
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@@
 	(wire
 		(pts
+			(xy 68.58 41.91) (xy 68.58 44.45)
+		)
+		(stroke
+			(width 0)
+			(type default)
+		)
+	)
+	(wire
+		(pts
 			(xy 152.4 53.34) (xy 146.05 53.34)
 		)
@@
 	(wire
 		(pts
-			(xy 68.58 41.91) (xy 68.58 44.45)
-		)
-		(stroke
-			(width 0)
-			(type default)
-		)
-	)
-	(wire
-		(pts
 			(xy 204.47 99.06) (xy 203.2 99.06)
 		)
@@
 			)
 		)
-		(property "Footprint" "Capacitor_SMD:CP_Elec_6.3x7.7"
+		(property "Footprint" "Capacitor_SMD:CP_Elec_10x10"
 			(at 54.61 38.1 0)
 			(effects
@@
 	(symbol
 		(lib_id "Connector:Conn_01x08_Pin")
-		(at 92.71 50.8 0)
+		(at 92.71 53.34 0)
+		(mirror x)
 		(unit 1)
 		(exclude_from_sim no)
@@
 		(on_board yes)
 		(dnp no)
-		(fields_autoplaced yes)
 		(property "Reference" "J320"
-			(at 93.345 38.1 0)
+			(at 93.345 66.04 0)
 			(effects
 				(font
@@
 		)
 		(property "Value" "BM08B-PASS"
-			(at 93.345 40.64 0)
+			(at 93.345 63.5 0)
 			(effects
 				(font
@@
 		)
 		(property "Footprint" "Bluesat:BM08B-PASS"
-			(at 92.71 50.8 0)
+			(at 92.71 53.34 0)
 			(effects
 				(font
@@
 		)
 		(property "Datasheet" "~"
-			(at 92.71 50.8 0)
+			(at 92.71 53.34 0)
 			(effects
 				(font
@@
 		)
 		(property "Description" "Generic connector, single row, 01x08, script generated"
-			(at 92.71 50.8 0)
+			(at 92.71 53.34 0)
 			(effects
 				(font
@@
 	(symbol
 		(lib_id "Connector:Conn_01x08_Pin")
-		(at 157.48 50.8 0)
-		(mirror y)
+		(at 157.48 53.34 180)
 		(unit 1)
 		(exclude_from_sim no)
@@
 		(dnp no)
 		(property "Reference" "J321"
-			(at 156.845 38.1 0)
+			(at 156.845 66.04 0)
 			(effects
 				(font
@@
 		)
 		(property "Value" "BM08B-PASS"
-			(at 156.845 40.64 0)
+			(at 156.845 63.5 0)
 			(effects
 				(font
@@
 		)
 		(property "Footprint" "Bluesat:BM08B-PASS"
-			(at 157.48 50.8 0)
+			(at 157.48 53.34 0)
 			(effects
 				(font
@@
 		)
 		(property "Datasheet" "~"
-			(at 157.48 50.8 0)
+			(at 157.48 53.34 0)
 			(effects
 				(font
@@
 		)
 		(property "Description" "Generic connector, single row, 01x08, script generated"
-			(at 157.48 50.8 0)
+			(at 157.48 53.34 0)
 			(effects
 				(font
@@
 			)
 		)
-		(property "Footprint" "Bluesat:S2P-VH"
+		(property "Footprint" "Bluesat:B2P-VH"
 			(at 46.99 69.85 0)
 			(effects

Commit message: Clean up (fix footprints, DRC etc.) for production
Other:
- company: (none) -> Bluesat OWR
- title: (none) -> Computing Power Module (CPM), a.k.a. Computing Power Hub
Changed lines of the file:
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@@
 	(generator_version "9.0")
 	(paper "A4")
+	(title_block
+		(title "Computing Power Module (CPM), a.k.a. Computing Power Hub")
+		(date "2026-02-25")
+		(rev "2.0")
+		(company "Bluesat OWR")
+	)
 	(rectangle
 		(start 25.4 86.36)
