File: src/can_converter/Can_converter_v2/PSU.kicad_sch (KiCad schematic)
At the start: 3 parts

Commit message: Rebase usb-can branch onto main
Parts:
- PS1: footprint Package_TO_SOT_SMD:SOT-23-5_HandSoldering -> Package_TO_SOT_SMD:SOT-23-5
Changed lines of the file:
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@@
 			)
 		)
-		(property "Footprint" "Package_TO_SOT_SMD:SOT-23-5_HandSoldering"
+		(property "Footprint" "Package_TO_SOT_SMD:SOT-23-5"
 			(at 152.4 209.22 0)
 			(effects
