Commit message: Add model of manipulator to URDF

File: src/rover/description/chassis/chassis.xacro (robot description, xacro)
@@ -3,14 +3,12 @@
     <xacro:property name="chassis_length" value="0.600"/>
     <xacro:property name="chassis_width" value="0.450"/>
-    <xacro:property name="chassis_height" value="0.100"/>
+    <xacro:property name="chassis_height" value="0.166"/>
     <xacro:property name="chassis_mass" value="10.0"/>
-    <!-- BASE LINK -->
-    <link name="base_link">
-    </link>
+    <xacro:property name="chassis_pivot_offset" value="-0.05"/>
     <!-- CHASSIS LINK -->
     <joint name="chassis_joint" type="fixed">
         <parent link="base_link"/>
         <child link="chassis"/>
-        <origin xyz="0 0 0"/>
+        <origin xyz="0 0 ${chassis_pivot_offset}"/>
     </joint>
     <link name="chassis">

File: src/rover/description/drivebase/drivebase.xacro (robot description, xacro)
@@ -14,5 +14,5 @@
     <!-- TODO: Fix effort and velocity limits. Current values are arbitrary. -->
     <joint name="ldb_pivot_joint" type="revolute">
-        <parent link="chassis"/>
+        <parent link="base_link"/>
         <child link="ldb_pivot"/>
         <origin xyz="0 ${chassis_width/2 + 0.014 + diff_bar_bearing_seat_width} 0" rpy="-${pi/2} 0 0" />
@@ -33,5 +33,5 @@
     <!-- TODO: Fix effort and velocity limits -->
     <joint name="rdb_pivot_joint" type="continuous">
-        <parent link="chassis"/>
+        <parent link="base_link"/>
         <child link="rdb_pivot"/>
         <origin xyz="0 -${chassis_width/2 + 0.014 + diff_bar_bearing_seat_width} 0" rpy="-${pi/2} 0 0" />

File: src/rover/description/robot.urdf.xacro (robot description, xacro)
@@ -4,5 +4,9 @@
     <xacro:include filename="utils/inertial_macros.xacro" />
     <xacro:include filename="utils/materials.xacro" />
+    <!-- BASE LINK -->
+    <link name="base_link">
+    </link>
     <xacro:include filename="chassis/chassis.xacro" />
+    <xacro:include filename="manipulator/manipulator.xacro" />
     <xacro:include filename="drivebase/drivebase.xacro" />
     <xacro:include filename="utils/gazebo_plugins.xacro" />

Commit message: Fixed up urdf for current rover design and added 3 depth cameras

File: src/rover/description/chassis/chassis.xacro (robot description, xacro)
@@ -3,5 +3,5 @@
     <xacro:property name="chassis_length" value="0.600"/>
     <xacro:property name="chassis_width" value="0.450"/>
-    <xacro:property name="chassis_height" value="0.100"/>
+    <xacro:property name="chassis_height" value="0.200"/>
     <xacro:property name="chassis_mass" value="10.0"/>
     <!-- BASE LINK -->

File: src/rover/description/drivebase/db_helpers.xacro (robot description, xacro)
@@ -2,15 +2,16 @@
 <robot xmlns:xacro="http://www.ros.org/wiki/xacro" >
     <!-- flipped = -1, normal = 1 for flip_x and isrear -->
-    <xacro:macro name="db_module_corner" params="prefix parent flip_x:=1 isrear:=1">
+	<xacro:macro name="db_module_corner" params="prefix parent flip_x:=1 isrear:=1">
+	<!-- This is the pivot point -->
         <joint name="${prefix}_joint" type="fixed">
             <parent link="${parent}"/>
             <child link="${prefix}"/>
-            <origin xyz="${isrear*(diff_bar_length/2 + 0.056/2)*cos(pi/6)} ${(diff_bar_length/2 + 0.056/2)*sin(pi/6)} 0" rpy="0 0 ${isrear*pi/6}" />
+            <origin xyz="${isrear*(diff_bar_length/2 + 0.056/2)} 0 0" rpy="0 0 0" />
         </joint>
-        <!-- TODO: Fix xyz -->
+        <!-- This is the "arms" connected to the steering joint -->
         <joint name="${prefix}_bar_smount_joint" type="fixed">
             <parent link="${prefix}"/>
             <child link="${prefix}_smount"/>
-            <origin xyz="${isrear*diff_bar_length/2} ${0.05} ${(0.0425 + 0.02975)*flip_x}" rpy="${pi/2} 0 ${isrear*(pi/-6)}" />
+            <origin xyz="${isrear*0.865/8} ${0.04} ${(0.04)*flip_x}" rpy="${pi/2} 0 0" />
         </joint>
         <!-- This is the steering joint -->
@@ -18,5 +19,5 @@
             <parent link="${prefix}_smount"/>
             <child link="${prefix}_wheel_fork"/>
-            <origin xyz="0 0 ${-0.213/2 - 0.03/2}" rpy="0 0 0" />
+	    <origin xyz="${0} ${0} ${-0.213/2 - 0.03/2}" rpy="0 0 0"/>
             <axis xyz="0 0 1"/>
             <limit lower="${-pi/2}" upper="${pi/2}" effort="40.0" velocity="12.8"/>
@@ -30,16 +31,18 @@
         </joint>
         <!-- ALL LINKS BELOW THIS LINE -->
+	<!-- arm -->
         <link name="${prefix}">
             <visual>
                 <geometry>
-                    <box size="${diff_bar_length} ${diff_bar_bearing_seat_width} ${diff_bar_bearing_seat_width}"/>
-                </geometry>
+			<box size="${0.865/2} ${diff_bar_bearing_seat_width} ${diff_bar_bearing_seat_width}"/>
+		</geometry>
+		<origin xyz="${isrear*-0.865/1.5} 0 0" rpy="0 0 0"/>
                 <material name="orange"/>
             </visual>
-            <xacro:inertial_box mass="2" x="${diff_bar_length}" y="${diff_bar_bearing_seat_width}" z="${diff_bar_bearing_seat_width}">
-                <origin xyz="0 0 0" rpy="0 0 0"/>
+	    <xacro:inertial_box mass="2" x="${0.865/2}" y="${diff_bar_bearing_seat_width}" z="${diff_bar_bearing_seat_width}">
+		    <origin xyz="${isrear*-0.865/1.5} 0 0" rpy="0 0 0"/>
             </xacro:inertial_box>
         </link>
-        <!-- Steering mount -->
+        <!-- Steering motor mount -->
         <link name="${prefix}_smount">
             <visual>
@@ -66,5 +69,5 @@
             <visual>
                 <geometry>
-                    <cylinder radius="${0.125}" length="0.150"/>
+			<cylinder radius="${wheel_radius}" length="${wheel_thickness}"/>
                 </geometry>
                 <material name="black"/>
@@ -72,5 +75,5 @@
             <collision>
                 <geometry>
-                    <sphere radius="${0.125}"/>
+                    <sphere radius="${wheel_radius}"/>
                 </geometry>
             </collision>

File: src/rover/description/drivebase/drivebase.xacro (robot description, xacro)
@@ -5,10 +5,10 @@
     <xacro:property name="diff_bar_bearing_seat_width" value="0.04"/>
     <xacro:property name="diff_bar_length" value="0.600"/>
-    <xacro:property name="wheel_radius" value="0.033"/>
-    <xacro:property name="wheel_thickness" value="0.026"/>
+    <xacro:property name="wheel_radius" value="${0.245/2}"/>
+    <xacro:property name="wheel_thickness" value="0.11"/>
     <xacro:property name="wheel_mass" value="0.05"/>
-    <xacro:property name="wheel_offset_x" value="0.226"/>
-    <xacro:property name="wheel_offset_y" value="0.3"/>
-    <xacro:property name="wheel_offset_z" value="0.01"/>
+    <xacro:property name="wheel_offset_x" value="0.29"/>
+    <xacro:property name="wheel_offset_y" value="0.4325"/>
+    <xacro:property name="wheel_offset_z" value="2"/>
     <!-- LEFT SIDE STUFF -->
     <!-- TODO: Fix effort and velocity limits. Current values are arbitrary. -->

File: src/rover/description/robot.urdf.xacro (robot description, xacro)
@@ -5,4 +5,5 @@
         <xacro:include filename="utils/bg431_motor.xacro"/>
     </xacro:unless>
+    <xacro:include filename="cameras/depth_cams.xacro" />
     <xacro:include filename="utils/inertial_macros.xacro" />
     <xacro:include filename="utils/materials.xacro" />
