File: src/stepper_driver_elec/channel.kicad_sch (KiCad schematic)
At the start: 47 parts, among them J1 Conn_01x06_Pin, J2 VH4, U10 TMC5160A-TA, U2 DMHT6016LFJ, U3 DMHT6016LFJ

Commit message: IMPERIAL SCUM
Parts:
- removed C10, C11, C15: 100n, symbol Bluesat:C_CompactV
- removed C12, C13, C14, C19: 1n, symbol Bluesat:C_CompactV
- removed C16, C6: 3n3, symbol Bluesat:C_CompactV
- removed C17, C18, C7, C8: 470n, symbol Bluesat:C_CompactV
- removed C2, C5: 270u, symbol Device:C_Polarized_Small_US
- removed C20: 2u2, symbol Bluesat:C_CompactH
- removed C21: 470n, symbol Bluesat:C_CompactH
- removed C3, C4: 4u7, symbol Bluesat:C_CompactV
- removed C67: 1u, symbol Bluesat:C_CompactH
- removed C9: 22n, symbol Bluesat:C_CompactH
- removed D8: D_TVS_Dual_Compact, symbol Bluesat:D_TVS_Quad_Compact
- removed J2: VH4, symbol Connector:Conn_01x04_Pin
- removed R1, R17: 20k, symbol Bluesat:R_CompactV
- removed R11, R12, R14, R15: 47R, symbol Bluesat:R_CompactH
- removed R13, R16: 33m, symbol Bluesat:R_CompactV
- removed R69: 10k, symbol Bluesat:R_CompactV
- removed R9: 2R2, symbol Bluesat:R_CompactV
- removed U10: TMC5160A-TA, Package_QFP:TQFP-48-1EP_7x7mm_P0.5mm_EP5x5mm_ThermalVias, symbol Bluesat:TMC5160A-TA
- removed U2, U3: DMHT6016LFJ, symbol Bluesat:DMHT6016LFJ
- added C301: 330n, Capacitor_SMD:C_0805_2012Metric, symbol Bluesat:C_CompactV
- added C302, C305, C317: 100n, Capacitor_SMD:C_0402_1005Metric, symbol Bluesat:C_CompactV
- added C303: 33n, Capacitor_SMD:C_0603_1608Metric, symbol Bluesat:C_CompactV
- added C304, C316: 3n3, Capacitor_SMD:C_0402_1005Metric, symbol Bluesat:C_CompactV
- added C306, C307, C318: 2u2, Capacitor_SMD:C_0603_1608Metric, symbol Bluesat:C_CompactV
- added C308, C309, C310, C315: 330n, Capacitor_SMD:C_0603_1608Metric, symbol Bluesat:C_CompactV
- added C311, C312, C313, C314: 1n, Capacitor_SMD:C_0402_1005Metric, symbol Bluesat:C_CompactV
- added C319, C320, C326: 220n, Capacitor_SMD:C_0402_1005Metric, symbol Bluesat:C_CompactV
- added C321: 4u7, Capacitor_SMD:C_1206_3216Metric, symbol Bluesat:C_CompactV
- added C322, C323: 270u, Capacitor_SMD:CP_Elec_10x10, symbol Device:C_Polarized_Small_US
- added C324, C325: 4u7, Capacitor_SMD:C_1210_3225Metric, symbol Bluesat:C_CompactV
- added D302: WS2812B-2020, LED_SMD:LED_WS2812B-2020_PLCC4_2.0x2.0mm, symbol LED:WS2812B-2020
- added J301: S4P-VH, Bluesat:S4P-VH, symbol Connector:Conn_01x04_Pin
- added R301: 2R2, Resistor_SMD:R_0402_1005Metric, symbol Bluesat:R_CompactH
- added R306, R309, R314, R316: 47R, Resistor_SMD:R_0402_1005Metric, symbol Bluesat:R_CompactH
- added R307: 2R2, Resistor_SMD:R_0402_1005Metric, symbol Bluesat:R_CompactV
- added R308, R315: 20m, Resistor_SMD:R_2512_6332Metric, symbol Bluesat:R_CompactV
- added R317: 2k2, Resistor_SMD:R_0402_1005Metric, symbol Bluesat:R_CompactV
- added U301, U303: DMHT6016LFJ, Bluesat:VDFN5045-12, symbol Bluesat:DMHT6016LFJ
- added U302: TMC5160A-TA, Package_QFP:TQFP-48-1EP_7x7mm_P0.5mm_EP5x5mm, symbol Bluesat:TMC5160A-TA
- D301: renamed from D7; value D_TVS_Dual_Compact -> 3V3; footprint (none) -> Package_DFN_QFN:Diodes_UDFN-10_1.0x2.5mm_P0.5mm
- J302: renamed from J1; value Conn_01x06_Pin -> BM06B-PASK; footprint (none) -> Bluesat:BM06B-PASK
- R302: renamed from R10; footprint (none) -> Resistor_SMD:R_0402_1005Metric
- R303: renamed from R2; footprint (none) -> Resistor_SMD:R_0402_1005Metric
- R304: renamed from R3; footprint (none) -> Resistor_SMD:R_0402_1005Metric
- R305: renamed from R4; footprint (none) -> Resistor_SMD:R_0402_1005Metric
- R310: renamed from R5; footprint (none) -> Resistor_SMD:R_0402_1005Metric
- R311: renamed from R6; footprint (none) -> Resistor_SMD:R_0402_1005Metric
- R312: renamed from R7; footprint (none) -> Resistor_SMD:R_0402_1005Metric
- R313: renamed from R8; footprint (none) -> Resistor_SMD:R_0402_1005Metric
- TH301: renamed from TH1; value Thermistor -> 10k; footprint (none) -> Resistor_SMD:R_0402_1005Metric
Connections:
- net +12V: now also C321.2, U302.3 (12VOUT), U302.4 (VSA)
- net CHA.C1: now also C308.2, U302.42 (CA1)
- net CHA.C2: now also C309.2, U302.35 (CA2)
- net CHA.H1: now also R302.2, U301.1 (G1_AH); no longer R302.1
- net CHA.H2: now also R304.2, U301.12 (G4_BH); no longer R304.1
- net CHA.L1: now also R303.2, U301.4 (G2_AL); no longer R303.1
- net CHA.L2: now also R305.2, U301.9 (G3_BL); no longer R305.1
- net CHA.SRH: now also C304.2, R306.1, U302.8 (SRAH)
- net CHA.SRL: now also C304.1, R309.1, U302.7 (SRAL)
- net CHB.C1: now also C310.2, U302.2 (CB1)
- net CHB.C2: now also C315.2, U302.43 (CB2)
- net CHB.H1: now also R310.2, U303.1 (G1_AH); no longer R310.1
- net CHB.H2: now also R312.2, U303.12 (G4_BH); no longer R312.1
- net CHB.L1: now also R311.2, U303.4 (G2_AL); no longer R311.1
- net CHB.L2: now also R313.2, U303.9 (G3_BL); no longer R313.1
- net CHB.SRH: now also C316.2, R314.1, U302.9 (SRBH)
- net CHB.SRL: now also C316.1, R316.1, U302.10 (SRBL)
- net CLK: now also U302.12 (CLK)
- net CSN: now also U302.13 (~{CS}/CFG3)
- net D1/D4: now also C322.1, C323.1, C324.2, C325.2, R301.1, U301.11 (D1/D4), U301.2 (D1/D4), U301.A (D1/D4), U303.11 (D1/D4), U303.2 (D1/D4), U303.A (D1/D4)
- net ENCA: now also D301.4, D301.7, J302.5 (Pin_5), U302.24 (ENCA/DCIN/CFG5); no longer D301.5, D301.6, J302.6 (Pin_6)
- net ENCB: now also D301.5, D301.6, J302.6 (Pin_6), U302.23 (ENCB/DCEN/CFG4); no longer D301.4, D301.7, J302.5 (Pin_5)
- net GND: now also C301.1, C305.1, C306.1, C307.1, C311.1, C312.1, C313.1, C314.1, C317.1, C318.1, C319.1, C320.1, C321.1, C322.2, C323.2, C324.1, C325.1, C326.1, D302.2 (VSS), R308.2, R309.2, R315.2, R316.2, R317.2, U302.11 (TST_MODE), U302.19 (GNDD), U302.21 (SD_MODE), U302.30 (GNDD), U302.49 (EP), U302.6 (GNDA)
- net MISO: now also U302.16 (SDO/CFG0)
- net MOSI: now also U302.15 (SDI/CFG1)
- net NEN: now also U302.28 (~{DRV_EN})
- net REFL: now also U302.17 (REFL/STEP)
- net REFR: now also U302.18 (REFR/DIR)
- net SCLK: now also U302.14 (SCK/CFG2)
- net STEP_DIAG: now also U302.26 (SWN/DIAG0), U302.27 (SWP/DIAG1)
- net TEMP: now also C326.2, R317.1
- net VDD: now also J302.2 (Pin_2), C318.2, C319.2, U302.20 (VCC_IO), U302.22 (SPI_MODE)
- new net: C306.2, R307.1, U302.5 (5VOUT)
- new net +5V: C320.2, D302.4 (VDD)
- new net +A: C309.1, C313.2, J301.3 (Pin_3), U301.10 (S4/D3_B), U301.C (S4/D3_B), U302.37 (BMA2)
- new net +B: C311.2, C315.1, J301.1 (Pin_1), U302.45 (BMB2), U303.10 (S4/D3_B), U303.C (S4/D3_B)
- new net -A: C308.1, C314.2, J301.4 (Pin_4), U301.3 (S1/D2_A), U301.B (S1/D2_A), U302.40 (BMA1)
- new net -B: C310.1, C312.2, J301.2 (Pin_2), U302.48 (BMB1), U303.3 (S1/D2_A), U303.B (S1/D2_A)
- new net 5V_{FLT}: C307.2, R307.2, U302.29 (VCC)
- new net ARGB_{I}: D302.3 (DIN)
- new net ARGB_{O}: D302.1 (DOUT)
- new net CHA.H1_UT: R302.1, U302.41 (HA1)
- new net CHA.H2_UT: R304.1, U302.36 (HA2)
- new net CHA.L1_UT: R303.1, U302.39 (LA1)
- new net CHA.L2_UT: R305.1, U302.38 (LA2)
- new net CHA.SRC: C305.2, R306.2, R308.1, U301.5 (S2_A), U301.6 (S2_A), U301.7 (S3_B), U301.8 (S3_B)
- new net CHB.H1_UT: R310.1, U302.1 (HB1)
- new net CHB.H2_UT: R312.1, U302.44 (HB2)
- new net CHB.L1_UT: R311.1, U302.47 (LB1)
- new net CHB.L2_UT: R313.1, U302.46 (LB2)
- new net CHB.SRC: C317.2, R314.2, R315.1, U303.5 (S2_A), U303.6 (S2_A), U303.7 (S3_B), U303.8 (S3_B)
- new net CPI: C303.1, U302.32 (CPI)
- new net CPO: C303.2, U302.31 (CPO)
- new net VCP: C302.1, U302.34 (VCP)
- new net VS: C301.2, C302.2, R301.2, U302.33 (VS)
Other:
- note added: "BW=1/(2π*2*47R*3n3)=513kHz"
- note added: "BW=1/(2π*2k2*220n)=329Hz"
- note added: "Capacitors CX01, CX03, CX08, CX09, CX10, CX15, CX24 and CX25 must be 50V rated. Capacitors CX02, CX21 must be 25V rated."
- note removed: "BW=1/(47R*2 * 3n3 * 2π=513 Hz"
- note removed: "C1, C2, C3, C4, C15, C18 must all be rated for 30V"
- note removed: "C_E"
- note removed: "Channel"
- note removed: "Gate Voltage Regulator"
- note removed: "Must be < 47k"
- moved on the sheet: D301, J302, R302, R303, R304, R305, R310, R311, R312, R313, TH301

Commit message: Re:layout
Parts:
- removed C323: 270u, Capacitor_SMD:CP_Elec_10x10, symbol Device:C_Polarized_Small_US
Connections:
- net 5V_{RAW}: now reaches C306.2, R307.1, U302.5 (5VOUT)
Other:
- moved on the sheet: C324, C325
Changed lines of the file:
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@@
 	)
 	(junction
+		(at 62.23 160.02)
+		(diameter 0)
+		(color 0 0 0 0)
+	)
+	(junction
 		(at 166.37 80.01)
 		(diameter 0)
@@
 	)
 	(junction
-		(at 60.96 160.02)
-		(diameter 0)
-		(color 0 0 0 0)
-	)
-	(junction
 		(at 93.98 93.98)
 		(diameter 0)
@@
 	)
 	(junction
-		(at 68.58 160.02)
-		(diameter 0)
-		(color 0 0 0 0)
-	)
-	(junction
 		(at 170.18 77.47)
 		(diameter 0)
@@
 	(wire
 		(pts
-			(xy 54.61 160.02) (xy 60.96 160.02)
-		)
-		(stroke
-			(width 0)
-			(type default)
-		)
-	)
-	(wire
-		(pts
 			(xy 20.32 95.25) (xy 35.56 95.25)
 		)
@@
 	(wire
 		(pts
-			(xy 68.58 162.56) (xy 68.58 160.02)
+			(xy 62.23 162.56) (xy 62.23 160.02)
 		)
 		(stroke
@@
 	(wire
 		(pts
-			(xy 68.58 160.02) (xy 60.96 160.02)
-		)
-		(stroke
-			(width 0)
-			(type default)
-		)
-	)
-	(wire
-		(pts
-			(xy 60.96 162.56) (xy 60.96 160.02)
+			(xy 54.61 160.02) (xy 62.23 160.02)
 		)
 		(stroke
@@
 	(wire
 		(pts
+			(xy 62.23 160.02) (xy 66.04 160.02)
+		)
+		(stroke
+			(width 0)
+			(type default)
+		)
+	)
+	(wire
+		(pts
 			(xy 73.66 124.46) (xy 73.66 123.19)
 		)
@@
 	(wire
 		(pts
-			(xy 68.58 160.02) (xy 72.39 160.02)
-		)
-		(stroke
-			(width 0)
-			(type default)
-		)
-	)
-	(wire
-		(pts
 			(xy 101.6 171.45) (xy 104.14 171.45)
 		)
@@
 	(wire
 		(pts
-			(xy 72.39 162.56) (xy 72.39 160.02)
+			(xy 66.04 162.56) (xy 66.04 160.02)
 		)
 		(stroke
@@
 	)
 	(label "5V_{FLT}"
-		(at 57.15 53.34 180)
+		(at 55.88 53.34 180)
 		(effects
 			(font
@@
 		)
 	)
+	(label "5V_{RAW}"
+		(at 55.88 48.26 180)
+		(effects
+			(font
+				(size 0.762 0.762)
+			)
+			(justify right bottom)
+		)
+	)
 	(label "ENCA"
 		(at 20.32 92.71 0)
@@
 		(on_board yes)
 		(dnp no)
-		(fields_autoplaced yes)
 		(property "Reference" "C326"
 			(at 100.711 175.768 90)
@@
 	(symbol
 		(lib_id "power:GND")
-		(at 68.58 167.64 0)
+		(at 62.23 167.64 0)
 		(unit 1)
 		(exclude_from_sim no)
@@
 		(dnp no)
 		(property "Reference" "#PWR0336"
-			(at 68.58 173.99 0)
+			(at 62.23 173.99 0)
 			(effects
 				(font
@@
 		)
 		(property "Value" "GND"
-			(at 68.58 170.942 0)
+			(at 62.23 170.942 0)
 			(effects
 				(font
@@
 		)
 		(property "Footprint" ""
-			(at 68.58 167.64 0)
+			(at 62.23 167.64 0)
 			(effects
 				(font
@@
 		)
 		(property "Datasheet" ""
-			(at 68.58 167.64 0)
+			(at 62.23 167.64 0)
 			(effects
 				(font
@@
 		)
 		(property "Description" "Power symbol creates a global label with name \"GND\" , ground"
-			(at 68.58 167.64 0)
+			(at 62.23 167.64 0)
 			(effects
 				(font
@@
 	(symbol
 		(lib_id "power:GND")
-		(at 72.39 167.64 0)
+		(at 66.04 167.64 0)
 		(unit 1)
 		(exclude_from_sim no)
@@
 		(dnp no)
 		(property "Reference" "#PWR0337"
-			(at 72.39 173.99 0)
+			(at 66.04 173.99 0)
 			(effects
 				(font
@@
 		)
 		(property "Value" "GND"
-			(at 72.39 170.942 0)
+			(at 66.04 170.942 0)
 			(effects
 				(font
@@
 		)
 		(property "Footprint" ""
-			(at 72.39 167.64 0)
+			(at 66.04 167.64 0)
 			(effects
 				(font
@@
 		)
 		(property "Datasheet" ""
-			(at 72.39 167.64 0)
+			(at 66.04 167.64 0)
 			(effects
 				(font
@@
 		)
 		(property "Description" "Power symbol creates a global label with name \"GND\" , ground"
-			(at 72.39 167.64 0)
+			(at 66.04 167.64 0)
 			(effects
 				(font
@@
 	(symbol
 		(lib_id "Bluesat:C_CompactV")
-		(at 72.39 165.1 0)
+		(at 66.04 165.1 0)
 		(unit 1)
 		(exclude_from_sim no)
@@
 		(fields_autoplaced yes)
 		(property "Reference" "C325"
-			(at 71.501 164.338 90)
+			(at 65.151 164.338 90)
 			(do_not_autoplace yes)
 			(effects
@@
 		)
 		(property "Value" "4u7"
-			(at 73.279 164.338 90)
+			(at 66.929 164.338 90)
 			(do_not_autoplace yes)
 			(effects
@@
 		)
 		(property "Footprint" "Capacitor_SMD:C_1210_3225Metric"
-			(at 72.39 165.1 90)
+			(at 66.04 165.1 90)
 			(effects
 				(font
@@
 		)
 		(property "Datasheet" "~"
-			(at 72.39 165.1 90)
+			(at 66.04 165.1 90)
 			(effects
 				(font
@@
 		)
 		(property "Description" "Unpolarized capacitor, compact symbol"
-			(at 72.39 165.1 0)
+			(at 66.04 165.1 0)
 			(effects
 				(font
@@
 	)
 	(symbol
-		(lib_id "Device:C_Polarized_Small_US")
-		(at 60.96 165.1 0)
-		(unit 1)
-		(exclude_from_sim no)
-		(in_bom yes)
-		(on_board yes)
-		(dnp no)
-		(property "Reference" "C323"
-			(at 61.214 162.052 0)
-			(effects
-				(font
-					(size 1.016 1.016)
-				)
-				(justify left)
-			)
-		)
-		(property "Value" "270u"
-			(at 61.214 163.576 0)
-			(effects
-				(font
-					(size 1.016 1.016)
-				)
-				(justify left)
-			)
-		)
-		(property "Footprint" "Capacitor_SMD:CP_Elec_10x10"
-			(at 60.96 165.1 0)
-			(effects
-				(font
-					(size 1.27 1.27)
-				)
-				(hide yes)
-			)
-		)
-		(property "Datasheet" "~"
-			(at 60.96 165.1 0)
-			(effects
-				(font
-					(size 1.27 1.27)
-				)
-				(hide yes)
-			)
-		)
-		(property "Description" "Polarized capacitor, small US symbol"
-			(at 60.96 165.1 0)
-			(effects
-				(font
-					(size 1.27 1.27)
-				)
-				(hide yes)
-			)
-		)
-		(pin "2"
-		)
-		(pin "1"
-		)
-		(instances
-			(project "stepper-driver"
-				(path "/22ad96d7-4eff-4ee6-90ff-f4a9952d1282/2cef1f8a-4b90-4951-aa93-aa8829702e75"
-					(reference "C323")
-					(unit 1)
-				)
-				(path "/22ad96d7-4eff-4ee6-90ff-f4a9952d1282/738e42ff-f14e-468b-9899-23383737ec06"
-					(reference "C423")
-					(unit 1)
-				)
-				(path "/22ad96d7-4eff-4ee6-90ff-f4a9952d1282/d626509a-f966-4c5a-b45d-5fadd303ffda"
-					(reference "C623")
-					(unit 1)
-				)
-				(path "/22ad96d7-4eff-4ee6-90ff-f4a9952d1282/dbb20285-96b5-4155-a55f-44c759eb4683"
-					(reference "C523")
-					(unit 1)
-				)
-			)
-		)
-	)
-	(symbol
 		(lib_id "power:+12V")
 		(at 46.99 158.75 0)
@@
 	(symbol
 		(lib_id "Bluesat:C_CompactV")
-		(at 68.58 165.1 0)
+		(at 62.23 165.1 0)
 		(unit 1)
 		(exclude_from_sim no)
@@
 		(fields_autoplaced yes)
 		(property "Reference" "C324"
-			(at 67.691 164.338 90)
+			(at 61.341 164.338 90)
 			(do_not_autoplace yes)
 			(effects
@@
 		)
 		(property "Value" "4u7"
-			(at 69.469 164.338 90)
+			(at 63.119 164.338 90)
 			(do_not_autoplace yes)
 			(effects
@@
 		)
 		(property "Footprint" "Capacitor_SMD:C_1210_3225Metric"
-			(at 68.58 165.1 90)
+			(at 62.23 165.1 90)
 			(effects
 				(font
@@
 		)
 		(property "Datasheet" "~"
-			(at 68.58 165.1 90)
+			(at 62.23 165.1 90)
 			(effects
 				(font
@@
 		)
 		(property "Description" "Unpolarized capacitor, compact symbol"
-			(at 68.58 165.1 0)
+			(at 62.23 165.1 0)
 			(effects
 				(font
@@
 					(unit 1)
 				)
-			)
-		)
-	)
-	(symbol
-		(lib_id "power:GND")
-		(at 60.96 167.64 0)
-		(unit 1)
-		(exclude_from_sim no)
-		(in_bom yes)
-		(on_board yes)
-		(dnp no)
-		(property "Reference" "#PWR0335"
-			(at 60.96 173.99 0)
-			(effects
-				(font
-					(size 1.27 1.27)
-				)
-				(hide yes)
-			)
-		)
-		(property "Value" "GND"
-			(at 60.96 170.942 0)
-			(effects
-				(font
-					(size 0.762 0.762)
-				)
-			)
-		)
-		(property "Footprint" ""
-			(at 60.96 167.64 0)
-			(effects
-				(font
-					(size 1.27 1.27)
-				)
-				(hide yes)
-			)
-		)
-		(property "Datasheet" ""
-			(at 60.96 167.64 0)
-			(effects
-				(font
-					(size 1.27 1.27)
-				)
-				(hide yes)
-			)
-		)
-		(property "Description" "Power symbol creates a global label with name \"GND\" , ground"
-			(at 60.96 167.64 0)
-			(effects
-				(font
-					(size 1.27 1.27)
-				)
-				(hide yes)
-			)
-		)
-		(pin "1"
-		)
-		(instances
-			(project "stepper-driver"
-				(path "/22ad96d7-4eff-4ee6-90ff-f4a9952d1282/2cef1f8a-4b90-4951-aa93-aa8829702e75"
-					(reference "#PWR0335")
-					(unit 1)
-				)
-				(path "/22ad96d7-4eff-4ee6-90ff-f4a9952d1282/738e42ff-f14e-468b-9899-23383737ec06"
-					(reference "#PWR0435")
-					(unit 1)
-				)
-				(path "/22ad96d7-4eff-4ee6-90ff-f4a9952d1282/d626509a-f966-4c5a-b45d-5fadd303ffda"
-					(reference "#PWR0635")
-					(unit 1)
-				)
-				(path "/22ad96d7-4eff-4ee6-90ff-f4a9952d1282/dbb20285-96b5-4155-a55f-44c759eb4683"
-					(reference "#PWR0535")
-					(unit 1)
-				)

Commit message: Resolve issues on the stepper board found in initial testing
Parts:
- D302: footprint LED_SMD:LED_WS2812B-2020_PLCC4_2.0x2.0mm -> Bluesat:WS2812B-2020
- J302: footprint Bluesat:BM06B-PASK -> Bluesat:BM06B-PASS
- U302: footprint Package_QFP:TQFP-48-1EP_7x7mm_P0.5mm_EP5x5mm -> Bluesat:TQFP-48-0.5-EP
Changed lines of the file:
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@@
 			)
 		)
-		(property "Footprint" "LED_SMD:LED_WS2812B-2020_PLCC4_2.0x2.0mm"
+		(property "Footprint" "Bluesat:WS2812B-2020"
 			(at 140.97 172.72 0)
 			(effects
@@
 			)
 		)
-		(property "Footprint" "Bluesat:BM06B-PASK"
+		(property "Footprint" "Bluesat:BM06B-PASS"
 			(at 15.24 87.63 0)
 			(effects
@@
 			)
 		)
-		(property "Footprint" "Package_QFP:TQFP-48-1EP_7x7mm_P0.5mm_EP5x5mm"
+		(property "Footprint" "Bluesat:TQFP-48-0.5-EP"
 			(at 76.2 127 0)
 			(effects
