File: src/usb_power_board/powerboard.kicad_sch (KiCad schematic)
At the start: 64 parts, among them J201 XT30M, Q201 40N06D, Q202 40N06D, Q203 40N06D, Q204 40N06D, U201 TPS565201, U202 LM5148, U203 TPS565201, U204 LM5148

Commit message: [GIT] Unfuck Sean's git smh
Parts:
- U202, U204: footprint Package_DFN_QFN:Texas_RGY_R-PVQFN-N24_EP2.05x3.1mm -> Bluesat:RGY0024E-MFG; symbol Bluesat:LM5148_USB_Board -> Bluesat:LM5148
Changed lines of the file:
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@@
 	)
 	(symbol
-		(lib_id "Bluesat:LM5148_USB_Board")
+		(lib_id "Bluesat:LM5148")
 		(at 168.91 67.31 0)
 		(unit 1)
@@
 			)
 		)
-		(property "Footprint" "Package_DFN_QFN:Texas_RGY_R-PVQFN-N24_EP2.05x3.1mm"
+		(property "Footprint" "Bluesat:RGY0024E-MFG"
 			(at 168.91 67.31 0)
 			(effects
@@
 	)
 	(symbol
-		(lib_id "Bluesat:LM5148_USB_Board")
+		(lib_id "Bluesat:LM5148")
 		(at 66.04 67.31 0)
 		(unit 1)
@@
 			)
 		)
-		(property "Footprint" "Package_DFN_QFN:Texas_RGY_R-PVQFN-N24_EP2.05x3.1mm"
+		(property "Footprint" "Bluesat:RGY0024E-MFG"
 			(at 66.04 67.31 0)
 			(effects
