File: src/usb_power_board/usb_power_board.kicad_sch (KiCad schematic)
At the start: 3 parts, among them J101 USB_C_Receptacle

Commit message: aaavin's changes
Parts:
- J101: footprint Connector_USB:USB_C_Receptacle_Amphenol_12401548E4-2A -> Bluesat:USB_C_Receptacle_24P
Other:
- note removed: "FIND REAL FOOTPRINT"
Changed lines of the file:
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@@
 	(generator_version "9.0")
 	(paper "A4")
-	(text "FIND REAL FOOTPRINT"
-		(exclude_from_sim no)
-		(at 158.75 84.582 0)
-		(effects
-			(font
-				(size 1.27 1.27)
-			)
-		)
-	)
 	(junction
 		(at 69.85 85.09)
@@
 			)
 		)
-		(property "Footprint" "Connector_USB:USB_C_Receptacle_Amphenol_12401548E4-2A"
+		(property "Footprint" "Bluesat:USB_C_Receptacle_24P"
 			(at 154.94 114.3 0)
 			(effects
