File: src/usb_power_board_elec/powerboard.kicad_sch (KiCad schematic)
At the start: 64 parts, among them J201 XT30M, Q201 40N06D, Q202 40N06D, Q203 40N06D, Q204 40N06D, U201 TPS565201, U202 LM5148, U203 TPS565201, U204 LM5148

Commit message: hopefully evan hasn't landed yet
Parts:
- Q201, Q202, Q203, Q204: footprint Package_DFN_QFN:DFN-8-1EP_3x3mm_P0.65mm_EP1.55x2.4mm -> Bluesat:PQFN_5x6mm_E_DGS
Changed lines of the file:
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@@
 			)
 		)
-		(property "Footprint" "Package_DFN_QFN:DFN-8-1EP_3x3mm_P0.65mm_EP1.55x2.4mm"
+		(property "Footprint" "Bluesat:PQFN_5x6mm_E_DGS"
 			(at 203.2 66.04 0)
 			(effects
@@
 			)
 		)
-		(property "Footprint" "Package_DFN_QFN:DFN-8-1EP_3x3mm_P0.65mm_EP1.55x2.4mm"
+		(property "Footprint" "Bluesat:PQFN_5x6mm_E_DGS"
 			(at 100.33 78.74 0)
 			(effects
@@
 			)
 		)
-		(property "Footprint" "Package_DFN_QFN:DFN-8-1EP_3x3mm_P0.65mm_EP1.55x2.4mm"
+		(property "Footprint" "Bluesat:PQFN_5x6mm_E_DGS"
 			(at 203.2 78.74 0)
 			(effects
@@
 			)
 		)
-		(property "Footprint" "Package_DFN_QFN:DFN-8-1EP_3x3mm_P0.65mm_EP1.55x2.4mm"
+		(property "Footprint" "Bluesat:PQFN_5x6mm_E_DGS"
 			(at 100.33 66.04 0)
 			(effects

Commit message: GG Sean
Parts:
- removed Q201, Q202, Q203, Q204: 40N06D, Bluesat:PQFN_5x6mm_E_DGS, symbol Transistor_FET:Q_NMOS_GSD
- added Q1, Q2, Q3, Q4: IRFH7440TRPBF, symbol Transistor_FET:Q_NMOS_DGS
Connections:
- net GND: now also Q2.3 (S), Q4.3 (S)
- net HO_{12V}: now also Q1.2 (G)
- net HO_{5V}: now also Q3.2 (G)
- net LO_{12V}: now also Q2.2 (G)
- net LO_{5V}: now also Q4.2 (G)
- net SW_{12V}: now also Q1.3 (S), Q2.1 (D)
- net SW_{5V}: now also Q3.3 (S), Q4.1 (D)
- net VBUS: now also Q1.1 (D), Q3.1 (D)
