File: src/usb_power_board_elec/STM_memory.kicad_sch (KiCad schematic)
At the start: 46 parts, among them J301 SM02B-PASS, J302 IDC6, U301 STM32G474, U302 ZD24C128A, U303 TCAN1462V, Y301 24Mhz

Commit message: Fix routing around STM32 / fix IDC6
Connections:
- net DBG.NRST: now also J302.5 (Pin_5); no longer J302.6 (Pin_6)
- net DBG.SWCLK: now also J302.1 (Pin_1); no longer J302.2 (Pin_2)
- net DBG.SWDIO: now also J302.2 (Pin_2); no longer J302.1 (Pin_1)
- net DBG.SWO: now also J302.6 (Pin_6); no longer J302.5 (Pin_5)
- net GND: now also J302.4 (Pin_4); no longer J302.3 (Pin_3)
- net VDD: now also J302.3 (Pin_3); no longer J302.4 (Pin_4)
Changed lines of the file:
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@@
 	(symbol
 		(lib_id "Connector_Generic:Conn_02x03_Odd_Even")
-		(at 54.61 128.27 0)
+		(at 57.15 128.27 0)
+		(mirror y)
 		(unit 1)
 		(exclude_from_sim no)
@@
 		)
 		(property "Footprint" "Bluesat:IDC6"
-			(at 54.61 128.27 0)
+			(at 57.15 128.27 0)
 			(effects
 				(font
@@
 		)
 		(property "Datasheet" "~"
-			(at 54.61 128.27 0)
+			(at 57.15 128.27 0)
 			(effects
 				(font
@@
 		)
 		(property "Description" "Generic connector, double row, 02x03, odd/even pin numbering scheme (row 1 odd numbers, row 2 even numbers), script generated (kicad-library-utils/schlib/autogen/connector/)"
-			(at 54.61 128.27 0)
+			(at 57.15 128.27 0)
 			(effects
 				(font

Commit message: [ELEC] REV markers on all PCB's, Fix USB hub passives
Add mounting holes to all PCB schematics
Parts:
- C304: value 220n -> 10n
- R301: value 10K -> 1k
- R307: value 100R -> 470R
- U301: footprint LQFP64-10x10mm -> (none)
Changed lines of the file:
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@@
 			)
 		)
-		(property "Value" "220n"
+		(property "Value" "10n"
 			(at 78.359 105.918 90)
 			(do_not_autoplace yes)
@@
 			)
 		)
-		(property "Footprint" "LQFP64-10x10mm"
+		(property "Footprint" ""
 			(at 101.6 63.5 0)
 			(effects
@@
 			)
 		)
-		(property "Footprint" "LQFP64-10x10mm"
+		(property "Footprint" ""
 			(at 52.07 161.29 0)
 			(effects
@@
 			)
 		)
-		(property "Value" "100R"
+		(property "Value" "470R"
 			(at 68.58 81.28 0)
 			(do_not_autoplace yes)
@@
 			)
 		)
-		(property "Value" "10K"
+		(property "Value" "1k"
 			(at 66.04 29.21 90)
 			(do_not_autoplace yes)

Commit message: Fix rotated IDC6 on CPM/MPM/VESC/Stepper/USB Hub (#120)
* Fix rotated IDC6 on CPM/MPM/VESC/Stepper/USB Hub

* Fix VESC
Connections:
- net DBG.NRST: now also J302.2 (Pin_2); no longer J302.5 (Pin_5)
- net DBG.SWCLK: now also J302.6 (Pin_6); no longer J302.1 (Pin_1)
- net DBG.SWDIO: now also J302.5 (Pin_5); no longer J302.2 (Pin_2)
- net DBG.SWO: now also J302.1 (Pin_1); no longer J302.6 (Pin_6)
- net GND: now also J302.3 (Pin_3); no longer J302.4 (Pin_4)
- net VDD: now also J302.4 (Pin_4); no longer J302.3 (Pin_3)
Changed lines of the file:
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@@
 	(symbol
 		(lib_id "Connector_Generic:Conn_02x03_Odd_Even")
-		(at 57.15 128.27 0)
-		(mirror y)
+		(at 54.61 128.27 0)
+		(mirror x)
 		(unit 1)
 		(exclude_from_sim no)
@@
 		(dnp no)
 		(property "Reference" "J302"
-			(at 55.88 120.65 0)
+			(at 55.88 135.89 0)
 			(effects
 				(font
@@
 		)
 		(property "Value" "IDC6"
-			(at 55.88 123.19 0)
+			(at 55.88 133.35 0)
 			(effects
 				(font
@@
 		)
 		(property "Footprint" "Bluesat:IDC6"
-			(at 57.15 128.27 0)
+			(at 54.61 128.27 0)
 			(effects
 				(font
@@
 		)
 		(property "Datasheet" "~"
-			(at 57.15 128.27 0)
+			(at 54.61 128.27 0)
 			(effects
 				(font
@@
 		)
 		(property "Description" "Generic connector, double row, 02x03, odd/even pin numbering scheme (row 1 odd numbers, row 2 even numbers), script generated (kicad-library-utils/schlib/autogen/connector/)"
-			(at 57.15 128.27 0)
+			(at 54.61 128.27 0)
 			(effects
 				(font

Commit message: Fix can trans on UPB
Connections:
- net GND: now also U303.8 (STB)
- net VDD: no longer U303.8 (STB)
Changed lines of the file:
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@@
+	(wire
+		(pts
+			(xy 60.96 99.06) (xy 62.23 99.06)
+		)
+		(stroke
+			(width 0)
+			(type default)
+		)
+	)
 	(wire
 		(pts
@@
 	(wire
 		(pts
+			(xy 62.23 99.06) (xy 62.23 102.87)
+		)
+		(stroke
+			(width 0)
+			(type default)
+		)
+	)
+	(wire
+		(pts
 			(xy 41.91 181.61) (xy 40.64 181.61)
 		)
@@
 	(wire
 		(pts
-			(xy 62.23 99.06) (xy 62.23 88.9)
-		)
-		(stroke
-			(width 0)
-			(type default)
-		)
-	)
-	(wire
-		(pts
 			(xy 76.2 160.02) (xy 81.28 160.02)
 		)
@@
 		(pts
 			(xy 163.83 73.66) (xy 163.83 74.93)
-		)
-		(stroke
-			(width 0)
-			(type default)
-		)
-	)
-	(wire
-		(pts
-			(xy 60.96 99.06) (xy 62.23 99.06)
 		)
 		(stroke
@@
 	)
 	(symbol
-		(lib_id "power:VDD")
-		(at 62.23 88.9 0)
-		(unit 1)
-		(exclude_from_sim no)
-		(in_bom yes)
-		(on_board yes)
-		(dnp no)
-		(property "Reference" "#PWR0325"
-			(at 62.23 92.71 0)
-			(effects
-				(font
-					(size 1.27 1.27)
-				)
-				(hide yes)
-			)
-		)
-		(property "Value" "VDD"
-			(at 62.23 85.725 0)
-			(effects
-				(font
-					(size 1.016 1.016)
-				)
-			)
-		)
-		(property "Footprint" ""
-			(at 62.23 88.9 0)
-			(effects
-				(font
-					(size 1.27 1.27)
-				)
-				(hide yes)
-			)
-		)
-		(property "Datasheet" ""
-			(at 62.23 88.9 0)
-			(effects
-				(font
-					(size 1.27 1.27)
-				)
-				(hide yes)
-			)
-		)
-		(property "Description" "Power symbol creates a global label with name \"VDD\""
-			(at 62.23 88.9 0)
-			(effects
-				(font
-					(size 1.27 1.27)
-				)
-				(hide yes)
-			)
-		)
-		(pin "1"
-		)
-		(instances
-			(project "usb_power_board"
-				(path "/922f9068-b2a9-46a1-aa76-e40e554fdd94/a12047df-37ee-456f-980c-409a1d825304"
-					(reference "#PWR0325")
-					(unit 1)
-				)
-			)
-		)
-	)
-	(symbol
 		(lib_id "Bluesat:R_CompactV")
 		(at 134.62 62.23 0)
@@
 					(unit 1)
 				)
+			)
+		)
+	)
+	(symbol
+		(lib_id "power:GND")
+		(at 62.23 102.87 0)
+		(unit 1)
+		(exclude_from_sim no)
+		(in_bom yes)
+		(on_board yes)
+		(dnp no)
+		(property "Reference" "#PWR0325"
+			(at 62.23 109.22 0)
+			(effects
+				(font
+					(size 1.27 1.27)
+				)
+				(hide yes)
+			)
+		)
+		(property "Value" "GND"
+			(at 62.23 106.045 0)
+			(effects
+				(font
+					(size 0.762 0.762)
+				)
+			)
+		)
+		(property "Footprint" ""
+			(at 62.23 102.87 0)
+			(effects
+				(font
+					(size 1.27 1.27)
+				)
+				(hide yes)
+			)
+		)
+		(property "Datasheet" ""
+			(at 62.23 102.87 0)
+			(effects
+				(font
+					(size 1.27 1.27)
+				)
+				(hide yes)
+			)
+		)
+		(property "Description" "Power symbol creates a global label with name \"GND\" , ground"
+			(at 62.23 102.87 0)
+			(effects
+				(font
+					(size 1.27 1.27)
+				)
+				(hide yes)
+			)
+		)
+		(pin "1"
+		)
+		(instances
+			(project "usb_power_board"
+				(path "/922f9068-b2a9-46a1-aa76-e40e554fdd94/a12047df-37ee-456f-980c-409a1d825304"
+					(reference "#PWR0325")
+					(unit 1)
+				)
