File: src/owr_wifi_router/_autosave-owr_wifi_router.kicad_sch (KiCad schematic)
At the start: 129 parts, among them U1 MT7981B_BGA

Commit message: Began work on DC-DC
Parts:
- removed CD1, CD16, CD17, CD21, CD22: 10uF, 0402, symbol 1-altium-import:root_0_CAPACITOR-DOT
- removed CD10, CD12, CD14, CD19, CD2: 1uF, 0402, symbol 1-altium-import:root_0_CAPACITOR-DOT
- removed CD11, CD13, CD15, CD18, CD20, CD23, CD24, CD25, CD26, CD27, CD28, CD29, CD3, CD30, CD31, CD32, CD33, CD34, CD36, CD37, CD4, CD5, CD8, CD9: 104, 0402, symbol 1-altium-import:root_0_CAPACITOR-DOT
- removed CD35: 22uF, 0402, symbol 1-altium-import:root_0_CAPACITOR-DOT
- removed CD6: 104, 0402, symbol 1-altium-import:root_3_CAPACITOR-DOT
- removed CD7: N~{C}104, 0402, symbol 1-altium-import:root_3_CAPACITOR-DOT
- removed CP1, CP9: 10uF, C0402, symbol 1-altium-import:root_2_mirrored_CAPACITOR-NonPole
- removed CP10, CP3: 10uF, C0402, symbol 1-altium-import:root_1_mirrored_CAPACITOR-NonPole
- removed CP11, CP5, CP6: 104, C0402, symbol 1-altium-import:root_0_CAPACITOR-NonPole
- removed CP2: 10uF, C0402, symbol 1-altium-import:root_0_CAPACITOR-NonPole
- removed CP4: 22pF, C0402, symbol 1-altium-import:root_0_CAPACITOR-NonPole
- removed CP7: 22uF, 0402, symbol 1-altium-import:root_0_mirrored_CAPACITOR-DOT
- removed CP8: 104, 0402, symbol 1-altium-import:root_0_mirrored_CAPACITOR-DOT
- removed L1: MWSA0402S-2R2MT, IND0402S, symbol 1-altium-import:root_1_INDUCTOR
- removed RD1, RD14, RD15: 0R, R0603, symbol 1-altium-import:root_1_R_Dup2
- removed RD10: 100R-1%, R0402/SMD, symbol 1-altium-import:root_0_mirrored_R0402_1
- removed RD11, RD7: N~{C}680R, R0402/SMD, symbol 1-altium-import:root_0_mirrored_R0402_1
- removed RD12, RD13: 10K-1%, R0402/SMD, symbol 1-altium-import:root_0_mirrored_R0402_1
- removed RD2, RD3: 56R-1%, R0402/SMD, symbol 1-altium-import:root_0_mirrored_R0402_1
- removed RD4, RD5: 1K-1%, R0402/SMD, symbol 1-altium-import:root_3_mirrored_R0402_1
- removed RD6: 10K-1%, R0402/SMD, symbol 1-altium-import:root_3_mirrored_R0402_1
- removed RD8: 240R-1%, R0402/SMD, symbol 1-altium-import:root_3_mirrored_R0402_1
- removed RD9: 22R, R0402/SMD, symbol 1-altium-import:root_3_mirrored_R0402_1
- removed RP1, RP9: 10K, R-0603, symbol 1-altium-import:root_1_Resistance-00_Dup2
- removed RP10: 10K-1%, R-0603, symbol 1-altium-import:root_1_mirrored_Resistance-00_Dup2
- removed RP11, RP4: 20K-1%, R-0603, symbol 1-altium-import:root_2_Resistance-00_Dup2
- removed RP2: 43K2-1%, R-0603, symbol 1-altium-import:root_1_mirrored_Resistance-00_Dup2
- removed RP3: 100K-1%, R0402, symbol 1-altium-import:root_1_RESISTOR
- removed RP5, RP6: 100K-1%, R-0603, symbol 1-altium-import:root_2_Resistance-00_Dup2
- removed RP7: NC, R0402, symbol 1-altium-import:root_1_RESISTOR
- removed RP8: N~{C}0R, R0603, symbol 1-altium-import:root_1_R_Dup2
- removed TP1, TP2, TP3: N~{C}VDDFB-CPUB, stp30, symbol 1-altium-import:root_3_T_POINT_R
- removed TPD1, TPD10, TPD11, TPD12, TPD13, TPD14, TPD15, TPD16, TPD17, TPD18, TPD19, TPD2, TPD20, TPD21, TPD22, TPD23, TPD24, TPD25, TPD26, TPD27, TPD28, TPD29, TPD3, TPD30, TPD31, TPD32, TPD4, TPD5, TPD6, TPD7, TPD8, TPD9: NC, TP0_3mm, symbol 1-altium-import:root_2_TP-SMD_1
- removed U1: MT7981B_BGA, MT7981_TFBGA338, symbol 1-altium-import:root_0_MT7981B_BGA
- removed UD1: NT5AD512M16C4-JR, FBGA96-9X14, symbol 1-altium-import:root_0_DDR4_0
- removed UP1: AP7366-W5-7, SOT23-5, symbol 1-altium-import:root_0_SGM2032
- removed UP2: SY8089AAAC, SOT23-5, symbol 1-altium-import:root_0_SY8089AAC
- removed UP3: N~{C}AP7366-W5-7, SOT23-5, symbol 1-altium-import:root_0_SGM2032
Connections:
- no-connect marks 1 -> 0
Other:
- added sheet POE_step_down (POE_step_down_sch.kicad_sch)
- note removed: "100R"
- note removed: "DRAM"
- note removed: "Doesn't include interaction with NAND/NOR flash yet"
- moved on the sheet: C?, J?, R?, TR?
