File: src/owr_wifi_router/ethernet_phy.kicad_sch (KiCad schematic)
At the start: 1 part, among them U16 DP83TG720S-Q1

Commit message: progress
Parts:
- removed U16: DP83TG720S-Q1, Package_DFN_QFN:Texas_RHH0036C_VQFN-36-1EP_6x6mm_P0.5mm_EP4.4x4.4mm, symbol Bluesat:DP83TG720S-Q1
Other:
- note added: "Accidentally found automotive ethernet phy. FInd 2.5G normal one."
Changed lines of the file:
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@@
 	(generator_version "9.0")
 	(paper "A4")
-	(symbol
-		(lib_id "Bluesat:DP83TG720S-Q1")
-		(at 73.66 66.04 0)
-		(unit 1)
+	(text "Accidentally found automotive ethernet phy. FInd 2.5G normal one."
 		(exclude_from_sim no)
-		(in_bom yes)
-		(on_board yes)
-		(dnp no)
-		(fields_autoplaced yes)
-		(property "Reference" "U16"
-			(at 106.2833 22.86 0)
-			(effects
-				(font
-					(size 1.27 1.27)
-				)
-				(justify left)
+		(at 70.612 44.704 0)
+		(effects
+			(font
+				(size 1.27 1.27)
+				(thickness 0.254)
+				(bold yes)
 			)
 		)
-		(property "Value" "DP83TG720S-Q1"
-			(at 106.2833 25.4 0)
-			(effects
-				(font
-					(size 1.27 1.27)
-				)
-				(justify left)
-			)
-		)
-		(property "Footprint" "Package_DFN_QFN:Texas_RHH0036C_VQFN-36-1EP_6x6mm_P0.5mm_EP4.4x4.4mm"
-			(at 69.596 128.778 0)
-			(effects
-				(font
-					(size 1.27 1.27)
-				)
-				(hide yes)
-			)
-		)
-		(property "Datasheet" "https://www.ti.com/lit/ds/symlink/dp83tg720s-q1.pdf?ts=1764383753180&ref_url=https%253A%252F%252Fwww.ti.com%252Fproduct%252FDP83TG720S-Q1"
-			(at 72.898 123.444 0)
-			(effects
-				(font
-					(size 1.27 1.27)
-				)
-				(hide yes)
-			)
-		)
-		(property "Description" ""
-			(at 73.66 66.04 0)
-			(effects
-				(font
-					(size 1.27 1.27)
-				)
-				(hide yes)
-			)
-		)
-		(pin "32"
-		)
-		(pin "20"
-		)
-		(pin "29"
-		)
-		(pin "34"
-		)
-		(pin "36"
-		)
-		(pin "3"
-		)
-		(pin "6"
-		)
-		(pin "15"
-		)
-		(pin "9"
-		)
-		(pin "1"
-		)
-		(pin "26"
-		)
-		(pin "28"
-		)
-		(pin "31"
-		)
-		(pin "35"
-		)
-		(pin "27"
-		)
-		(pin "23"
-		)
-		(pin "33"
-		)
-		(pin "2"
-		)
-		(pin "25"
-		)
-		(pin "24"
-		)
-		(pin "5"
-		)
-		(pin "22"
-		)
-		(pin "21"
-		)
-		(pin "7"
-		)
-		(pin "30"
-		)
-		(pin "5"
-		)
-		(pin "8"
-		)
-		(pin "19"
-		)
-		(pin "18"
-		)
-		(pin "16"
-		)
-		(pin "14"
-		)
-		(pin "17"
-		)
-		(pin "13"
-		)
-		(pin "12"
-		)
-		(pin "11"
-		)
-		(pin "10"
-		)
-		(pin "37"
-		)
-		(instances
-			(project ""
-				(path "/61fde5ba-3326-42bd-a4dd-8dab8d594031/a4db3929-a7e6-47d5-836f-632ae16fa9cf"
-					(reference "U16")
-					(unit 1)
-				)
-			)
-		)
