File: src/owr_wifi_router/owr_wifi_router.kicad_sch (KiCad schematic)
At the start: 14 parts

Commit message: finished power board
Parts:
- removed J?: BM08B-PASS, Bluesat:BM08B-PASS, symbol Connector:Conn_01x08_Pin
Connections:
- net VDD-POE renamed +24V
Other:
- added sheet Ethernet PHY (ethernet_phy.kicad_sch)
- added sheet Memory (memory.kicad_sch)
- note added: "-Figure out how to do this split up big IC thing the original does. -Make schematic for new Etherney PHY Chip -Figure out hierarchical pins"
- moved on the sheet: C?

Commit message: progress
Connections:
- net IS_{24V}: no longer names the net of C?.1, C?.2, R?.1, TR?.10 (CT), TR?.4 (CT)
Other:
- moved on the sheet: C?
Changed lines of the file:
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@@
 		(color 0 0 0 0)
 	)
-	(junction
-		(at 92.71 63.5)
-		(diameter 0)
-		(color 0 0 0 0)
-	)
 	(wire
 		(pts
@@
 	(wire
 		(pts
-			(xy 92.71 71.12) (xy 92.71 69.85)
+			(xy 82.55 71.12) (xy 82.55 69.85)
 		)
 		(stroke
@@
 	(wire
 		(pts
-			(xy 74.93 63.5) (xy 92.71 63.5)
+			(xy 74.93 63.5) (xy 82.55 63.5)
 		)
 		(stroke
@@
 	(wire
 		(pts
-			(xy 92.71 64.77) (xy 92.71 63.5)
+			(xy 82.55 64.77) (xy 82.55 63.5)
 		)
 		(stroke
@@
 		(pts
 			(xy 76.2 50.8) (xy 69.85 50.8)
-		)
-		(stroke
-			(width 0)
-			(type default)
-		)
-	)
-	(wire
-		(pts
-			(xy 92.71 63.5) (xy 93.98 63.5)
 		)
 		(stroke
@@
 			)
 			(justify left bottom)
-		)
-	)
-	(hierarchical_label "IS_{24V}"
-		(shape output)
-		(at 93.98 63.5 0)
-		(effects
-			(font
-				(size 1.27 1.27)
-			)
-			(justify left)
 		)
 	)
@@
 	(symbol
 		(lib_id "Bluesat:C_CompactV")
-		(at 92.71 67.31 180)
+		(at 82.55 67.31 180)
 		(unit 1)
 		(exclude_from_sim no)
@@
 		(dnp no)
 		(property "Reference" "C?"
-			(at 93.599 68.072 90)
+			(at 83.439 68.072 90)
 			(do_not_autoplace yes)
 			(effects
@@
 		)
 		(property "Value" "2u2"
-			(at 91.821 68.072 90)
+			(at 81.661 68.072 90)
 			(do_not_autoplace yes)
 			(effects
@@
 		)
 		(property "Footprint" "Capacitor_SMD:C_1206_3216Metric"
-			(at 92.71 67.31 90)
+			(at 82.55 67.31 90)
 			(effects
 				(font
@@
 		)
 		(property "Datasheet" "~"
-			(at 92.71 67.31 90)
+			(at 82.55 67.31 90)
 			(effects
 				(font
@@
 		)
 		(property "Description" "Unpolarized capacitor, compact symbol"
-			(at 92.71 67.31 0)
+			(at 82.55 67.31 0)
 			(effects
 				(font
@@
 	(symbol
 		(lib_id "power:+24V")
-		(at 92.71 71.12 180)
+		(at 82.55 71.12 180)
 		(unit 1)
 		(exclude_from_sim no)
@@
 		(fields_autoplaced yes)
 		(property "Reference" "#PWR02"
-			(at 92.71 67.31 0)
+			(at 82.55 67.31 0)
 			(effects
 				(font
@@
 		)
 		(property "Value" "+24V"
-			(at 92.71 76.2 0)
+			(at 82.55 76.2 0)
 			(effects
 				(font
@@
 		)
 		(property "Footprint" ""
-			(at 92.71 71.12 0)
+			(at 82.55 71.12 0)
 			(effects
 				(font
@@
 		)
 		(property "Datasheet" ""
-			(at 92.71 71.12 0)
+			(at 82.55 71.12 0)
 			(effects
 				(font
@@
 		)
 		(property "Description" "Power symbol creates a global label with name \"+24V\""
-			(at 92.71 71.12 0)
+			(at 82.55 71.12 0)
 			(effects
 				(font
@@
 	)
 	(sheet
-		(at 106.68 24.13)
+		(at 99.06 24.13)
 		(size 25.4 35.56)
 		(exclude_from_sim no)
@@
 		)
 		(property "Sheetname" "Ethernet PHY"
-			(at 106.68 23.4184 0)
+			(at 99.06 23.4184 0)
 			(effects
 				(font
@@
 		)
 		(property "Sheetfile" "ethernet_phy.kicad_sch"
-			(at 106.68 60.2746 0)
-			(effects
-				(font
+			(at 99.06 60.2746 0)
+			(effects
+				(font

Commit message: [progress]
Other:
- removed sheet Ethernet PHY
Changed lines of the file:
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@@
-		)
-	)
-	(sheet
-		(at 99.06 24.13)
-		(size 25.4 35.56)
-		(exclude_from_sim no)
-		(in_bom yes)
-		(on_board yes)
-		(dnp no)
-		(fields_autoplaced yes)
-		(stroke
-			(width 0.1524)
-			(type solid)
-		)
-		(fill
-			(color 0 0 0 0.0000)
-		)
-		(property "Sheetname" "Ethernet PHY"
-			(at 99.06 23.4184 0)
-			(effects
-				(font
-					(size 1.27 1.27)
-				)
-				(justify left bottom)
-			)
-		)
-		(property "Sheetfile" "ethernet_phy.kicad_sch"
-			(at 99.06 60.2746 0)
-			(effects
-				(font
-					(size 1.27 1.27)
-				)
-				(justify left top)
-			)
-		)
-		(instances
-			(project "owr_wifi_router"
-				(path "/61fde5ba-3326-42bd-a4dd-8dab8d594031"
-					(page "4")
-				)
-			)
 		)
 	)

Commit message: Additional Progress on motherboard
Other:
- removed sheet Memory
- added sheet Indicators (indicators.kicad_sch)
- added sheet JTAG (JTAG.kicad_sch)
- added sheet RF_CHIP (RF.kicad_sch)
- added sheet nand_nor (nand_nor.kicad_sch)
- note added: "Look at raspberry pi HIROSE connector setup"
- note added: "RF Chip alone requires 40 pins to be connected to the other board"
- note removed: "-Figure out how to do this split up big IC thing the original does. -Make schematic for new Etherney PHY Chip -Figure out hierarchical pins"
- moved on the sheet: C?, J?, R?, TR?

Commit message: more progress
Parts:
- added Module1: ComputeModule5-CM5, CM5IO:Raspberry-Pi-5-Compute-Module, symbol CM5IO:ComputeModule5-CM5
Connections:
- net GND: now also Module1.1 (GND), Module1.13 (GND), Module1.14 (GND), Module1.2 (GND), Module1.22 (GND), Module1.23 (GND), Module1.32 (GND), Module1.33 (GND), Module1.42 (GND), Module1.43 (GND), Module1.52 (GND), Module1.53 (GND), Module1.59 (GND), Module1.60 (GND), Module1.66 (GND), Module1.7 (GND), Module1.71 (GND), Module1.74 (GND), Module1.8 (GND), Module1.98 (GND)
- net ETH_{OA+} renamed ETHOA+
- net ETHOA+: now also Module1.12 (Ethernet_Pair0_P)
- net ETH_{OA-} renamed ETHOA-
- net ETHOA-: now also Module1.10 (Ethernet_Pair0_N)
- net ETH_{OB+} renamed ETHOB+
- net ETHOB+: now also Module1.4 (Ethernet_Pair1_P)
- net ETH_{OB-} renamed ETHOB-
- net ETHOB-: now also Module1.6 (Ethernet_Pair1_N)
- net ETH_{OC+} renamed ETHOC+
- net ETHOC+: now also Module1.3 (Ethernet_Pair3_P)
- net ETH_{OC-} renamed ETHOC-
- net ETHOC-: now also Module1.5 (Ethernet_Pair3_N)
- net ETH_{OD+} renamed ETHOD+
- net ETHOD+: now also Module1.11 (Ethernet_Pair2_P)
- net ETH_{OD-} renamed ETHOD-
- net ETHOD-: now also Module1.9 (Ethernet_Pair2_N)
Other:
- sheet nand_nor ports: added SPI0_CLK, SPI0_CS, SPI0_HOLD, SPI0_MISO, SPI0_MOSI, SPI0_WP; removed none

Commit message: progress
Other:
- note added: "100 pins for power"
Changed lines of the file:
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@@
 	(generator_version "9.0")
 	(paper "A4")
+	(text "100 pins for power\n"
+		(exclude_from_sim no)
+		(at 142.24 23.114 0)
+		(effects
+			(font
+				(size 1.27 1.27)
+			)
+		)
+	)
 	(text "Look at raspberry pi HIROSE connector setup\n"
 		(exclude_from_sim no)
@@
 	)
 	(sheet
-		(at 184.15 12.7)
+		(at 204.47 15.24)
 		(size 24.13 22.86)
 		(exclude_from_sim no)
@@
 		)
 		(property "Sheetname" "Power"
-			(at 184.15 11.9884 0)
+			(at 204.47 14.5284 0)
 			(effects
 				(font
@@
 		)
 		(property "Sheetfile" "POE_step_down_sch.kicad_sch"
-			(at 184.15 36.1446 0)
+			(at 204.47 38.6846 0)
 			(effects
 				(font
