File: src/vesc_elec/Power.kicad_sch (KiCad schematic)
At the start: 52 parts, among them U2 DRV8301, U4 TP2604-SR

Commit message: Remove unused pins on VESC schematic
Parts:
- removed D210: 30V, Diode_SMD:D_SMF, symbol Device:D_TVS_Small
Changed lines of the file:
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@@
 	)
 	(junction
-		(at 280.67 68.58)
-		(diameter 0)
-		(color 0 0 0 0)
-	)
-	(junction
 		(at 193.04 67.31)
 		(diameter 0)
@@
 	(wire
 		(pts
-			(xy 280.67 68.58) (xy 276.86 68.58)
-		)
-		(stroke
-			(width 0)
-			(type default)
-		)
-	)
-	(wire
-		(pts
 			(xy 128.27 105.41) (xy 130.81 105.41)
 		)
@@
 	(wire
 		(pts
-			(xy 280.67 64.77) (xy 280.67 68.58)
-		)
-		(stroke
-			(width 0)
-			(type default)
-		)
-	)
-	(wire
-		(pts
 			(xy 255.27 104.14) (xy 259.08 104.14)
 		)
@@
 	(wire
 		(pts
-			(xy 280.67 68.58) (xy 280.67 69.85)
-		)
-		(stroke
-			(width 0)
-			(type default)
-		)
-	)
-	(wire
-		(pts
 			(xy 95.25 33.02) (xy 95.25 35.56)
 		)
@@
 		)
 	)
-	(global_label "V_SUPPLY"
-		(shape input)
-		(at 276.86 68.58 180)
-		(effects
-			(font
-				(size 1.524 1.524)
-			)
-			(justify right)
-		)
-		(property "Intersheetrefs" "${INTERSHEET_REFS}"
-			(at 276.86 68.58 0)
-			(effects
-				(font
-					(size 1.27 1.27)
-				)
-				(hide yes)
-			)
-		)
-	)
 	(global_label "SNC"
 		(shape input)
@@
 	)
 	(symbol
-		(lib_id "BLDC_4-rescue:PWR_FLAG")
-		(at 280.67 64.77 0)
-		(unit 1)
-		(exclude_from_sim no)
-		(in_bom yes)
-		(on_board yes)
-		(dnp no)
-		(property "Reference" "#FLG02"
-			(at 280.67 62.357 0)
-			(effects
-				(font
-					(size 0.762 0.762)
-				)
-				(hide yes)
-			)
-		)
-		(property "Value" "PWR_FLAG"
-			(at 280.67 60.198 0)
-			(effects
-				(font
-					(size 0.762 0.762)
-				)
-			)
-		)
-		(property "Footprint" ""
-			(at 280.67 64.77 0)
-			(effects
-				(font
-					(size 1.524 1.524)
-				)
-				(hide yes)
-			)
-		)
-		(property "Datasheet" ""
-			(at 280.67 64.77 0)
-			(effects
-				(font
-					(size 1.524 1.524)
-				)
-				(hide yes)
-			)
-		)
-		(property "Description" ""
-			(at 280.67 64.77 0)
-			(effects
-				(font
-					(size 1.27 1.27)
-				)
-			)
-		)
-		(pin "1"
-		)
-		(instances
-			(project "Cheap FOCer 2 60mm"
-				(path "/8b53313b-c20e-4d2c-aeda-56c30dbca1c0/00000000-0000-0000-0000-0000504f83be"
-					(reference "#FLG02")
-					(unit 1)
-				)
-			)
-		)
-	)
-	(symbol
 		(lib_id "BLDC_4-rescue:GND-RESCUE-BLDC_4")
 		(at 87.63 21.59 0)
@@
 	)
 	(symbol
-		(lib_id "Device:D_TVS_Small")
-		(at 280.67 72.39 270)
+		(lib_id "Device:R")
+		(at 60.96 154.94 90)
 		(unit 1)
 		(exclude_from_sim no)
@@
 		(on_board yes)
 		(dnp no)
-		(property "Reference" "D210"
-			(at 279.4 73.025 90)
+		(property "Reference" "R69"
+			(at 60.96 152.654 90)
 			(effects
 				(font
-					(size 1.016 1.016)
+					(size 1.27 1.27)
 				)
-				(justify right)
 			)
 		)
-		(property "Value" "30V"
-			(at 279.4 71.755 90)
+		(property "Value" "10k"
+			(at 61.214 154.94 90)
 			(effects
 				(font
-					(size 1.016 1.016)
+					(size 1.27 1.27)
 				)
-				(justify right)
 			)
 		)
-		(property "Footprint" "Diode_SMD:D_SMF"
-			(at 280.67 72.39 0)
+		(property "Footprint" "Resistor_SMD:R_0402_1005Metric"
+			(at 60.96 156.718 90)
 			(effects
 				(font
@@
 		)
 		(property "Datasheet" "~"
-			(at 280.67 72.39 0)
+			(at 60.96 154.94 0)
 			(effects
 				(font
@@
 			)
 		)
-		(property "Description" "Bidirectional transient-voltage-suppression diode, small symbol"
-			(at 280.67 72.39 0)
+		(property "Description" "Resistor"
+			(at 60.96 154.94 0)
 			(effects
 				(font
@@
 		)
 		(instances
-			(project "Cheap FOCer 2 60mm"
+			(project ""
 				(path "/8b53313b-c20e-4d2c-aeda-56c30dbca1c0/00000000-0000-0000-0000-0000504f83be"
-					(reference "D210")
+					(reference "R69")
 					(unit 1)
 				)
@@
 	)
 	(symbol
-		(lib_id "Device:R")
-		(at 60.96 154.94 90)
+		(lib_id "power:PWR_FLAG")
+		(at 233.68 57.15 0)
 		(unit 1)
 		(exclude_from_sim no)
@@
 		(on_board yes)
 		(dnp no)
-		(property "Reference" "R69"
-			(at 60.96 152.654 90)
+		(fields_autoplaced yes)
+		(property "Reference" "#FLG01"
+			(at 233.68 55.245 0)
 			(effects
 				(font
 					(size 1.27 1.27)
 				)
+				(hide yes)
 			)
 		)
-		(property "Value" "10k"
-			(at 61.214 154.94 90)
+		(property "Value" "PWR_FLAG"
+			(at 233.68 52.07 0)
 			(effects
 				(font
@@
 			)
 		)
-		(property "Footprint" "Resistor_SMD:R_0402_1005Metric"
-			(at 60.96 156.718 90)
+		(property "Footprint" ""
+			(at 233.68 57.15 0)
 			(effects
 				(font
@@
 		)
 		(property "Datasheet" "~"
-			(at 60.96 154.94 0)
+			(at 233.68 57.15 0)
 			(effects
 				(font
@@
 			)
 		)
-		(property "Description" "Resistor"
-			(at 60.96 154.94 0)
+		(property "Description" "Special symbol for telling ERC where power comes from"
+			(at 233.68 57.15 0)
 			(effects
 				(font
@@
 		(pin "1"
 		)
-		(pin "2"
-		)
 		(instances
 			(project ""
 				(path "/8b53313b-c20e-4d2c-aeda-56c30dbca1c0/00000000-0000-0000-0000-0000504f83be"
-					(reference "R69")
+					(reference "#FLG01")
 					(unit 1)
 				)
@@
 					(unit 1)
 				)
-			)
-		)
-	)
-	(symbol
-		(lib_id "power:GND")
-		(at 280.67 74.93 0)
-		(unit 1)
-		(exclude_from_sim no)
-		(in_bom yes)
-		(on_board yes)
-		(dnp no)
-		(property "Reference" "#PWR0203"
-			(at 280.67 81.28 0)
-			(effects
-				(font
-					(size 1.27 1.27)
-				)
-				(hide yes)
-			)
-		)
-		(property "Value" "GND"
-			(at 280.67 78.105 0)
-			(effects
-				(font
-					(size 0.762 0.762)
-				)
-			)
-		)
-		(property "Footprint" ""
-			(at 280.67 74.93 0)
-			(effects
-				(font
-					(size 1.27 1.27)
-				)
-				(hide yes)
-			)
-		)
-		(property "Datasheet" ""
-			(at 280.67 74.93 0)
-			(effects
-				(font
-					(size 1.27 1.27)
-				)
-				(hide yes)
-			)
-		)
-		(property "Description" "Power symbol creates a global label with name \"GND\" , ground"
-			(at 280.67 74.93 0)
-			(effects
-				(font
-					(size 1.27 1.27)
-				)
-				(hide yes)
-			)
-		)
-		(pin "1"
-		)
-		(instances
-			(project "Cheap FOCer 2 60mm"
-				(path "/8b53313b-c20e-4d2c-aeda-56c30dbca1c0/00000000-0000-0000-0000-0000504f83be"
-					(reference "#PWR0203")
-					(unit 1)
-				)

Commit message: [VESC] Swap phase A and C MOSFET labels (#123)
Connections:
- net GH_A: now also U2.47 (GH_A); no longer U2.37 (GH_C)
- net GH_C: now also U2.37 (GH_C); no longer U2.47 (GH_A)
- net GL_A: now also U2.45 (GL_A); no longer U2.35 (GL_C)
- net GL_C: now also U2.35 (GL_C); no longer U2.45 (GL_A)
- net H1_LOW: now also U2.44 (SL_A); no longer U2.34 (SL_C)
- net H1_VS: now also C27.2, R27.1, U2.46 (SH_A); no longer C18.2, R36.1, U2.36 (SH_C)
- net H3_LOW: now also U2.34 (SL_C); no longer U2.44 (SL_A)
- net H3_VS: now also C18.2, R36.1, U2.36 (SH_C); no longer C27.2, R27.1, U2.46 (SH_A)
- net SNA: now also C29.2, U2.33 (SN2); no longer C34.1, R66.2
- net SNC: now also C34.1, R66.2; no longer C29.2, U2.33 (SN2)
Changed lines of the file:
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@@
 		)
 	)
-	(global_label "SNC"
+	(global_label "SNA"
 		(shape input)
 		(at 194.31 97.79 0)
@@
 		)
 	)
-	(global_label "SNA"
+	(global_label "SNC"
 		(shape input)
 		(at 97.79 156.21 0)
@@
 		)
 	)
-	(hierarchical_label "H3_LOW"
+	(hierarchical_label "H1_LOW"
 		(shape passive)
 		(at 173.99 72.39 0)
@@
 		)
 	)
-	(hierarchical_label "GH_A"
+	(hierarchical_label "GH_C"
 		(shape output)
 		(at 173.99 90.17 0)
@@
 		)
 	)
-	(hierarchical_label "GH_C"
+	(hierarchical_label "GH_A"
 		(shape output)
 		(at 173.99 64.77 0)
@@
 		)
 	)
-	(hierarchical_label "H1_LOW"
+	(hierarchical_label "H3_LOW"
 		(shape passive)
 		(at 173.99 97.79 0)
@@
 		)
 	)
+	(hierarchical_label "H1_VS"
+		(shape input)
+		(at 259.08 91.44 0)
+		(effects
+			(font
+				(size 1.524 1.524)
+			)
+			(justify left)
+		)
+	)
+	(hierarchical_label "H3"
+		(shape input)
+		(at 124.46 92.71 180)
+		(effects
+			(font
+				(size 1.524 1.524)
+			)
+			(justify right)
+		)
+	)
+	(hierarchical_label "L3"
+		(shape input)
+		(at 124.46 95.25 180)
+		(effects
+			(font
+				(size 1.524 1.524)
+			)
+			(justify right)
+		)
+	)
+	(hierarchical_label "EN_GATE"
+		(shape input)
+		(at 124.46 80.01 180)
+		(effects
+			(font
+				(size 1.524 1.524)
+			)
+			(justify right)
+		)
+	)
+	(hierarchical_label "GL_A"
+		(shape output)
+		(at 173.99 69.85 0)
+		(effects
+			(font
+				(size 1.524 1.524)
+			)
+			(justify left)
+		)
+	)
+	(hierarchical_label "SLCK"
+		(shape input)
+		(at 127 67.31 180)
+		(effects
+			(font
+				(size 1.524 1.524)
+			)
+			(justify right)
+		)
+	)
+	(hierarchical_label "SENS1"
+		(shape output)
+		(at 237.49 91.44 180)
+		(effects
+			(font
+				(size 1.524 1.524)
+			)
+			(justify right)
+		)
+	)
 	(hierarchical_label "H3_VS"
 		(shape input)
-		(at 259.08 91.44 0)
-		(effects
-			(font
-				(size 1.524 1.524)
-			)
-			(justify left)
-		)
-	)
-	(hierarchical_label "H3"
-		(shape input)
-		(at 124.46 92.71 180)
-		(effects
-			(font
-				(size 1.524 1.524)
-			)
-			(justify right)
-		)
-	)
-	(hierarchical_label "L3"
-		(shape input)
-		(at 124.46 95.25 180)
-		(effects
-			(font
-				(size 1.524 1.524)
-			)
-			(justify right)
-		)
-	)
-	(hierarchical_label "EN_GATE"
-		(shape input)
-		(at 124.46 80.01 180)
+		(at 259.08 115.57 0)
+		(effects
+			(font
+				(size 1.524 1.524)
+			)
+			(justify left)
+		)
+	)
+	(hierarchical_label "BR_SO3"
+		(shape input)
+		(at 24.13 161.29 90)
+		(effects
+			(font
+				(size 1.524 1.524)
+			)
+			(justify left)
+		)
+	)
+	(hierarchical_label "H1_VS"
+		(shape output)
+		(at 198.12 67.31 0)
+		(effects
+			(font
+				(size 1.524 1.524)
+			)
+			(justify left)
+		)
+	)
+	(hierarchical_label "H3_VS"
+		(shape output)
+		(at 198.12 92.71 0)
+		(effects
+			(font
+				(size 1.524 1.524)
+			)
+			(justify left)
+		)
+	)
+	(hierarchical_label "H1"
+		(shape input)
+		(at 124.46 82.55 180)
+		(effects
+			(font
+				(size 1.524 1.524)
+			)
+			(justify right)
+		)
+	)
+	(hierarchical_label "SDI"
+		(shape input)
+		(at 125.73 62.23 180)
+		(effects
+			(font
+				(size 1.524 1.524)
+			)
+			(justify right)
+		)
+	)
+	(hierarchical_label "BR_SO1"
+		(shape input)
+		(at 104.14 102.87 180)
 		(effects
 			(font
@@
 	(hierarchical_label "GL_C"
 		(shape output)
-		(at 173.99 69.85 0)
-		(effects
-			(font
-				(size 1.524 1.524)
-			)
-			(justify left)
-		)
-	)
-	(hierarchical_label "SLCK"
-		(shape input)
-		(at 127 67.31 180)
-		(effects
-			(font
-				(size 1.524 1.524)
-			)
-			(justify right)
-		)
-	)
-	(hierarchical_label "SENS1"
-		(shape output)
-		(at 237.49 91.44 180)
-		(effects
-			(font
-				(size 1.524 1.524)
-			)
-			(justify right)
-		)
-	)
-	(hierarchical_label "H1_VS"
-		(shape input)
-		(at 259.08 115.57 0)
-		(effects
-			(font
-				(size 1.524 1.524)
-			)
-			(justify left)
-		)
-	)
-	(hierarchical_label "BR_SO3"
-		(shape input)
-		(at 24.13 161.29 90)
-		(effects
-			(font
-				(size 1.524 1.524)
-			)
-			(justify left)
-		)
-	)
-	(hierarchical_label "H3_VS"
-		(shape output)
-		(at 198.12 67.31 0)
-		(effects
-			(font
-				(size 1.524 1.524)
-			)
-			(justify left)
-		)
-	)
-	(hierarchical_label "H1_VS"
-		(shape output)
-		(at 198.12 92.71 0)
-		(effects
-			(font
-				(size 1.524 1.524)
-			)
-			(justify left)
-		)
-	)
-	(hierarchical_label "H1"
-		(shape input)
-		(at 124.46 82.55 180)
-		(effects
-			(font
-				(size 1.524 1.524)
-			)
-			(justify right)
-		)
-	)
-	(hierarchical_label "SDI"
-		(shape input)
-		(at 125.73 62.23 180)
-		(effects
-			(font
-				(size 1.524 1.524)
-			)
-			(justify right)
-		)
-	)
-	(hierarchical_label "BR_SO1"
-		(shape input)
-		(at 104.14 102.87 180)
-		(effects
-			(font
-				(size 1.524 1.524)
-			)
-			(justify right)
-		)
-	)
-	(hierarchical_label "GL_A"
-		(shape output)
 		(at 173.99 95.25 0)
