File: src/vesc2_elec/mosfets.kicad_sch (KiCad schematic)
At the start: 13 parts

Commit message: made evans changes
Parts:
- removed R306: 1m, Resistor_SMD:R_2512_6332Metric, symbol Bluesat:R_CompactV
- renumbered Q to Q?
Changed lines of the file:
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@@
-	)
-	(junction
-		(at 138.43 142.24)
-		(diameter 0)
-		(color 0 0 0 0)
 	)
 	(junction
@@
 	(wire
 		(pts
-			(xy 142.24 142.24) (xy 142.24 139.7)
-		)
-		(stroke
-			(width 0)
-			(type default)
-		)
-	)
-	(wire
-		(pts
 			(xy 134.62 128.27) (xy 138.43 128.27)
 		)
@@
 	(wire
 		(pts
-			(xy 138.43 139.7) (xy 138.43 142.24)
+			(xy 138.43 139.7) (xy 138.43 144.78)
 		)
 		(stroke
@@
 	(wire
 		(pts
-			(xy 138.43 142.24) (xy 138.43 144.78)
-		)
-		(stroke
-			(width 0)
-			(type default)
-		)
-	)
-	(wire
-		(pts
 			(xy 134.62 104.14) (xy 138.43 104.14)
 		)
@@
 	(wire
 		(pts
-			(xy 138.43 142.24) (xy 142.24 142.24)
-		)
-		(stroke
-			(width 0)
-			(type default)
-		)
-	)
-	(wire
-		(pts
 			(xy 154.94 111.76) (xy 154.94 115.57)
 		)
@@
 		(pts
 			(xy 123.19 111.76) (xy 125.73 111.76)
-		)
-		(stroke
-			(width 0)
-			(type default)
-		)
-	)
-	(wire
-		(pts
-			(xy 142.24 132.08) (xy 142.24 134.62)
-		)
-		(stroke
-			(width 0)
-			(type default)
-		)
-	)
-	(wire
-		(pts
-			(xy 138.43 132.08) (xy 142.24 132.08)
 		)
 		(stroke
@@
 		(dnp no)
 		(fields_autoplaced yes)
-		(property "Reference" "Q"
+		(property "Reference" "Q?"
 			(at 142.24 86.3599 0)
 			(effects
@@
 		(instances
 			(project "vesc2"
+				(path "/2059a583-03d9-42e7-b042-844898d8f177/1b823304-293f-4595-a426-e06902eaf0d9"
+					(reference "Q?")
+					(unit 1)
+				)
 				(path "/2059a583-03d9-42e7-b042-844898d8f177/395e1093-67ec-4614-b25c-b37e14ae8318"
 					(reference "Q401")
@@
 					(unit 1)
 				)
-			)
-		)
-	)
-	(symbol
-		(lib_id "Bluesat:R_CompactV")
-		(at 142.24 137.16 0)
-		(unit 1)
-		(exclude_from_sim no)
-		(in_bom yes)
-		(on_board yes)
-		(dnp no)
-		(fields_autoplaced yes)
-		(property "Reference" "R306"
-			(at 141.351 137.16 90)
-			(do_not_autoplace yes)
-			(effects
-				(font
-					(size 1.016 1.016)
-				)
-				(justify bottom)
-			)
-		)
-		(property "Value" "1m"
-			(at 142.24 137.16 90)
-			(do_not_autoplace yes)
-			(effects
-				(font
-					(size 0.762 0.762)
-				)
-			)
-		)
-		(property "Footprint" "Resistor_SMD:R_2512_6332Metric"
-			(at 142.24 137.16 0)
-			(effects
-				(font
-					(size 1.27 1.27)
-				)
-				(hide yes)
-			)
-		)
-		(property "Datasheet" "~"
-			(at 142.24 137.16 0)
-			(effects
-				(font
-					(size 1.27 1.27)
-				)
-				(hide yes)
-			)
-		)
-		(property "Description" "Resistor, compact symbol"
-			(at 142.24 137.16 0)
-			(effects
-				(font
-					(size 1.27 1.27)
-				)
-				(hide yes)
-			)
-		)
-		(pin "2"
-		)
-		(pin "1"
-		)
-		(instances
-			(project "vesc2"
-				(path "/2059a583-03d9-42e7-b042-844898d8f177/1b823304-293f-4595-a426-e06902eaf0d9"
-					(reference "R306")
-					(unit 1)
-				)
-				(path "/2059a583-03d9-42e7-b042-844898d8f177/395e1093-67ec-4614-b25c-b37e14ae8318"
-					(reference "R406")
-					(unit 1)
-				)
-				(path "/2059a583-03d9-42e7-b042-844898d8f177/43e157cb-6b50-47c8-9e44-0b1971389d5f"
-					(reference "R506")
-					(unit 1)
-				)

Commit message: Final commit before routing just incase
Parts:
- removed Q302, Q?: ~, symbol Bluesat:NMOS_Heatsink
- added Q301, Q302: IRFH7440TRPBF, Bluesat:PQFN_5x6mm_E_DGS, symbol Transistor_FET:Q_NMOS_DGS
- renumbered R302 to R301, R304 to R302, R301 to R303, R303 to R304, R307 to R306, R308 to R307
Connections:
- net LOW: now also Q302.3 (S)
- net PHASE: now also Q301.3 (S), Q302.1 (D)
- net V_SUPPLY: now also Q301.1 (D)
- net at C301.2, R301.2, R303.1: now also Q301.2 (G)
- net at C302.2, R302.2, R304.1: now also Q302.2 (G)
Other:
- moved on the sheet: C303, R306, R307

Commit message: finished routing :)
Connections:
- net V_SUPPLY renamed VBUS
Changed lines of the file:
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@@
-		)
-	)
-	(global_label "V_SUPPLY"
-		(shape input)
-		(at 138.43 78.74 90)
-		(fields_autoplaced yes)
-		(effects
-			(font
-				(size 1.27 1.27)
-			)
-			(justify left)
-		)
-		(property "Intersheetrefs" "${INTERSHEET_REFS}"
-			(at 138.43 66.5019 90)
-			(effects
-				(font
-					(size 1.27 1.27)
-				)
-				(justify left)
-				(hide yes)
-			)
 		)
 	)
@@
 					(unit 1)
 				)
+			)
+		)
+	)
+	(symbol
+		(lib_id "power:VBUS")
+		(at 138.43 78.74 0)
+		(unit 1)
+		(exclude_from_sim no)
+		(in_bom yes)
+		(on_board yes)
+		(dnp no)
+		(property "Reference" "#PWR0303"
+			(at 138.43 82.55 0)
+			(effects
+				(font
+					(size 1.27 1.27)
+				)
+				(hide yes)
+			)
+		)
+		(property "Value" "VBUS"
+			(at 138.43 74.93 0)
+			(effects
+				(font
+					(size 1.27 1.27)
+				)
+			)
+		)
+		(property "Footprint" ""
+			(at 138.43 78.74 0)
+			(effects
+				(font
+					(size 1.27 1.27)
+				)
+				(hide yes)
+			)
+		)
+		(property "Datasheet" ""
+			(at 138.43 78.74 0)
+			(effects
+				(font
+					(size 1.27 1.27)
+				)
+				(hide yes)
+			)
+		)
+		(property "Description" "Power symbol creates a global label with name \"VBUS\""
+			(at 138.43 78.74 0)
+			(effects
+				(font
+					(size 1.27 1.27)
+				)
+				(hide yes)
+			)
+		)
+		(pin "1"
+		)
+		(instances
+			(project "vesc2"
+				(path "/2059a583-03d9-42e7-b042-844898d8f177/1b823304-293f-4595-a426-e06902eaf0d9"
+					(reference "#PWR0303")
+					(unit 1)
+				)
+				(path "/2059a583-03d9-42e7-b042-844898d8f177/395e1093-67ec-4614-b25c-b37e14ae8318"
+					(reference "#PWR0403")
+					(unit 1)
+				)
+				(path "/2059a583-03d9-42e7-b042-844898d8f177/43e157cb-6b50-47c8-9e44-0b1971389d5f"
+					(reference "#PWR0503")
+					(unit 1)
+				)
