File: src/wark_min/power.kicad_sch (KiCad schematic)
At the start: 44 parts, among them J201 XT30M, Q201 SSM3K333R, U201 MP2459GJ-Z-MS, U202 AP62200TWU, U203 HX4002

Commit message: Small pile becomes big pile
Parts:
- added C360, C361: 270u, Capacitor_SMD:CP_Elec_10x10, symbol Device:C_Polarized_Small_US
- J201: footprint Connector_AMASS:AMASS_XT30PW-M_1x02_P2.50mm_Horizontal -> Connector_AMASS:AMASS_XT30U-M_1x02_P5.0mm_Vertical
Connections:
- net GND: now also C360.2, C361.2
- net VBUS: now also C360.1, C361.1

Commit message: Pre-stupid
Parts:
- removed C208: 10n, Capacitor_SMD:C_0402_1005Metric, symbol Bluesat:C_CompactV
- removed C211, C212: 10u, Capacitor_SMD:C_1206_3216Metric, symbol Bluesat:C_CompactV
- removed C218: 2u2, Capacitor_SMD:C_0603_1608Metric, symbol Bluesat:C_CompactH
- removed C219, C220: 2u2, Capacitor_SMD:C_0603_1608Metric, symbol Bluesat:C_CompactV
- removed C360, C361: 270u, Capacitor_SMD:CP_Elec_10x10, symbol Device:C_Polarized_Small_US
- removed D201: 30V, Diode_SMD:D_SOD-123F, symbol Device:D_Zener_Small
- removed J201: XT30M, Connector_AMASS:AMASS_XT30U-M_1x02_P5.0mm_Vertical, symbol Connector:Conn_01x02_Pin
- removed L205: 600R, Resistor_SMD:R_0402_1005Metric, symbol Device:L_Ferrite_Small
- removed R202: 220k, Resistor_SMD:R_0402_1005Metric, symbol Bluesat:R_CompactV
- removed R204: 10k, Resistor_SMD:R_0402_1005Metric, symbol Bluesat:R_CompactV
- removed U203: HX4002, Package_TO_SOT_SMD:SOT-23-6, symbol Regulator_SwitchedCapacitor:LTC1754
Other:
- note removed: "1. VBUS Input"
- note removed: "4. 3V3 (VDD) -> 5V Charge Pump (250mA)"
- note removed: "5. VDD -> VDDA Filter"
- note removed: "BW=1/(2π*10k*10n)=1.6kHz"
