File: src/wark_min/wark_min.kicad_pcb (KiCad board)
At the start: 2 copper layers, 180 parts, among them J101 SM02B-PASS, J102 MR60, J103 BM12B-ZPDSS, J104 IDC6, J105 SM06B-PASS, J201 XT30M, Q201 SSM3K333R, Q301 CJ3439KDW, Q302 IRFH7440TRPBF, Q303 BC846S, Q304 CJ3439KDW, Q305 IRFH7440TRPBF, Q401 CJ3439KDW, Q403 BC846S, Q404 CJ3439KDW, Q406 IRFH7440TRPBF, Q407 IRFH7440TRPBF, Q501 CJ3439KDW, Q503 BC846S, Q504 CJ3439KDW, Q506 IRFH7440TRPBF, Q507 IRFH7440TRPBF, U101 STM32G474_WarkMin, U102 TCAN1462V, U103 ZD24C128A, U104 ZD25WQ16C, U201 MP2459GJ-Z-MS, U202 AP62200TWU, U203 HX4002, Y101 24Mhz

Commit message: Small pile becomes big pile
Parts:
- removed C304, C404, C504: 270u, Capacitor_SMD:CP_Elec_10x10
- added C360: 270u, Capacitor_SMD:CP_Elec_10x10, F.Cu at (8.00, -6.00)
- added C361: 270u, Capacitor_SMD:CP_Elec_10x10, F.Cu at (8.00, 6.00)
- added H101: M2.5, Bluesat:M2.5, F.Cu at (22.5, -13.5)
- added H102: M2.5, Bluesat:M2.5, F.Cu at (22.5, 13.5)
- added R313: 1k, Resistor_SMD:R_0402_1005Metric, B.Cu at (3.00, -12.2)
- added R318: 1k, Resistor_SMD:R_0402_1005Metric, B.Cu at (7.50, -12.2)
- added R413: 1k, Resistor_SMD:R_0402_1005Metric, B.Cu at (3.00, -3.75)
- added R418: 1k, Resistor_SMD:R_0402_1005Metric, B.Cu at (7.50, -3.75)
- added R513: 1k, Resistor_SMD:R_0402_1005Metric, B.Cu at (3.00, 4.75)
- added R518: 1k, Resistor_SMD:R_0402_1005Metric, B.Cu at (7.50, 4.75)
- C106, C107, C216, D101, D102, D201, D203, L202, L203: moved to F.Cu
- J101: footprint Bluesat:SM02B-PASS -> Bluesat:BM02B-PASS
- J105: footprint Bluesat:SM06B-PASS -> Bluesat:BM06B-PASS
- J201: footprint Connector_AMASS:AMASS_XT30PW-M_1x02_P2.50mm_Horizontal -> Connector_AMASS:AMASS_XT30U-M_1x02_P5.0mm_Vertical
- moved R511 192.8 mm to (-67.1, -6.25), turned to -90 degrees
- moved R411 182.9 mm to (-67.1, -14.8), turned to -90 degrees
- moved C508 181.3 mm to (-75.3, 6.12)
- moved R516 176.8 mm to (-60.1, 4.38), turned to 90 degrees
- moved R504 175.8 mm to (-53.5, 5.00), turned to 0 degrees
- moved C503 174.0 mm to (-66.4, 5.34)
- moved R507 173.2 mm to (-58.4, 4.62), turned to 0 degrees
- moved C509 172.9 mm to (-58.4, 3.38)
- moved R508 172.7 mm to (-65.6, 15.2), turned to 90 degrees
- moved C502 171.7 mm to (-66.3, 6.62)
- moved R514 170.5 mm to (-55.2, 4.50), turned to 90 degrees
- moved C408 170.2 mm to (-75.3, -2.38)
- moved R416 166.9 mm to (-60.1, -4.12), turned to 90 degrees
- moved R404 165.9 mm to (-53.5, -3.50), turned to 0 degrees
- moved C409 164.3 mm to (-58.4, -5.12)
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Connections:
- C305 pad 1: /Phase A/LOW -> GND
- C309 pad 2: /Phase A/LOW -> /Phase A/LOWSH
- C405 pad 1: /Phase B/LOW -> GND
- C409 pad 2: /Phase B/LOW -> /Phase B/LOWSH
- C505 pad 1: /Phase C/LOW -> GND
- C509 pad 2: /Phase C/LOW -> /Phase C/LOWSH
- Q304 pad 1: /Phase A/LOW -> /Phase A/LOWSH
- Q305 pad 3: /Phase A/LOW -> /Phase A/LOWSH
- Q404 pad 1: /Phase B/LOW -> /Phase B/LOWSH
- Q407 pad 3: /Phase B/LOW -> /Phase B/LOWSH
- Q504 pad 1: /Phase C/LOW -> /Phase C/LOWSH
- Q507 pad 3: /Phase C/LOW -> /Phase C/LOWSH
- R311 pad 1: /Phase A/TEMP -> VDD
- R311 pad 2: GND -> /Phase A/TEMP
- R316 pad 1: /Phase A/LOW -> /Phase A/LOWSH
- R317 pad 1: /Phase A/LOW -> /Phase A/LOWSH
- R411 pad 1: /Phase B/TEMP -> VDD
- R411 pad 2: GND -> /Phase B/TEMP
- R416 pad 1: /Phase B/LOW -> /Phase B/LOWSH
- R417 pad 1: /Phase B/LOW -> /Phase B/LOWSH
- R511 pad 1: /Phase C/TEMP -> VDD
- R511 pad 2: GND -> /Phase C/TEMP
- R516 pad 1: /Phase C/LOW -> /Phase C/LOWSH
- R517 pad 1: /Phase C/LOW -> /Phase C/LOWSH
- TH301 pad 1: VDD -> /Phase A/TEMP
- TH301 pad 2: /Phase A/TEMP -> GND
- TH401 pad 1: VDD -> /Phase B/TEMP
- TH401 pad 2: /Phase B/TEMP -> GND
- TH501 pad 1: VDD -> /Phase C/TEMP
- TH501 pad 2: /Phase C/TEMP -> GND
Routing:
- net VBST: track 0.00 -> 33.3 mm, vias 0 -> 5
- net +12V: track 0.00 -> 27.4 mm, vias 0 -> 5
- net /Phase B/LOWSH: track 0.00 -> 25.2 mm, vias 0 -> 4
- net /Phase A/GH: track 0.00 -> 21.0 mm, vias 0 -> 2
- net /Phase A/LOWSH: track 0.00 -> 18.3 mm, vias 0 -> 4
- net /Phase C/LOWSH: track 0.00 -> 17.7 mm, vias 0 -> 3
- net /Phase C/GL: track 0.00 -> 15.7 mm, vias 0 -> 3
- net /Phase B/GL: track 0.00 -> 15.4 mm, vias 0 -> 3
- net /Phase A/GL: track 0.00 -> 15.4 mm, vias 0 -> 3
- net /Phase B/PHASE: track 0.00 -> 14.5 mm, vias 0 -> 2
- net /Phase A/DL: track 0.00 -> 13.6 mm, vias 0 -> 2
- net Net-(Q401A-D1): track 0.00 -> 12.9 mm, vias 0 -> 3
- net /Phase B/GH: track 0.00 -> 11.8 mm
- net /Phase C/DL: track 0.00 -> 11.7 mm
- net /Phase C/PHASE: track 0.00 -> 11.5 mm, vias 0 -> 3
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- added copper zone on B.Cu, net /Phase A/LOWSH
- added copper zone on B.Cu, net /Phase B/LOWSH
- added copper zone on B.Cu, net /Phase B/PHASE
- added copper zone on B.Cu, net /Phase C/LOWSH
- added copper zone on B.Cu, net /Phase C/PHASE
- added copper zone on B.Cu, net GND
- added copper zone on F.Cu, net GND
- added copper zone on In1.Cu, net GND
- added copper zone on In4.Cu, net GND
- added copper zone on F.Cu, net VBUS
- removed copper zone on B.Cu, net /Phase A/LOW
Other:
- board outline added: 65 x 27 mm
- copper layers 2 -> 6

Commit message: Hiiiiiiiiiiiiiiiii
Parts:
- C106, C107, C216, D101, D102, D201, D203, H101, H102, L202, L203: moved to B.Cu
- moved C301 205.9 mm to (-67.7, 177.6)
- moved C307 199.9 mm to (-59.6, 181.1), turned to 180 degrees
- moved C309 199.4 mm to (-67.7, 185.5)
- moved R306 198.9 mm to (-59.0, 174.4), turned to 180 degrees
- moved Q304 198.2 mm to (-76.2, 173.3)
- moved R313 197.6 mm to (-61.9, 174.4)
- moved TH301 195.6 mm to (-64.8, 170.4), turned to 180 degrees
- moved R318 194.6 mm to (-64.8, 168.4), turned to 180 degrees
- moved C308 194.6 mm to (-67.7, 183.5)
- moved C306 194.4 mm to (-59.6, 178.6), turned to 180 degrees
- moved R311 193.7 mm to (-61.9, 170.4), turned to 180 degrees
- moved C303 193.2 mm to (-67.7, 181.6)
- moved R312 193.2 mm to (-61.9, 172.4), turned to 180 degrees
- moved C409 191.1 mm to (-44.9, 185.5)
- moved R303 190.3 mm to (-59.0, 168.4)
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Routing:
- net VBST: track 33.3 -> 0.00 mm, vias 5 -> 0
- net +12V: track 27.4 -> 0.00 mm, vias 5 -> 0
- net /Phase B/LOWSH: track 25.2 -> 0.00 mm, vias 4 -> 0
- net /Phase A/GH: track 21.0 -> 0.00 mm, vias 2 -> 0
- net /Phase A/LOWSH: track 18.3 -> 0.00 mm, vias 4 -> 0
- net /Phase C/LOWSH: track 17.7 -> 0.00 mm, vias 3 -> 0
- net /Phase C/GL: track 15.7 -> 0.00 mm, vias 3 -> 0
- net /Phase B/GL: track 15.4 -> 0.00 mm, vias 3 -> 0
- net /Phase A/GL: track 15.4 -> 0.00 mm, vias 3 -> 0
- net /Phase B/PHASE: track 14.5 -> 0.00 mm, vias 2 -> 0
- net /Phase A/DL: track 13.6 -> 0.00 mm, vias 2 -> 0
- net Net-(Q401A-D1): track 12.9 -> 0.00 mm, vias 3 -> 0
- net /Phase B/GH: track 11.8 -> 0.00 mm
- net /Phase C/DL: track 11.7 -> 0.00 mm
- net /Phase C/PHASE: track 11.5 -> 0.00 mm, vias 3 -> 0
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- removed copper zone on B.Cu, net /Phase A/LOWSH
- removed copper zone on B.Cu, net /Phase A/PHASE
- removed copper zone on B.Cu, net /Phase B/LOWSH
- removed copper zone on B.Cu, net /Phase B/PHASE
- removed copper zone on B.Cu, net /Phase C/LOWSH
- removed copper zone on B.Cu, net /Phase C/PHASE
- removed copper zone on B.Cu, net GND
- removed copper zone on F.Cu, net GND
- removed copper zone on In1.Cu, net GND
- removed copper zone on In4.Cu, net GND
- removed copper zone on B.Cu, net VBUS
- removed copper zone on F.Cu, net VBUS
Other:
- board size 65 x 27 mm -> 52 x 26 mm

Commit message: Pre-stupid
Parts:
- removed C204, C207: 68u, Capacitor_SMD:CP_Elec_6.3x7.7
- removed C205, C214, C215: 33p, Capacitor_SMD:C_0402_1005Metric
- removed C206: 1u-M, Capacitor_SMD:C_0805_2012Metric
- removed C208, C501: 10n, Capacitor_SMD:C_0402_1005Metric
- removed C209, C503: 220n, Capacitor_SMD:C_0402_1005Metric
- removed C210: 4u7-M, Capacitor_SMD:C_1206_3216Metric
- removed C211, C212: 10u, Capacitor_SMD:C_1206_3216Metric
- removed C213: 1u-H, Capacitor_SMD:C_1206_3216Metric
- removed C216: 22u, Capacitor_SMD:C_1210_3225Metric
- removed C217: 2u2-H, Capacitor_SMD:C_1206_3216Metric
- removed C218, C219, C220: 2u2, Capacitor_SMD:C_0603_1608Metric
- removed C305, C405, C505: 4u7-H, Capacitor_SMD:C_1210_3225Metric
- removed C306, C307, C406, C407, C506, C507: 100n-H, Capacitor_SMD:C_0603_1608Metric
- removed C308, C408, C502, C508: 1n, Capacitor_SMD:C_0402_1005Metric
- removed C309, C409, C509: 100n, Capacitor_SMD:C_0402_1005Metric
- removed C360, C361: 270u, Capacitor_SMD:CP_Elec_10x10
- removed D201: 30V, Diode_SMD:D_SOD-123F
- removed D202, D203: 500mA, Diode_SMD:D_SOD-123
- removed J201: XT30M, Connector_AMASS:AMASS_XT30U-M_1x02_P5.0mm_Vertical
- removed L201: 120R, Resistor_SMD:R_0603_1608Metric
- removed L202: 15u-2A, Inductor_SMD:L_Changjiang_FNR5040S
- removed L203: 4u7-2A, Inductor_SMD:L_Changjiang_FNR4020S
- removed L204: 100u-100mA, Inductor_SMD:L_0805_2012Metric
- removed L205: 600R, Resistor_SMD:R_0402_1005Metric
- removed Q303, Q403, Q503: BC846S, Bluesat:SOT-363
- removed Q304, Q404, Q501, Q504: CJ3439KDW, Bluesat:SOT-363
- removed Q305, Q406, Q407, Q506, Q507: IRFH7440TRPBF, Bluesat:PQFN_5x6mm_E_DGS
- removed R205, R208, R210, R211, R309, R314, R409, R414, R501, R504, R509, R514, TH301, TH401, TH501: 10k, Resistor_SMD:R_0402_1005Metric
- removed R206: 22k, Resistor_SMD:R_0402_1005Metric
- removed R207: 220k, Resistor_SMD:R_0402_1005Metric
- removed R209: 100K, Resistor_SMD:R_0402_1005Metric
- removed R305, R313, R315, R318, R405, R413, R415, R418, R505, R513, R515, R518: 1k, Resistor_SMD:R_0402_1005Metric
- removed R306, R310, R312, R316, R406, R410, R412, R416, R502, R503, R506, R510, R512, R516: 10R, Resistor_SMD:R_0402_1005Metric
- removed R307, R407, R507: 220K, Resistor_SMD:R_0402_1005Metric
- removed R308, R408, R508: 10K, Resistor_SMD:R_0402_1005Metric
- removed R311, R411, R511: 2k2, Resistor_SMD:R_0402_1005Metric
- removed R317, R417, R517: 1m, Resistor_SMD:R_2512_6332Metric
- removed U201: MP2459GJ-Z-MS, Package_TO_SOT_SMD:TSOT-23-6
- removed U202: AP62200TWU, Package_TO_SOT_SMD:TSOT-23-6
- removed U203: HX4002, Package_TO_SOT_SMD:SOT-23-6
- added C121: 220n, Capacitor_SMD:C_0402_1005Metric, B.Cu at (0.49, 78.5)
- added C122: 220n, Capacitor_SMD:C_0402_1005Metric, B.Cu at (0.49, 80.5)
- added C123: 220n, Capacitor_SMD:C_0402_1005Metric, B.Cu at (-2.38, 68.6)
- added C124: 220n, Capacitor_SMD:C_0402_1005Metric, B.Cu at (42.8, -7.25)
- added C125: 220n, Capacitor_SMD:C_0402_1005Metric, B.Cu at (32.0, -3.50)
- added C126: 220n, Capacitor_SMD:C_0402_1005Metric, B.Cu at (35.8, 7.25)
- added C127: 220n, Capacitor_SMD:C_0402_1005Metric, B.Cu at (46.5, 3.50)
- added C128: 2u2, Capacitor_SMD:C_0603_1608Metric, B.Cu at (31.3, 96.2)
- added C129: 2u2, Capacitor_SMD:C_0603_1608Metric, B.Cu at (31.3, 98.7)
- added C130: 220n, Capacitor_SMD:C_0402_1005Metric, B.Cu at (-2.38, 78.5)
- added C131: 100n, Capacitor_SMD:C_0402_1005Metric, B.Cu at (31.8, 3.50)
- added C132: 1u-M, Capacitor_SMD:C_0805_2012Metric, B.Cu at (32.2, 6.25)
- added C133: 22u, Capacitor_SMD:C_1210_3225Metric, B.Cu at (30.2, 9.75)
- added C134: 10n, Capacitor_SMD:C_0402_1005Metric, B.Cu at (-5.25, 68.6)
- added C135: 33n, Capacitor_SMD:C_0402_1005Metric, B.Cu at (29.0, 7.25)
- added C136: 10u, Capacitor_SMD:C_1206_3216Metric, B.Cu at (46.2, -6.50)
- added C137: 10u, Capacitor_SMD:C_1206_3216Metric, B.Cu at (50.0, -8.75)
- added C138: 2u2, Capacitor_SMD:C_0603_1608Metric, B.Cu at (43.5, -9.50)
- added C139: 1u, Capacitor_SMD:C_0603_1608Metric, B.Cu at (29.8, -2.50)
- added C140: 220n, Capacitor_SMD:C_0402_1005Metric, B.Cu at (25.0, -2.25)
- added C141: 100n-H, Capacitor_SMD:C_0603_1608Metric, B.Cu at (31.3, 106.2)
- added C142: 4u7-H, Capacitor_SMD:C_1210_3225Metric, B.Cu at (-6.01, 105.9)
- added C143: 220n, Capacitor_SMD:C_0402_1005Metric, B.Cu at (-5.25, 74.5)
- added D108: 30V, Diode_SMD:D_SOD-123F, F.Cu at (29.3, -4.50)
- added D109: 500mA, Diode_SMD:D_SOD-123, F.Cu at (27.5, 2.00)
- added J106: XT30M, Connector_AMASS:AMASS_XT30U-M_1x02_P5.0mm_Vertical, F.Cu at (32.0, -9.00)
- added L101: 600R, Resistor_SMD:R_0402_1005Metric, B.Cu at (4.09, 92.0)
- added L102: 47u-1A, Inductor_SMD:L_Changjiang_FXL0630, F.Cu at (28.0, 7.75)
- added Q202: IRFH7440TRPBF, Bluesat:PQFN_5x6mm_E_DGS, B.Cu at (14.8, 8.25)
- added Q402: IRFH7440TRPBF, Bluesat:PQFN_5x6mm_E_DGS, B.Cu at (14.8, -8.50)
- added R107: 100k, Resistor_SMD:R_0402_1005Metric, B.Cu at (1.18, 94.0)
- added R108: 10k, Resistor_SMD:R_0402_1005Metric, B.Cu at (1.18, 96.0)
- added R109: 220k, Resistor_SMD:R_0402_1005Metric, B.Cu at (28.5, -15.2)
- added R110: 33k, Resistor_SMD:R_0402_1005Metric, B.Cu at (26.8, 10.8)
- added R111: 10k, Resistor_SMD:R_0402_1005Metric, B.Cu at (28.5, -14.0)
- added R112: 10k, Resistor_SMD:R_0402_1005Metric, B.Cu at (24.5, 10.8)
- added TH101: 10k, Resistor_SMD:R_0402_1005Metric, B.Cu at (17.2, -4.00)
- added TH102: 10k, Resistor_SMD:R_0402_1005Metric, B.Cu at (17.2, 4.25)
- added U105: ZD25WQ16C, Package_SON:Winbond_USON-8-1EP_3x2mm_P0.5mm_EP0.2x1.6mm, B.Cu at (49.2, -3.25)
- added U106: ZD25WQ16C, Package_SON:Winbond_USON-8-1EP_3x2mm_P0.5mm_EP0.2x1.6mm, B.Cu at (49.2, 0.41)
- added U107: HX4002, Package_TO_SOT_SMD:SOT-23-6, B.Cu at (46.5, -9.50)
- C102: value 10p -> 220n
- C103: value 10n -> 10p
- C104: value 1u-M -> 100n; footprint Capacitor_SMD:C_0805_2012Metric -> Capacitor_SMD:C_0402_1005Metric
- C105: value 2u2 -> 100n; footprint Capacitor_SMD:C_0603_1608Metric -> Capacitor_SMD:C_0402_1005Metric
- C106, C303, C403: value 220n -> 100n
- C108: value 220n -> 270u; footprint Capacitor_SMD:C_0402_1005Metric -> Capacitor_SMD:CP_Elec_10x10; moved to F.Cu
- C109: value 10u -> 270u; footprint Capacitor_SMD:C_1206_3216Metric -> Capacitor_SMD:CP_Elec_10x10; moved to F.Cu
- C110, C111: value 2u2 -> 4u7-H; footprint Capacitor_SMD:C_0603_1608Metric -> Capacitor_SMD:C_1210_3225Metric
- C112: value 2u2 -> 330n-H; footprint Capacitor_SMD:C_0603_1608Metric -> Capacitor_SMD:C_0805_2012Metric
- C116: value 220n -> 10n
- C117, C118, C119: value 220n -> 2u2; footprint Capacitor_SMD:C_0402_1005Metric -> Capacitor_SMD:C_0603_1608Metric
- C201: value 100n-M -> 10n
- C202: value 1u-H -> 1n; footprint Capacitor_SMD:C_1206_3216Metric -> Capacitor_SMD:C_0402_1005Metric
- C203: value 1u-H -> 100n; footprint Capacitor_SMD:C_1206_3216Metric -> Capacitor_SMD:C_0402_1005Metric
- D101, D102: moved to F.Cu
- D104, D105, D106, D107: footprint Package_DFN_QFN:Diodes_UDFN-10_1x2.5mm_P0.5mm -> Package_DFN_QFN:UDFN-10_1.35x2.6mm_P0.5mm
- Q201: value SSM3K333R -> IRFH7440TRPBF; footprint Package_TO_SOT_SMD:TSOT-23 -> Bluesat:PQFN_5x6mm_E_DGS
- Q301, Q401: value CJ3439KDW -> IRFH7440TRPBF; footprint Bluesat:SOT-363 -> Bluesat:PQFN_5x6mm_E_DGS
- R102: value 470R -> 2k2
- R103: value 10k -> 470R
- R104: value 100k -> 2k2
- R105: value 100k -> 10k
- R106: value 10k -> 100k
- R201: value 100k -> 10R
- R202: value 220k -> 220K
- R203: value 47k -> 10K
- R204, R304, R404: value 10k -> 1m; footprint Resistor_SMD:R_0402_1005Metric -> Resistor_SMD:R_2512_6332Metric
- R301, R401: value 10k -> 10R
- R302, R402: value 10R -> 220K
- R303, R403: value 10R -> 10K
- U101: value STM32G474_WarkMin -> STM32G474
- U102: value TCAN1462V -> DRV8323RH; footprint Package_SO:JEITA_SOIC-8_3.9x4.9mm_P1.27mm -> Package_DFN_QFN:Texas_RGZ0048A_VQFN-48-1EP_7x7mm_P0.5mm_EP5.15x5.15mm
- U103: value ZD24C128A -> TCAN1462V; footprint Bluesat:TSSOP-8_4.4x3.0-0.65 -> Package_SO:SOIC-8_3.9x4.9mm_P1.27mm
- U104: value ZD25WQ16C -> ZD24C128A; footprint Package_SON:Winbond_USON-8-1EP_3x2mm_P0.5mm_EP0.2x1.6mm -> Bluesat:TSSOP-8_4.4x3.0-0.65
- moved Q301 191.4 mm to (20.0, 0.00), turned to 90 degrees
- moved Q401 188.8 mm to (20.0, -8.50), turned to 90 degrees
- moved R102 188.1 mm to (110.3, 5.00)
- moved R104 188.1 mm to (110.3, 8.98)
- moved C301 186.7 mm to (1.50, 4.25), turned to -90 degrees
- moved C401 184.8 mm to (1.50, -1.25), turned to -90 degrees
- moved R404 184.3 mm to (10.0, -8.00), turned to -90 degrees
- moved R304 183.9 mm to (10.0, 0.00), turned to -90 degrees
- moved U104 178.2 mm to (38.8, -9.50)
- moved D106 175.9 mm to (36.2, -16.5), turned to 90 degrees
- moved R201 175.8 mm to (1.50, -6.75), turned to -90 degrees
- moved R403 175.6 mm to (-18.0, -6.25), turned to 0 degrees
- moved R402 173.4 mm to (-20.2, -6.25), turned to 0 degrees
- moved R301 168.9 mm to (1.50, 6.75), turned to 90 degrees
- moved C201 168.6 mm to (1.50, -4.25), turned to 90 degrees
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Connections:
- net Net-(D101-DIN) renamed /ARGB_{1}
- net Net-(D102-DIN) renamed /ARGB_{0}
- C102 pad 2: /OSC_OUT_L -> /TMPA
- C103 pad 2: /DBG.NRST -> /OSC_OUT_L
- C104 pad 2: +12V -> /ISA
- C105 pad 2: +5V -> /ISB
- C106 pad 2: +5V -> /ISC
- C107 pad 2: +5V -> /TMPB
- C108 pad 1: GND -> VBUS
- C108 pad 2: +5V -> GND
- C109 pad 1: GND -> VBUS
- C109 pad 2: VDD -> GND
- C110 pad 2: VDD -> VBUS
- C111 pad 2: VDD -> VBUS
- C112 pad 2: VDD -> VBUS
- C113 pad 2: VDD -> +5V
- C114 pad 2: VDD -> +5V
- C115 pad 2: VDD -> +5V
- C116 pad 2: VDD -> /DBG.NRST
- C120 pad 2: VDDA -> VDD
- C201 pad 1: /Power/12V_{BST} -> GND
- C201 pad 2: /Power/12V_{SW} -> /Phase A/FLT_{M}
- C202 pad 2: VBUS -> /VSA
- C203 pad 2: /Power/VBUS_{FLT} -> /Phase A/SP
- C301 pad 2: /Phase A/FLT_{M} -> /Phase B/FLT_{M}
- C302 pad 2: /Phase A/V_{SENSE} -> /VSB
- C303 pad 2: /Phase A/TEMP -> /Phase B/SP
- C401 pad 2: /Phase B/FLT_{M} -> /Phase C/FLT_{M}
- C402 pad 2: /Phase B/V_{SENSE} -> /VSC
- C403 pad 2: /Phase B/TEMP -> /Phase C/SP
- D104 pad 1: /DBG.SWDIO -> /XIO0
- D104 pad 10: /DBG.SWDIO -> /XIO0
- D104 pad 2: /DBG.SWCLK -> /XIO1
- D104 pad 4: /DBG.SWO -> /XIO2
- D104 pad 5: /DBG.NRST -> /XIO3
- D104 pad 6: /DBG.NRST -> /XIO3
- D104 pad 7: /DBG.SWO -> /XIO2
- D104 pad 9: /DBG.SWCLK -> /XIO1
- D105 pad 1: Net-(J105-Pin_4) -> /XIO4
- D105 pad 10: Net-(J105-Pin_4) -> /XIO4
- D105 pad 2: Net-(J105-Pin_3) -> /XIO5
- D105 pad 4: Net-(J105-Pin_4) -> /XIO6
- D105 pad 5: Net-(J105-Pin_3) -> /XIO7
- D105 pad 6: Net-(J105-Pin_3) -> /XIO7
- D105 pad 7: Net-(J105-Pin_4) -> /XIO6
- D105 pad 9: Net-(J105-Pin_3) -> /XIO5
- D106 pad 1: /XIO0 -> /DBG.SWDIO
- D106 pad 10: /XIO0 -> /DBG.SWDIO
- D106 pad 2: /XIO1 -> /DBG.SWCLK
- D106 pad 4: /XIO2 -> /DBG.SWO
- D106 pad 5: /XIO3 -> /DBG.NRST
- D106 pad 6: /XIO3 -> /DBG.NRST
- D106 pad 7: /XIO2 -> /DBG.SWO
- D106 pad 9: /XIO1 -> /DBG.SWCLK
- D107 pad 1: /XIO4 -> /ENCU
- D107 pad 10: /XIO4 -> /ENCU
- D107 pad 2: /XIO5 -> /ENCV
- D107 pad 4: /XIO6 -> /ENCW
- D107 pad 5: /XIO7 -> /TMPM
- D107 pad 6: /XIO7 -> /TMPM
- D107 pad 7: /XIO6 -> /ENCW
- D107 pad 9: /XIO5 -> /ENCV
- J102 pad 1: /Phase A/PHASE -> /Phase C/PH
- J102 pad 2: /Phase B/PHASE -> /Phase B/PH
- J102 pad 3: /Phase C/PHASE -> /Phase A/PH
- J103 pad 9: +12V -> VBUS
- J105 pad 3: Net-(J105-Pin_3) -> /TMPM
- J105 pad 4: Net-(J105-Pin_4) -> /ENCW
- J105 pad 5: Net-(J105-Pin_3) -> /ENCV
- J105 pad 6: Net-(J105-Pin_4) -> /ENCU
- Q201 pad 1: /Power/VBST_{SW} -> VBUS
- Q201 pad 2: /Power/VBST_{PWM} -> /Phase A/GH
- Q201 pad 3: GND -> /Phase A/PH
- Q301 pad 1: /Phase A/PHASE -> VBUS
- Q301 pad 2: /Phase A/DH -> /Phase B/GH
- Q301 pad 3: Net-(Q301B-D2) -> /Phase B/PH
- Q302 pad 1: VBUS -> /Phase B/PH
- Q302 pad 2: /Phase A/GH -> /Phase B/GL
- Q302 pad 3: /Phase A/PHASE -> /Phase B/SP
- Q401 pad 1: /Phase B/PHASE -> VBUS
- Q401 pad 2: /Phase B/DH -> /Phase C/GH
- Q401 pad 3: Net-(Q401B-D2) -> /Phase C/PH
- R102 pad 1: /OSC_OUT_L -> VDD
- R102 pad 2: /OSC_OUT -> /TMPA
- R103 pad 1: VDD -> /OSC_OUT_L
- R103 pad 2: /QSPI.NCS -> /OSC_OUT
- R104 pad 2: /DBG.SWDIO -> /TMPB
- R105 pad 1: /DBG.SWCLK -> VDD
- R105 pad 2: GND -> /QSPI.NCS
- R106 pad 1: Net-(U101A-PB8-BOOT) -> VDD
- R106 pad 2: GND -> /DBG.SWDIO
- R201 pad 1: +12V -> /Phase A/PH
- R201 pad 2: /Power/12V_{FBM} -> /Phase A/FLT_{M}
- R202 pad 1: VBUS -> /Phase A/PH
- R202 pad 2: /Power/VBUS_{SENSE} -> /VSA
- R203 pad 1: /Power/12V_{FBM} -> /VSA
- R203 pad 2: /Power/12V_{FB} -> GND
- R204 pad 1: /Power/VBUS_{SENSE} -> /Phase A/SP
- R301 pad 1: VBST -> /Phase B/PH
- R301 pad 2: /Phase A/DH -> /Phase B/FLT_{M}
- R302 pad 1: Net-(Q301B-D2) -> /Phase B/PH
- R302 pad 2: /Phase A/GH -> /VSB
- R303 pad 1: /Phase A/GH -> /VSB
- R303 pad 2: Net-(Q301A-D1) -> GND
- R304 pad 1: /Phase A/HIGH -> /Phase B/SP
- R401 pad 1: VBST -> /Phase C/PH
- R401 pad 2: /Phase B/DH -> /Phase C/FLT_{M}
- R402 pad 1: Net-(Q401B-D2) -> /Phase C/PH
- R402 pad 2: /Phase B/GH -> /VSC
- R403 pad 1: /Phase B/GH -> /VSC
- R403 pad 2: Net-(Q401A-D1) -> GND
- R404 pad 1: /Phase B/HIGH -> /Phase C/SP
- U101 pad 10: /Phase A/TEMP -> /QSPI.IO5
- U101 pad 11: /Phase A/I_{SENSE} -> /QSPI.IO6
- U101 pad 12: /Phase B/V_{SENSE} -> /ENCU
- U101 pad 13: Net-(J105-Pin_4) -> /TMPM
- U101 pad 14: /Phase C/V_{SENSE} -> /ENCW
- U101 pad 17: /Power/VBST_{FB} -> /TMPB
- U101 pad 18: /XIO0 -> /VSM
- U101 pad 19: Net-(J105-Pin_3) -> /VSA
- U101 pad 2: unconnected-(U101A-PC13-Pad2) -> /XIO0
- U101 pad 22: /Phase B/TEMP -> /QSPI.IO7
- U101 pad 23: /Phase C/TEMP -> /VSB
- U101 pad 26: Net-(J105-Pin_3) -> /VSC
- U101 pad 3: unconnected-(U101A-PC14-OSC32_IN-Pad3) -> /XIO1
- U101 pad 34: /Phase C/I_{SENSE} -> /ISC
- U101 pad 35: /Phase B/I_{SENSE} -> /ISB
- U101 pad 36: /Phase C/LOW -> /GLC
- U101 pad 37: /Phase C/HIGH -> /GHC
- U101 pad 38: /Phase B/LOW -> /GLB
- U101 pad 39: /Phase B/HIGH -> /GHB
- U101 pad 4: unconnected-(U101A-PC15-OSC32_OUT-Pad4) -> /XIO2
- U101 pad 40: /Phase A/LOW -> /GLA
- U101 pad 41: /Phase A/HIGH -> /GHA
- U101 pad 42: /XIO1 -> /XIO3
- U101 pad 43: Net-(J105-Pin_4) -> /ISA
- U101 pad 44: /XIO2 -> /ENABLE
- U101 pad 45: /XIO3 -> /CAL
- U101 pad 46: /Power/VBST_{PWM} -> Net-(U101A-PA12-FAULT)
- U101 pad 53: /XIO5 -> /XIO4
- U101 pad 54: /XIO6 -> /ENCV
- U101 pad 55: /XIO7 -> /XIO5
- U101 pad 57: /XIO4 -> /XIO6
- U101 pad 61: Net-(U101A-PB8-BOOT) -> /BOOT
- U101 pad 62: unconnected-(U101A-PB9-Pad62) -> /XIO7
- U101 pad 8: /Phase A/V_{SENSE} -> /TMPA
- U101 pad 9: /Power/VBUS_{SENSE} -> /QSPI.IO4
- U102 pad 1: /CAN_TX -> Net-(U102B-FB)
- U102 pad 3: +5V -> Net-(U102B-CPL)
- U102 pad 4: /CAN_RX -> Net-(U102B-CPH)
- U102 pad 5: VDD -> Net-(U102B-VCP)
- U102 pad 6: /CANL -> VBUS
- U102 pad 7: /CANH -> VBUS
- U102 pad 8: GND -> /Phase A/GH
- U103 pad 1: GND -> /CAN_TX
- U103 pad 3: GND -> +5V
- U103 pad 4: GND -> /CAN_RX
- U103 pad 5: /LI2C_SDA -> VDD
- U103 pad 6: /LI2C_SCL -> /CANL
- U103 pad 7: GND -> /CANH
- U103 pad 8: VDD -> GND
- U104 pad 1: /QSPI.NCS -> GND
- U104 pad 2: /QSPI.IO1 -> GND
- U104 pad 3: /QSPI.IO2 -> GND
- U104 pad 5: /QSPI.IO0 -> /LI2C_SDA
- U104 pad 6: /QSPI.SCK -> /LI2C_SCL
- U104 pad 7: /QSPI.IO3 -> GND
Routing:
- net VBUS: vias 0 -> 39
- net GND: vias 0 -> 33
- added copper zone on B.Cu, net /Phase A/PH
- added copper zone on B.Cu, net /Phase A/SP
- added copper zone on B.Cu, net /Phase B/PH
- added copper zone on B.Cu, net /Phase B/SP
- added copper zone on B.Cu, net /Phase C/PH
- added copper zone on B.Cu, net /Phase C/SP
- added copper zone on B.Cu, net GND
- added copper zone on In1.Cu, net GND
- added copper zone on In4.Cu, net GND
- added copper zone on B.Cu, net VBUS
- added copper zone on F.Cu, net VBUS
Other:
- outline, holes or cut-outs redrawn

Commit message: Progress
Parts:
- removed the C112 at (-11.1, 92.5)
- removed the C114 at (0.49, 70.6)
- removed the C118 at (31.3, 91.2)
- removed the C125 at (32.0, -3.50)
- removed the C126 at (35.8, 7.25)
- removed the C136 at (46.2, -6.50)
- removed the C137 at (50.0, -8.75)
- removed the C138 at (43.5, -9.50)
- removed the C143 at (-5.25, 74.5)
- added C116: 220n, Capacitor_SMD:C_0402_1005Metric, B.Cu at (106.4, 26.7)
- added C117: 220n, Capacitor_SMD:C_0402_1005Metric, B.Cu at (106.4, 28.6)
- added C120: 2u2, Capacitor_SMD:C_0603_1608Metric, B.Cu at (80.8, 41.0)
- added C128: 220n, Capacitor_SMD:C_0402_1005Metric, B.Cu at (32.0, -3.25)
- added C129: 220n, Capacitor_SMD:C_0402_1005Metric, B.Cu at (46.5, 3.50)
- added C130: 220n, Capacitor_SMD:C_0402_1005Metric, B.Cu at (106.4, 36.5)
- added C139: 10u, Capacitor_SMD:C_1206_3216Metric, B.Cu at (46.8, -7.00)
- added C140: 10u, Capacitor_SMD:C_1206_3216Metric, B.Cu at (48.0, -10.8)
- added C141: 2u2, Capacitor_SMD:C_0603_1608Metric, B.Cu at (41.8, -10.0)
- added H103: M2.5, Bluesat:M2.5, F.Cu at (0.00, -12.5)
- added H104: M2.5, Bluesat:M2.5, F.Cu at (0.00, 12.5)
- C113: value 220n -> 330n-H; footprint Capacitor_SMD:C_0402_1005Metric -> Capacitor_SMD:C_0805_2012Metric
- H101, H102: moved to F.Cu
- moved C115 116.2 mm to (106.4, 24.7)
- moved Y101 112.2 mm to (48.5, -1.50), turned to -90 degrees
- moved R106 107.9 mm to (97.9, 44.2)
- moved R107 107.9 mm to (97.9, 46.2)
- moved R103 107.7 mm to (46.5, -1.00), turned to 90 degrees
- moved R101 107.1 mm to (97.9, 42.2)
- moved D107 104.5 mm to (78.2, 16.9)
- moved D104 104.5 mm to (88.8, 16.9)
- moved D105 104.5 mm to (85.2, 16.9)
- moved C113 95.8 mm to (83.3, 20.5)
- moved D101 94.8 mm to (79.9, 25.5)
- moved D102 94.8 mm to (79.9, 29.1)
- moved C118 94.4 mm to (63.5, 4.25)
- moved D103 92.8 mm to (52.8, 8.50), turned to 0 degrees
- moved C101 85.3 mm to (48.5, -3.75), turned to 0 degrees
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- renumbered C142 to C112, C141 to C114, C116 to C118, C117 to C121, C120 to C122, C121 to C123, C122 to C124, C123 to C125, C124 to C126, C128 to C131, C129 to C132, C130 to C133, C131 to C134, C132 to C135, C133 to C136, C134 to C137, C135 to C138, C139 to C142, C140 to C143
Connections:
- C113 pad 2: +5V -> VBUS
Other:
- board size 52 x 26 mm -> 56 x 28 mm

Commit message: Progress
Parts:
- moved L102 1.80 mm to (29.8, 7.58)
- moved D108 0.71 mm to (30.0, -4.50)
- moved D109 0.56 mm to (28.0, 1.75)
- moved C111 0.25 mm to (25.2, 8.50)
Connections:
- net Net-(D109-K) renamed /SW_{VDD}
- net Net-(U102B-CB) renamed /CB_{VDD}
- net Net-(U102B-CPH) renamed /DRV_{CPH}
- net Net-(U102B-CPL) renamed /DRV_{CPL}
- net Net-(U102B-FB) renamed /FB_{VDD}
- net Net-(U102B-VCP) renamed /DRV_{CP}
- net Net-(U102B-VREF) renamed /DRV_{VREF}
Routing:
- net GND: vias 33 -> 60
- net /SW_{VDD}: vias 0 -> 2
- added copper zone on F.Cu, net /SW_{VDD}
- added copper zone on F.Cu, net GND

Commit message: Sussy-fus
Parts:
- removed C112: 4u7-H, Capacitor_SMD:C_1210_3225Metric
- removed C113: 330n-H, Capacitor_SMD:C_0805_2012Metric
- C104, C105, C106, C114, C137, R106: moved to F.Cu
- D104: footprint Package_DFN_QFN:UDFN-10_1.35x2.6mm_P0.5mm -> Package_DFN_QFN:Diodes_UDFN-10_1x2.5mm_P0.5mm
- D105, D106, D107: footprint Package_DFN_QFN:UDFN-10_1.35x2.6mm_P0.5mm -> Package_DFN_QFN:Diodes_UDFN-10_1x2.5mm_P0.5mm; moved to F.Cu
- moved R101 108.3 mm to (4.00, -11.8)
- moved C115 107.0 mm to (5.62, -11.1), turned to 90 degrees
- moved C202 106.6 mm to (43.8, 30.3)
- moved C203 106.6 mm to (43.8, 32.3)
- moved C114 104.5 mm to (32.8, 1.75), turned to 0 degrees
- moved C402 103.5 mm to (52.9, 24.1)
- moved C403 103.5 mm to (52.9, 26.1)
- moved C116 102.0 mm to (5.62, 11.4), turned to 90 degrees
- moved C124 101.4 mm to (53.0, -6.25), turned to 0 degrees
- moved C132 90.1 mm to (37.0, 8.75)
- moved C302 88.5 mm to (48.9, 24.5)
- moved L101 87.9 mm to (36.5, 10.2)
- moved C131 84.7 mm to (37.0, 11.8)
- moved D102 83.9 mm to (6.50, -11.5), turned to 180 degrees
- moved R108 83.4 mm to (41.2, 22.8)
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Connections:
- C203 pad 1: GND -> /Phase A/SN
- C303 pad 1: GND -> /Phase B/SN
- C403 pad 1: GND -> /Phase C/SN
- D104 pad 1: /XIO0 -> /XIO1
- D104 pad 10: /XIO0 -> /XIO1
- D104 pad 2: /XIO1 -> /XIO3
- D104 pad 5: /XIO3 -> /XIO0
- D104 pad 6: /XIO3 -> /XIO0
- D104 pad 9: /XIO1 -> /XIO3
- D105 pad 1: /XIO4 -> /XIO6
- D105 pad 10: /XIO4 -> /XIO6
- D105 pad 2: /XIO5 -> /XIO4
- D105 pad 4: /XIO6 -> /XIO5
- D105 pad 7: /XIO6 -> /XIO5
- D105 pad 9: /XIO5 -> /XIO4
- D106 pad 1: /DBG.SWDIO -> /DBG.SWCLK
- D106 pad 10: /DBG.SWDIO -> /DBG.SWCLK
- D106 pad 2: /DBG.SWCLK -> /DBG.SWDIO
- D106 pad 9: /DBG.SWCLK -> /DBG.SWDIO
- U102 pad 12: GND -> /Phase A/SN
- U102 pad 13: GND -> /Phase B/SN
- U102 pad 22: GND -> /Phase C/SN
Routing:
- net GND: track 0.00 -> 60.7 mm, vias 60 -> 78
- net /Phase C/SP: track 0.00 -> 27.6 mm, vias 0 -> 3
- net /Phase B/SP: track 0.00 -> 20.0 mm, vias 0 -> 3
- net /Phase C/GL: track 0.00 -> 19.3 mm, vias 0 -> 3
- net /Phase A/SP: track 0.00 -> 16.6 mm, vias 0 -> 2
- net /Phase A/GH: track 0.00 -> 15.1 mm, vias 0 -> 3
- net /Phase C/PH: track 0.00 -> 14.5 mm, vias 0 -> 3
- net /Phase B/GL: track 0.00 -> 13.1 mm, vias 0 -> 3
- net /Phase C/GH: track 0.00 -> 12.6 mm, vias 0 -> 2
- net /Phase A/GL: track 0.00 -> 9.91 mm, vias 0 -> 2
- net /FB_{VDD}: track 0.00 -> 8.40 mm, vias 0 -> 2
- net /Phase A/PH: track 0.00 -> 7.87 mm, vias 0 -> 2
- net /TMPB: track 0.00 -> 7.17 mm, vias 0 -> 1
- net /DRV_{CP}: track 0.00 -> 6.93 mm
- net /Phase B/GH: track 0.00 -> 6.16 mm, vias 0 -> 2
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
Commit message: >_<
Parts:
- added C112: 100n-H, Capacitor_SMD:C_0603_1608Metric, B.Cu at (36.0, -11.8)
- C102, C107, C115, C116, C117, C136, C202, C302, C402, R101, R202, R203, R302, R303, R402, R403, TH101, TH102: moved to F.Cu
- C104, C114, C137, D105, D106, D107, R106: moved to B.Cu
- moved R403 96.7 mm to (51.8, 74.0)
- moved R101 96.5 mm to (-9.88, 83.8), turned to 0 degrees
- moved R402 93.8 mm to (51.8, 72.0), turned to 0 degrees
- moved R203 93.4 mm to (51.8, 94.1)
- moved R202 92.8 mm to (51.8, 92.1), turned to 0 degrees
- moved C115 89.3 mm to (15.2, 77.6), turned to 0 degrees
- moved C117 79.1 mm to (15.2, 81.5), turned to 0 degrees
- moved C116 68.9 mm to (15.2, 79.6), turned to 0 degrees
- moved R303 63.6 mm to (51.8, 53.9)
- moved R302 63.1 mm to (51.8, 51.9), turned to 0 degrees
- moved H103 60.0 mm to (60.0, -12.2)
- moved H104 60.0 mm to (60.0, 12.2)
- moved H101 56.0 mm to (0.00, -12.2)
- moved H102 56.0 mm to (0.00, 12.2)
- moved C119 48.2 mm to (26.2, -9.25), turned to 90 degrees
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Routing:
- net GND: track 60.7 -> 1.42 mm, vias 78 -> 54
- net /Phase C/SP: track 27.6 -> 1.42 mm, vias 3 -> 0
- net /Phase C/GL: track 19.3 -> 0.00 mm, vias 3 -> 0
- net /Phase B/SP: track 20.0 -> 1.42 mm, vias 3 -> 0
- net /Phase A/SP: track 16.6 -> 1.34 mm, vias 2 -> 0
- net /Phase A/GH: track 15.1 -> 0.00 mm, vias 3 -> 0
- net /Phase C/PH: track 14.5 -> 0.00 mm, vias 3 -> 0
- net /Phase B/GL: track 13.1 -> 0.00 mm, vias 3 -> 0
- net /Phase C/GH: track 12.6 -> 0.00 mm, vias 2 -> 0
- net /Phase A/GL: track 9.91 -> 0.00 mm, vias 2 -> 0
- net /FB_{VDD}: track 8.40 -> 0.00 mm, vias 2 -> 0
- net /Phase A/PH: track 7.87 -> 0.00 mm, vias 2 -> 0
- net /TMPB: track 7.17 -> 0.00 mm, vias 1 -> 0
- net /DRV_{CP}: track 6.93 -> 0.00 mm
- net /Phase B/GH: track 6.16 -> 0.00 mm, vias 2 -> 0
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- added copper zone on B.Cu, net /DRV_{CP}
- added copper zone on B.Cu, net /DVDD
- added copper zone on In2.Cu, net GND
- added copper zone on In3.Cu, net GND
- removed copper zone on B.Cu, net /Phase A/PH
- removed copper zone on B.Cu, net /Phase A/SP
- removed copper zone on B.Cu, net /Phase B/PH
- removed copper zone on B.Cu, net /Phase B/SP
- removed copper zone on B.Cu, net /Phase C/PH
- removed copper zone on B.Cu, net /Phase C/SP
- removed copper zone on F.Cu, net /SW_{VDD}
- removed copper zone on F.Cu, net VBUS
Other:
- board size 56 x 28 mm -> 60 x 28 mm
