File: src/wark_min/wark_min.kicad_sch (KiCad schematic)
At the start: 43 parts, among them J101 SM02B-PASS, J102 MR60, J103 BM12B-ZPDSS, J104 IDC6, J105 SM06B-PASS, U101 STM32G474_WarkMin, U102 TCAN1462V, U103 ZD24C128A, U104 ZD25WQ16C, Y101 24Mhz

Commit message: Small pile becomes big pile
Parts:
- added H101, H102: M2.5, Bluesat:M2.5, symbol Mechanical:MountingHole
- J101: footprint Bluesat:SM02B-PASS -> Bluesat:BM02B-PASS
- J105: footprint Bluesat:SM06B-PASS -> Bluesat:BM06B-PASS
Changed lines of the file:
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@@
 	)
 	(symbol
+		(lib_id "Mechanical:MountingHole")
+		(at 190.5 152.4 0)
+		(unit 1)
+		(exclude_from_sim no)
+		(in_bom no)
+		(on_board yes)
+		(dnp no)
+		(fields_autoplaced yes)
+		(property "Reference" "H102"
+			(at 193.04 151.1299 0)
+			(effects
+				(font
+					(size 1.27 1.27)
+				)
+				(justify left)
+			)
+		)
+		(property "Value" "M2.5"
+			(at 193.04 153.6699 0)
+			(effects
+				(font
+					(size 1.27 1.27)
+				)
+				(justify left)
+			)
+		)
+		(property "Footprint" "Bluesat:M2.5"
+			(at 190.5 152.4 0)
+			(effects
+				(font
+					(size 1.27 1.27)
+				)
+				(hide yes)
+			)
+		)
+		(property "Datasheet" "~"
+			(at 190.5 152.4 0)
+			(effects
+				(font
+					(size 1.27 1.27)
+				)
+				(hide yes)
+			)
+		)
+		(property "Description" "Mounting Hole without connection"
+			(at 190.5 152.4 0)
+			(effects
+				(font
+					(size 1.27 1.27)
+				)
+				(hide yes)
+			)
+		)
+		(instances
+			(project "wark_min"
+				(path "/4290b658-b789-4580-aa76-416e95a5eb26"
+					(reference "H102")
+					(unit 1)
+				)
+			)
+		)
+	)
+	(symbol
 		(lib_id "Bluesat:ZD25WQ16C")
 		(at 25.4 80.01 0)
@@
 			)
 		)
-		(property "Footprint" "Bluesat:SM06B-PASS"
+		(property "Footprint" "Bluesat:BM06B-PASS"
 			(at 160.02 132.08 0)
 			(effects
@@
 		(on_board yes)
 		(dnp no)
-		(fields_autoplaced yes)
 		(property "Reference" "U101"
 			(at 114.3 19.05 0)
@@
 	)
 	(symbol
+		(lib_id "Mechanical:MountingHole")
+		(at 177.8 152.4 0)
+		(unit 1)
+		(exclude_from_sim no)
+		(in_bom no)
+		(on_board yes)
+		(dnp no)
+		(fields_autoplaced yes)
+		(property "Reference" "H101"
+			(at 180.34 151.1299 0)
+			(effects
+				(font
+					(size 1.27 1.27)
+				)
+				(justify left)
+			)
+		)
+		(property "Value" "M2.5"
+			(at 180.34 153.6699 0)
+			(effects
+				(font
+					(size 1.27 1.27)
+				)
+				(justify left)
+			)
+		)
+		(property "Footprint" "Bluesat:M2.5"
+			(at 177.8 152.4 0)
+			(effects
+				(font
+					(size 1.27 1.27)
+				)
+				(hide yes)
+			)
+		)
+		(property "Datasheet" "~"
+			(at 177.8 152.4 0)
+			(effects
+				(font
+					(size 1.27 1.27)
+				)
+				(hide yes)
+			)
+		)
+		(property "Description" "Mounting Hole without connection"
+			(at 177.8 152.4 0)
+			(effects
+				(font
+					(size 1.27 1.27)
+				)
+				(hide yes)
+			)
+		)
+		(instances
+			(project ""
+				(path "/4290b658-b789-4580-aa76-416e95a5eb26"
+					(reference "H101")
+					(unit 1)
+				)
+			)
+		)
+	)
+	(symbol
 		(lib_id "Bluesat:R_CompactV")
 		(at 91.44 129.54 0)
@@
 			)
 		)
-		(property "Footprint" "Bluesat:SM02B-PASS"
+		(property "Footprint" "Bluesat:BM02B-PASS"
 			(at 22.86 44.45 0)
 			(effects

Commit message: Pre-stupid
Parts:
- removed C103: 10n, Capacitor_SMD:C_0402_1005Metric, symbol Bluesat:C_CompactV
- removed C108: 220n, Capacitor_SMD:C_0402_1005Metric, symbol Bluesat:C_CompactV
- removed C109: 10u, Capacitor_SMD:C_1206_3216Metric, symbol Bluesat:C_CompactV
- removed D104: 3V3, Package_DFN_QFN:Diodes_UDFN-10_1x2.5mm_P0.5mm, symbol Bluesat:D_TVS_Quad_Compact
- removed R103: 10k, Resistor_SMD:R_0402_1005Metric, symbol Bluesat:R_CompactH
- added C102, C121, C122, C123, C124, C125, C126, C127, C130, C140, C143: 220n, Capacitor_SMD:C_0402_1005Metric, symbol Bluesat:C_CompactV
- added C108, C109: 270u, Capacitor_SMD:CP_Elec_10x10, symbol Device:C_Polarized_Small_US
- added C128, C129: 2u2, Capacitor_SMD:C_0603_1608Metric, symbol Bluesat:C_CompactV
- added C131: 100n, Capacitor_SMD:C_0402_1005Metric, symbol Bluesat:C_CompactH
- added C132: 1u-M, Capacitor_SMD:C_0805_2012Metric, symbol Bluesat:C_CompactH
- added C133: 22u, Capacitor_SMD:C_1210_3225Metric, symbol Bluesat:C_CompactV
- added C134: 10n, Capacitor_SMD:C_0402_1005Metric, symbol Bluesat:C_CompactV
- added C135: 33n, Capacitor_SMD:C_0402_1005Metric, symbol Bluesat:C_CompactH
- added C136, C137: 10u, Capacitor_SMD:C_1206_3216Metric, symbol Bluesat:C_CompactV
- added C138: 2u2, Capacitor_SMD:C_0603_1608Metric, symbol Bluesat:C_CompactH
- added C139: 1u, Capacitor_SMD:C_0603_1608Metric, symbol Bluesat:C_CompactV
- added C141: 100n-H, Capacitor_SMD:C_0603_1608Metric, symbol Bluesat:C_CompactV
- added C142: 4u7-H, Capacitor_SMD:C_1210_3225Metric, symbol Bluesat:C_CompactV
- added D106: 3V3, Package_DFN_QFN:UDFN-10_1.35x2.6mm_P0.5mm, symbol Bluesat:D_TVS_Quad_Compact
- added D108: 30V, Diode_SMD:D_SOD-123F, symbol Device:D_Zener_Small
- added D109: 500mA, Diode_SMD:D_SOD-123, symbol Device:D_Schottky_Small
- added J106: XT30M, Connector_AMASS:AMASS_XT30U-M_1x02_P5.0mm_Vertical, symbol Connector:Conn_01x02_Pin
- added L101: 600R, Resistor_SMD:R_0402_1005Metric, symbol Device:L_Ferrite_Small
- added L102: 47u-1A, Inductor_SMD:L_Changjiang_FXL0630, symbol Device:L_Small
- added R102, R104: 2k2, Resistor_SMD:R_0402_1005Metric, symbol Bluesat:R_CompactV
- added R105: 10k, Resistor_SMD:R_0402_1005Metric, symbol Bluesat:R_CompactH
- added R109: 220k, Resistor_SMD:R_0402_1005Metric, symbol Bluesat:R_CompactV
- added R110: 33k, Resistor_SMD:R_0402_1005Metric, symbol Bluesat:R_CompactV
- added R111, R112: 10k, Resistor_SMD:R_0402_1005Metric, symbol Bluesat:R_CompactV
- added TH101, TH102: 10k, Resistor_SMD:R_0402_1005Metric, symbol Device:Thermistor
- added U102: DRV8323RH, Package_DFN_QFN:Texas_RGZ0048A_VQFN-48-1EP_7x7mm_P0.5mm_EP5.15x5.15mm, symbol Bluesat:DRV8323RH
- added U105: ZD25WQ16C, Package_SON:Winbond_USON-8-1EP_3x2mm_P0.5mm_EP0.2x1.6mm, symbol Bluesat:ZD25WQ16C
- added U107: HX4002, Package_TO_SOT_SMD:SOT-23-6, symbol Regulator_SwitchedCapacitor:LTC1754
- C104: value 1u-M -> 100n; footprint Capacitor_SMD:C_0805_2012Metric -> Capacitor_SMD:C_0402_1005Metric
- C105: value 2u2 -> 100n; footprint Capacitor_SMD:C_0603_1608Metric -> Capacitor_SMD:C_0402_1005Metric
- C106: value 220n -> 100n
- C110, C111: value 2u2 -> 4u7-H; footprint Capacitor_SMD:C_0603_1608Metric -> Capacitor_SMD:C_1210_3225Metric
- C112: value 2u2 -> 330n-H; footprint Capacitor_SMD:C_0603_1608Metric -> Capacitor_SMD:C_0805_2012Metric
- C116: value 220n -> 10n
- C117, C118, C119: value 220n -> 2u2; footprint Capacitor_SMD:C_0402_1005Metric -> Capacitor_SMD:C_0603_1608Metric
- D104: renamed from D106; footprint Package_DFN_QFN:Diodes_UDFN-10_1x2.5mm_P0.5mm -> Package_DFN_QFN:UDFN-10_1.35x2.6mm_P0.5mm
- D105: renamed from D107; footprint Package_DFN_QFN:Diodes_UDFN-10_1x2.5mm_P0.5mm -> Package_DFN_QFN:UDFN-10_1.35x2.6mm_P0.5mm
- D107: renamed from D105; footprint Package_DFN_QFN:Diodes_UDFN-10_1x2.5mm_P0.5mm -> Package_DFN_QFN:UDFN-10_1.35x2.6mm_P0.5mm
- U101: value STM32G474_WarkMin -> STM32G474; Height (none) -> 1.6
- U103: renamed from U102; footprint Package_SO:JEITA_SOIC-8_3.9x4.9mm_P1.27mm -> Package_SO:SOIC-8_3.9x4.9mm_P1.27mm
- renumbered C102 to C103, R102 to R103, R104 to R106, R105 to R107, R106 to R108, U103 to U104, U104 to U106
Connections:
- net +5V: now also C113.2, C114.2, C115.2, C137.2, U107.1 (VOUT); no longer C105.2, C106.2, C107.2
- net DBG.NRST: now also C116.2, D106.5, D106.6
- net DBG.SWCLK: now also D106.2, D106.9
- net DBG.SWDIO: now also D106.1, D106.10
- net DBG.SWO: now also D106.4, D106.7
- net GND: now also C102.1, C108.2, C109.2, C121.1, C122.1, C123.1, C124.1, C125.1, C126.1, C127.1, C128.1, C129.1, C130.1, C133.1, C134.1, C136.1, C137.1, C139.1, C140.1, C141.1, C142.1, C143.1, D106.3, D106.8, D108.2 (A), D109.2 (A), J106.1 (Pin_1), R111.2, R112.2, TH101.2, TH102.2, U102.2 (PGND), U102.27 (DGND), U102.29 (MODE), U102.35 (AGND), U102.43 (BGND), U102.49 (EP), U105.4 (VSS), U107.2 (GND)
- net QSPI.NCS: now also R105.2, U105.1 (~{CS})
- net QSPI.SCK: now also U105.6 (SCK)
- net VDD: now also C120.2, C121.2, C122.2, C123.2, C124.2, C125.2, C126.2, C127.2, C128.2, C133.2, C136.2, L101.1, L102.2, R102.1, R104.1, R105.1, R110.1, U105.8 (VCC), U107.3 (~{SHDN}), U107.5 (VIN); no longer C110.2, C111.2, C112.2, C113.2, C114.2, C115.2, C116.2
- net VDDA: now also C129.2, C130.2, L101.2; no longer C120.2
- net XIO0: now also U101.2 (PC13-XIO0); no longer U101.18 (PA4-XIO0)
- net XIO1: now also U101.3 (PC14-XIO1); no longer U101.42 (PA8-XIO1)
- net XIO2: now also U101.4 (PC15-XIO2); no longer U101.44 (PA10-XIO2)
- net XIO3: now also U101.42 (PA8-XIO3); no longer U101.45 (PA11-XIO3)
- net XIO4: now also U101.53 (PC11-XIO4); no longer U101.57 (PB4-XIO4)
- net XIO5: now also U101.55 (PD2-XIO5); no longer U101.53 (PC11-XIO5)
- net XIO6: now also U101.57 (PB4-XIO6); no longer U101.54 (PC12-XIO6)
- net XIO7: now also U101.62 (PB9-XIO7); no longer U101.55 (PD2-XIO7)
- net ARGB_{0}: now reaches D102.3 (DIN), R101.2, U101.52 (PC10-ARGB)
- net BOOT: now reaches R108.1, U101.61 (PB8-BOOT)
- net ARGB_{1}: now reaches D101.3 (DIN), D102.1 (DOUT)
- net +12V renamed ISA
- net ISA: now also U101.43 (PA9-ISA), U102.25 (SOA); no longer J103.9 (Pin_9)
- net Phase A/HIGH renamed GHA
- net GHA: now also U102.37 (INHA)
- net Phase A/I_{SENSE} renamed QSPI.IO6
- net QSPI.IO6: now also U105.3 (IO2)
- net Phase A/LOW renamed GLA
- net GLA: now also U102.38 (INLA)
- net Phase A/PHASE renamed Phase C/PH
- net Phase A/TEMP renamed QSPI.IO5
- net QSPI.IO5: now also U105.2 (IO1)
- net Phase A/V_{SENSE} renamed TMPA
- net TMPA: now also C102.2, R102.2, TH101.1
- net Phase B/HIGH renamed GHB
- net GHB: now also U102.39 (INHB)
- net Phase B/I_{SENSE} renamed ISB
- net ISB: now also C105.2, U102.24 (SOB)
- net Phase B/LOW renamed GLB
- net GLB: now also U102.40 (INLB)
- net Phase B/PHASE renamed Phase B/PH
- net Phase B/TEMP renamed QSPI.IO7
- net QSPI.IO7: now also U105.7 (IO3)
- net Phase B/V_{SENSE} renamed ENCU
- net ENCU: now also D107.1, D107.10, J105.6 (Pin_6)
- net Phase C/HIGH renamed GHC
- net GHC: now also U102.41 (INHC)
- net Phase C/I_{SENSE} renamed ISC
- net ISC: now also C106.2, U102.23 (SOC)
- net Phase C/LOW renamed GLC
- net GLC: now also U102.42 (INLC)
- net Phase C/PHASE renamed Phase A/PH
- net Phase C/TEMP renamed VSB
- net Phase C/V_{SENSE} renamed ENCW
- net ENCW: now also D107.4, D107.7, J105.4 (Pin_4)
- net Power/VBST_{FB} renamed TMPB
- net TMPB: now also C107.2, R104.2, TH102.1
- net Power/VBST_{PWM}: no longer names the net of U101.46 (PA12-FAULT)
- net Power/VBST_{PWM}: now also U102.28 (~{FAULT})
- net Power/VBUS_{SENSE} renamed QSPI.IO4
- net QSPI.IO4: now also U105.5 (IO0)
- new net: C131.1, D109.1 (K), L102.1, U102.45 (SW)
- new net: C131.2, U102.44 (CB)
- new net: R110.2, R112.1, U102.1 (FB)
- new net: C140.2, U102.26 (VREF)
- new net: C135.1, U102.3 (CPL)
- new net: C135.2, U102.4 (CPH)
- new net: C132.1, U102.5 (VCP)
- new net CAL: U101.45 (PA11-CAL), U102.34 (CAL)
- new net CP+: C138.2, U107.6 (CP+)
- new net CP-: C138.1, U107.4 (CP-)
- new net DVDD: C139.2, U102.30 (IDRIVE), U102.31 (VDS), U102.32 (GAIN), U102.36 (DVDD)
- new net ENABLE: U101.44 (PA10-ENABLE), U102.33 (ENABLE)
- new net ENCV: D107.2, D107.9, J105.5 (Pin_5), U101.54 (PC12-ENCV)
- new net Phase A/GH: U102.8 (GHA)
- new net Phase A/GL: U102.10 (GLA)
- new net Phase A/SH: U102.9 (SHA)
- new net Phase A/SN: U102.12 (SNA)
- new net Phase A/SP: U102.11 (SPA)
- new net Phase B/GH: U102.17 (GHB)
- new net Phase B/GL: U102.15 (GLB)
- new net Phase B/SH: U102.16 (SHB)
- new net Phase B/SN: U102.13 (SNB)
- new net Phase B/SP: U102.14 (SPB)
- new net Phase C/GH: U102.18 (GHC)
- new net Phase C/GL: U102.20 (GLC)
- new net Phase C/SH: U102.19 (SHC)
- new net Phase C/SN: U102.22 (SNC)
- new net Phase C/SP: U102.21 (SPC)
- new net TMPM: C143.2, D107.5, D107.6, J105.3 (Pin_3), U101.13 (PA1-TMPM)
- new net VBUS: C108.1, C109.1, C110.2, C111.2, C112.2, C132.2, C141.2, C142.2, D108.1 (K), J103.9 (Pin_9), J106.2 (Pin_2), R109.1, U102.47 (VIN), U102.6 (VM), U102.7 (VDRAIN)
- new net VSA: U101.19 (PA5-VSA)
- new net VSC: U101.26 (PB2-VSC)
- new net VSM: C134.2, R109.2, R111.1, U101.18 (PA4-VSM)
- no-connect marks 1 -> 2
Other:
- removed sheet Power
- sheet Phase A ports: added GH, GL, PH, SH, SN, SP, VS; removed HIGH, I_{SENSE}, LOW, PHASE, TEMP, V_{SENSE}
- sheet Phase B ports: added GH, GL, PH, SH, SN, SP, VS; removed HIGH, I_{SENSE}, LOW, PHASE, TEMP, V_{SENSE}
- sheet Phase C ports: added GH, GL, PH, SH, SN, SP, VS; removed HIGH, I_{SENSE}, LOW, PHASE, TEMP, V_{SENSE}
- note added: "BW=1/(2π*10k*10n)=1.6kHz"
- note added: "BW=1/(2π*2k2*220n)=329Hz"
- note added: "MODE: 6x PWM Mode IDRIVE: 1/2A VDS: Disabled GAIN: 40V/V"
- moved on the sheet: C101, C103, D101, D102, D103, D104, D105, D107, H101, H102, J101, J102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

Commit message: Progress
Parts:
- added H103, H104: M2.5, Bluesat:M2.5, symbol Mechanical:MountingHole
- renumbered C142 to C112, C112 to C113, C141 to C114, C113 to C115, C114 to C116, C115 to C117, C116 to C118, C118 to C119, C119 to C120, C117 to C121, C120 to C122, C121 to C123, C122 to C124, C123 to C125, C124 to C126, C125 to C127, C126 to C128, C127 to C129, C143 to C130, C128 to C131, C129 to C132, C130 to C133, C131 to C134, C132 to C135, C133 to C136, C134 to C137, C135 to C138, C136 to C139, C137 to C140, C138 to C141, C139 to C142, C140 to C143
Other:
- moved on the sheet: C119, C120, C121, C139, C140, C141, U107

Commit message: Progress
Connections:
- net SW_{VDD}: now reaches C134.1, D109.1 (K), L102.1, U102.45 (SW)
- net CB_{VDD}: now reaches C134.2, U102.44 (CB)
- net FB_{VDD}: now reaches R110.2, R112.1, U102.1 (FB)
- net DRV_{VREF}: now reaches C143.2, U102.26 (VREF)
- net DRV_{CPL}: now reaches C138.1, U102.3 (CPL)
- net DRV_{CPH}: now reaches C138.2, U102.4 (CPH)
- net DRV_{CP}: now reaches C135.1, U102.5 (VCP)
Changed lines of the file:
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@@
+		)
+	)
+	(label "SW_{VDD}"
+		(at 104.14 162.56 0)
+		(effects
+			(font
+				(size 0.381 0.381)
+			)
+			(justify left bottom)
 		)
 	)
@@
 		)
 	)
+	(label "DRV_{CPL}"
+		(at 73.66 177.8 180)
+		(effects
+			(font
+				(size 0.381 0.381)
+			)
+			(justify right bottom)
+		)
+	)
 	(label "XIO3"
 		(at 168.91 119.38 90)
@@
 		)
 	)
+	(label "DRV_{CPH}"
+		(at 73.66 170.18 180)
+		(effects
+			(font
+				(size 0.381 0.381)
+			)
+			(justify right bottom)
+		)
+	)
 	(label "QSPI.SCK"
 		(at 44.45 85.09 0)
@@
 		)
 	)
+	(label "DRV_{VREF}"
+		(at 73.66 182.88 180)
+		(effects
+			(font
+				(size 0.381 0.381)
+			)
+			(justify right bottom)
+		)
+	)
 	(label "OSC_OUT"
 		(at 99.06 46.99 270)
@@
 		)
 	)
+	(label "CB_{VDD}"
+		(at 104.14 154.94 0)
+		(effects
+			(font
+				(size 0.381 0.381)
+			)
+			(justify left bottom)
+		)
+	)
 	(label "XIO1"
 		(at 177.8 96.52 0)
@@
 		)
 	)
+	(label "DRV_{CP}"
+		(at 73.66 167.64 180)
+		(effects
+			(font
+				(size 0.381 0.381)
+			)
+			(justify right bottom)
+		)
+	)
 	(label "QSPI.NCS"
 		(at 44.45 100.33 0)
@@
 			)
 			(justify left bottom)
+		)
+	)
+	(label "FB_{VDD}"
+		(at 104.14 165.1 0)
+		(effects
+			(font
+				(size 0.381 0.381)
+			)
+			(justify left bottom)

Commit message: Sussy-fus
Parts:
- removed C112: 4u7-H, Capacitor_SMD:C_1210_3225Metric, symbol Bluesat:C_CompactV
- removed C113: 330n-H, Capacitor_SMD:C_0805_2012Metric, symbol Bluesat:C_CompactV
- D104, D105, D106, D107: footprint Package_DFN_QFN:UDFN-10_1.35x2.6mm_P0.5mm -> Package_DFN_QFN:Diodes_UDFN-10_1x2.5mm_P0.5mm
Connections:
- net DBG.SWCLK: now also D106.1, D106.10; no longer D106.2, D106.9
- net DBG.SWDIO: now also D106.2, D106.9; no longer D106.1, D106.10
- net XIO0: now also D104.5, D104.6; no longer D104.1, D104.10
- net XIO1: now also D104.1, D104.10; no longer D104.2, D104.9
- net XIO3: now also D104.2, D104.9; no longer D104.5, D104.6
- net XIO4: now also D105.2, D105.9; no longer D105.1, D105.10
- net XIO5: now also D105.4, D105.7; no longer D105.2, D105.9
- net XIO6: now also D105.1, D105.10; no longer D105.4, D105.7
Other:
- moved on the sheet: C109, C110, C111, C114

Commit message: >_<
Parts:
- added C112: 100n-H, Capacitor_SMD:C_0603_1608Metric, symbol Bluesat:C_CompactV
Connections:
- net GND: now also C112.1
- net VBUS: now also C112.2
Changed lines of the file:
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@@
 	)
 	(junction
+		(at 246.38 87.63)
+		(diameter 0)
+		(color 0 0 0 0)
+	)
+	(junction
 		(at 241.3 109.22)
 		(diameter 0)
@@
 	(wire
 		(pts
+			(xy 246.38 87.63) (xy 250.19 87.63)
+		)
+		(stroke
+			(width 0)
+			(type default)
+		)
+	)
+	(wire
+		(pts
 			(xy 240.03 147.32) (xy 240.03 149.86)
 		)
@@
 		)
 	)
+	(wire
+		(pts
+			(xy 250.19 92.71) (xy 250.19 87.63)
+		)
+		(stroke
+			(width 0)
+			(type default)
+		)
+	)
 	(bus
 		(pts
@@
 		(lib_name "C_CompactV_2")
 		(lib_id "Bluesat:C_CompactV")
+		(at 250.19 95.25 0)
+		(unit 1)
+		(exclude_from_sim no)
+		(in_bom yes)
+		(on_board yes)
+		(dnp no)
+		(fields_autoplaced yes)
+		(property "Reference" "C112"
+			(at 249.301 94.488 90)
+			(do_not_autoplace yes)
+			(effects
+				(font
+					(size 1.016 1.016)
+				)
+				(justify left)
+			)
+		)
+		(property "Value" "100n-H"
+			(at 251.079 94.488 90)
+			(do_not_autoplace yes)
+			(effects
+				(font
+					(size 1.016 1.016)
+				)
+				(justify left)
+			)
+		)
+		(property "Footprint" "Capacitor_SMD:C_0603_1608Metric"
+			(at 250.19 95.25 90)
+			(effects
+				(font
+					(size 1.27 1.27)
+				)
+				(hide yes)
+			)
+		)
+		(property "Datasheet" "~"
+			(at 250.19 95.25 90)
+			(effects
+				(font
+					(size 1.27 1.27)
+				)
+				(hide yes)
+			)
+		)
+		(property "Description" "Unpolarized capacitor, compact symbol"
+			(at 250.19 95.25 0)
+			(effects
+				(font
+					(size 1.27 1.27)
+				)
+				(hide yes)
+			)
+		)
+		(pin "1"
+		)
+		(pin "2"
+		)
+		(instances
+			(project "wark_min"
+				(path "/4290b658-b789-4580-aa76-416e95a5eb26"
+					(reference "C112")
+					(unit 1)
+				)
+			)
+		)
+	)
+	(symbol
+		(lib_name "C_CompactV_2")
+		(lib_id "Bluesat:C_CompactV")
 		(at 237.49 152.4 0)
 		(unit 1)
@@
 				)
 			)
+		)
+	)
+	(symbol
+		(lib_id "power:GND")
+		(at 250.19 97.79 0)
+		(unit 1)
+		(exclude_from_sim no)
+		(in_bom yes)
+		(on_board yes)
+		(dnp no)
+		(property "Reference" "#PWR0138"
+			(at 250.19 104.14 0)
+			(effects
+				(font
+					(size 1.27 1.27)
+				)
+				(hide yes)
+			)
+		)
+		(property "Value" "GND"
+			(at 250.19 101.092 0)
+			(effects
+				(font
+					(size 0.762 0.762)
+				)
+			)
+		)
+		(property "Footprint" ""
+			(at 250.19 97.79 0)
+			(effects
+				(font
+					(size 1.27 1.27)
+				)
+				(hide yes)
+			)
+		)
+		(property "Datasheet" ""
+			(at 250.19 97.79 0)
+			(effects
+				(font
+					(size 1.27 1.27)
+				)
+				(hide yes)
+			)
+		)
+		(property "Description" "Power symbol creates a global label with name \"GND\" , ground"
+			(at 250.19 97.79 0)
+			(effects
+				(font
+					(size 1.27 1.27)
+				)
+				(hide yes)
+			)
+		)
+		(pin "1"
+		)
+		(instances
+			(project "wark_min"
+				(path "/4290b658-b789-4580-aa76-416e95a5eb26"
+					(reference "#PWR0138")
+					(unit 1)
+				)
+			)
