Commit message: Fix simulation, format files

File: src/rover/description/core/db_helpers.xacro (robot description, xacro)
@@ -21,5 +21,6 @@
 	    <origin xyz="${0} ${0} ${-0.213/2 - 0.03/2}" rpy="0 0 0"/>
             <axis xyz="0 0 1"/>
-            <limit lower="${-pi/2}" upper="${pi/2}" effort="40.0" velocity="12.8"/>
+            <!-- FIXME these are the actual limits <limit lower="${-pi/2}" upper="${pi/2}" velocity="5"/> -->
+            <limit lower="${-pi}" upper="${pi}" effort="400" velocity="5"/>
         </joint>
         <!-- This is the actual wheel -->

File: src/rover/description/core/ros2_control.xacro (robot description, xacro)
@@ -5,6 +5,6 @@
             <joint name="db_${name}_fork_tyre_joint">
                 <command_interface name="velocity">
-                    <param name="min">-2</param>
-                    <param name="max">2</param>
+                    <param name="min">-0.3</param>
+                    <param name="max">0.3</param>
                 </command_interface>
                 <state_interface name="position"/>
@@ -13,6 +13,7 @@
             <joint name="db_${name}_smount_fork_joint">
                 <command_interface name="position">
-                    <param name="min">-2</param>
-                    <param name="max">2</param>
+                    <limits enable="true"/>
+                    <param name="min">-1.6</param>
+                    <param name="max">1.6</param>
                 </command_interface>
                 <state_interface name="position"/>
@@ -50,10 +51,3 @@
         <!-- TODO: Drivebase turn motors -->
     </ros2_control>
-    <xacro:if value="$(arg is_simulation)">
-        <gazebo>
-            <plugin filename="gz_ros2_control-system" name="gz_ros2_control::GazeboSimROS2ControlPlugin">
-                <parameters>$(find rover)/config/drivebase/swerve_drive_controller.yaml</parameters>
-            </plugin>
-        </gazebo>
-    </xacro:if>
 </robot>

File: src/rover/description/robot.urdf.xacro (robot description, xacro)
@@ -11,4 +11,5 @@
     <xacro:include filename="utils/inertial_macros.xacro" />
     <xacro:include filename="utils/materials.xacro" />
+    <!-- simulation specific global stuff -->
     <xacro:if value="$(arg is_simulation)">
         <xacro:include filename="utils/gazebo_plugins.xacro" />
@@ -16,7 +17,3 @@
     <xacro:include filename="core/core.xacro" />
     <!--<xacro:include filename="cameras/depth_cams.xacro" /> -->
-    <!-- simulation specific global stuff -->
-    <xacro:if value="$(arg is_simulation)">
-        <xacro:include filename="utils/gazebo_plugins.xacro" />
-    </xacro:if>
 </robot>

File: src/rover/description/utils/gazebo_plugins.xacro (robot description, xacro)
@@ -1,4 +1,12 @@
 <?xml version="1.0"?>
 <robot xmlns:xacro="http://www.ros.org/wiki/xacro" >
+    <!-- ros_control plugin -->
+    <xacro:if value="$(arg is_simulation)">
+        <gazebo>
+            <plugin filename="gz_ros2_control-system" name="gz_ros2_control::GazeboSimROS2ControlPlugin">
+                <parameters>$(find rover)/config/core/shared_controllers.yaml</parameters>
+            </plugin>
+        </gazebo>
+    </xacro:if>
     <gazebo>
         <!-- Joint states publisher -->

Commit message: Clean up ros2control usage in URDF

File: src/rover/description/core/db_helpers.xacro (robot description, xacro)
@@ -19,8 +19,7 @@
             <parent link="${prefix}_smount"/>
             <child link="${prefix}_wheel_fork"/>
-	    <origin xyz="${0} ${0} ${-0.213/2 - 0.03/2}" rpy="0 0 0"/>
+	        <origin xyz="${0} ${0} ${-0.213/2 - 0.03/2}" rpy="0 0 0"/>
             <axis xyz="0 0 1"/>
-            <!-- FIXME these are the actual limits <limit lower="${-pi/2}" upper="${pi/2}" velocity="5"/> -->
-            <limit lower="${-pi}" upper="${pi}" effort="400" velocity="5"/>
+            <limit lower="${-pi/2}" upper="${pi/2}" effort="400" velocity="5"/>
         </joint>
         <!-- This is the actual wheel -->
@@ -30,4 +29,5 @@
             <origin xyz="0 0 ${-0.05}" rpy="${-pi/2} 0 0" />
             <axis xyz="0 0 1"/>
+            <limit effort="400" velocity="0.2"/>
         </joint>
         <!-- ALL LINKS BELOW THIS LINE -->

File: src/rover/description/core/ros2_control.xacro (robot description, xacro)
@@ -1,22 +1,26 @@
 <?xml version="1.0"?>
 <robot xmlns:xacro="http://www.ros.org/wiki/xacro">
+    <!-- Specify the joints that are in a single swerve module, limits are specified in joint declaration! -->
     <xacro:if value="$(arg is_simulation)">
         <xacro:macro name="ros2control_swerve_module_iface" params="name drive_id turn_id">
             <joint name="db_${name}_fork_tyre_joint">
                 <command_interface name="velocity">
-                    <param name="min">-0.3</param>
-                    <param name="max">0.3</param>
+                    <limits enable="true"/>
                 </command_interface>
-                <state_interface name="position"/>
-                <state_interface name="velocity"/>
+                <xacro:if value="$(arg is_simulation)">
+                    <!-- TODO: currently our hw interface doesn't have state publishing! -->
+                    <state_interface name="position"/>
+                    <state_interface name="velocity"/>
+                </xacro:if>
             </joint>
             <joint name="db_${name}_smount_fork_joint">
                 <command_interface name="position">
                     <limits enable="true"/>
-                    <param name="min">-1.6</param>
-                    <param name="max">1.6</param>
                 </command_interface>
-                <state_interface name="position"/>
-                <state_interface name="velocity"/>
+                <xacro:if value="$(arg is_simulation)">
+                    <!-- TODO: currently our hw interface doesn't have state publishing! -->
+                    <state_interface name="position"/>
+                    <state_interface name="velocity"/>
+                </xacro:if>
             </joint>
         </xacro:macro>
@@ -42,12 +46,10 @@
             </hardware>
         </xacro:if>
-        <!-- Drivebase drive motors -->
-        <xacro:ros2control_swerve_module_iface name="fl" drive_id="1" turn_id="2"/>
-        <xacro:ros2control_swerve_module_iface name="fr" drive_id="3" turn_id="4"/>
-        <xacro:ros2control_swerve_module_iface name="bl" drive_id="5" turn_id="6"/>
-        <xacro:ros2control_swerve_module_iface name="br" drive_id="7" turn_id="8"/>
+        <xacro:ros2control_swerve_module_iface name="fl" drive_id="3050" turn_id="3000"/>
+        <xacro:ros2control_swerve_module_iface name="fr" drive_id="3060" turn_id="3010"/>
+        <xacro:ros2control_swerve_module_iface name="bl" drive_id="3070" turn_id="3020"/>
+        <xacro:ros2control_swerve_module_iface name="br" drive_id="3080" turn_id="3030"/>
         <xacro:ros2control_drivebase_suspension_pivot side="l"/>
         <xacro:ros2control_drivebase_suspension_pivot side="r"/>
-        <!-- TODO: Drivebase turn motors -->
     </ros2_control>
 </robot>

File: src/rover/description/utils/motor_stepper.xacro (robot description, xacro)
@@ -1,27 +1,12 @@
 <?xml version="1.0"?>
 <robot xmlns:xacro="http://www.ros.org/wiki/xacro" >
-    <xacro:macro name="bg431_motor" params="name device_index ratio use_auxilary">
-        <ros2_control name="${name}_motor" type="actuator">
+    <xacro:macro name="motor_stepper" params="name subject_id">
+        <ros2_control name="$motor_stepper_{name}" type="actuator">
             <hardware>
                 <plugin>bg431esc1_actuator::Bg431esc1Actuator</plugin>
-                <param name="device_index">${device_index}</param>
-                <param name="ratio">${ratio}</param>
-                <param name="use_auxilary">${use_auxilary}</param>
+                <param name="subject_id">${subject_id}</param>
             </hardware>
             <joint name="${name}">
                 <command_interface name="position"/>
-                <command_interface name="velocity"/>
-                <command_interface name="torque"/>
-                <state_interface name="position"/>
-                <state_interface name="velocity"/>
-                <state_interface name="primary_position"/>
-                <state_interface name="primary_velocity"/>
-                <state_interface name="auxilary_position"/>
-                <state_interface name="auxilary_velocity"/>
-                <state_interface name="applied_voltage"/>
-                <state_interface name="stator_current"/>
-                <state_interface name="supply_current"/>
-                <state_interface name="bus_voltage"/>
-                <state_interface name="driver_temperature"/>
             </joint>
         </ros2_control>

File: src/rover/description/utils/motor_vesc.xacro (robot description, xacro)
@@ -1,27 +1,12 @@
 <?xml version="1.0"?>
 <robot xmlns:xacro="http://www.ros.org/wiki/xacro" >
-    <xacro:macro name="bg431_motor" params="name device_index ratio use_auxilary">
-        <ros2_control name="${name}_motor" type="actuator">
+    <xacro:macro name="motor_vesc" params="name subject_id">
+        <ros2_control name="$motor_vesc_{name}" type="actuator">
             <hardware>
                 <plugin>bg431esc1_actuator::Bg431esc1Actuator</plugin>
-                <param name="device_index">${device_index}</param>
-                <param name="ratio">${ratio}</param>
-                <param name="use_auxilary">${use_auxilary}</param>
+                <param name="subject_id">${subject_id}</param>
             </hardware>
             <joint name="${name}">
-                <command_interface name="position"/>
                 <command_interface name="velocity"/>
-                <command_interface name="torque"/>
-                <state_interface name="position"/>
-                <state_interface name="velocity"/>
-                <state_interface name="primary_position"/>
-                <state_interface name="primary_velocity"/>
-                <state_interface name="auxilary_position"/>
-                <state_interface name="auxilary_velocity"/>
-                <state_interface name="applied_voltage"/>
-                <state_interface name="stator_current"/>
-                <state_interface name="supply_current"/>
-                <state_interface name="bus_voltage"/>
-                <state_interface name="driver_temperature"/>
             </joint>
         </ros2_control>
