Commit message: Refactor ros (#161)
* Begin refactor

* More progress

* Moar progress

* Fix init.bash to be runnable from anywhere

* Fix swerve_drive_controller compilation

* Update swerve drive controller, no more warnings 😸

* Fix simulation, format files

* Clean up ros2control usage in URDF

* Fix control_station readme

* Scuffed angle optimization code, limit to ±90 deg

* Make mock cyphal VESC driver to test integration, pipe it up in rover pkg

* Mmm less toasty

* Add `uv` python package manager to devcontainer

File: src/rover/description/core/core.xacro (robot description, xacro)
@@ -29,3 +29,10 @@
         <material>Gazebo/Orange</material>
     </gazebo>
+    <xacro:include filename="drivebase.xacro" />
+    <xacro:if value="$(arg is_simulation)">
+        <xacro:include filename="ros2control_gazebo.xacro" />
+    </xacro:if>
+    <xacro:unless value="$(arg is_simulation)">
+        <xacro:include filename="ros2control.xacro" />
+    </xacro:unless>
 </robot>

File: src/rover/description/core/db_helpers.xacro (robot description, xacro)
@@ -19,7 +19,7 @@
             <parent link="${prefix}_smount"/>
             <child link="${prefix}_wheel_fork"/>
-	    <origin xyz="${0} ${0} ${-0.213/2 - 0.03/2}" rpy="0 0 0"/>
+	        <origin xyz="${0} ${0} ${-0.213/2 - 0.03/2}" rpy="0 0 0"/>
             <axis xyz="0 0 1"/>
-            <limit lower="${-pi/2}" upper="${pi/2}" effort="40.0" velocity="12.8"/>
+            <limit lower="${-pi/2}" upper="${pi/2}" effort="400" velocity="5"/>
         </joint>
         <!-- This is the actual wheel -->
@@ -29,4 +29,5 @@
             <origin xyz="0 0 ${-0.05}" rpy="${-pi/2} 0 0" />
             <axis xyz="0 0 1"/>
+            <limit effort="400" velocity="0.2"/>
         </joint>
         <!-- ALL LINKS BELOW THIS LINE -->

File: src/rover/description/robot.urdf.xacro (robot description, xacro)
@@ -2,14 +2,14 @@
 <robot xmlns:xacro="http://www.ros.org/wiki/xacro"  name="robot">
     <xacro:arg name="is_simulation" default="false"/>
-    <xacro:unless value="$(arg is_simulation)">
-        <xacro:include filename="utils/bg431_motor.xacro"/>
-    </xacro:unless>
-    <xacro:include filename="cameras/depth_cams.xacro" />
+    <!-- DISABLED (false) / ENABLED (true) -->
+    <!-- core subsystem can't be disabled! -->
+    <!-- utilities -->
     <xacro:include filename="utils/inertial_macros.xacro" />
     <xacro:include filename="utils/materials.xacro" />
-    <xacro:include filename="chassis/chassis.xacro" />
-    <xacro:include filename="drivebase/drivebase.xacro" />
+    <!-- simulation specific global stuff -->
     <xacro:if value="$(arg is_simulation)">
         <xacro:include filename="utils/gazebo_plugins.xacro" />
     </xacro:if>
+    <xacro:include filename="core/core.xacro" />
+    <!--<xacro:include filename="cameras/depth_cams.xacro" /> -->
 </robot>
