File: src/led_beacon_elec/led_beacon.kicad_pcb (KiCad board)
At the start: 2 copper layers, 100 x 68 mm, 105 parts, among them J1 Conn_01x03

Commit message: Fix bypass caps lmao
Parts:
- moved C1 7.95 mm to (161.2, 123.2), turned to -90 degrees
- moved C10 7.95 mm to (71.2, 123.2), turned to -90 degrees
- moved C11 7.95 mm to (78.8, 116.8), turned to 90 degrees
- moved C12 7.95 mm to (88.8, 116.8), turned to 90 degrees
- moved C13 7.95 mm to (98.8, 116.8), turned to 90 degrees
- moved C14 7.95 mm to (108.8, 116.8), turned to 90 degrees
- moved C15 7.95 mm to (118.8, 116.8), turned to 90 degrees
- moved C16 7.95 mm to (128.8, 116.8), turned to 90 degrees
- moved C17 7.95 mm to (138.8, 116.8), turned to 90 degrees
- moved C18 7.95 mm to (148.8, 116.8), turned to 90 degrees
- moved C19 7.95 mm to (158.8, 116.8), turned to 90 degrees
- moved C2 7.95 mm to (151.2, 123.2), turned to -90 degrees
- moved C20 7.95 mm to (168.8, 116.8), turned to 90 degrees
- moved C21 7.95 mm to (161.2, 103.2), turned to -90 degrees
- moved C22 7.95 mm to (151.2, 103.2), turned to -90 degrees
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Routing:
- net GND: track 128.2 -> 137.4 mm, vias 60 -> 110
- net Net-(D1-DIN): track 49.8 -> 52.0 mm
- net Net-(D10-DOUT): track 10.6 -> 12.4 mm
- net Net-(D30-DOUT): track 10.6 -> 12.2 mm
- net Net-(D40-DOUT): track 11.0 -> 11.7 mm
- net Net-(D20-DOUT): track 11.0 -> 11.7 mm
- net Net-(D8-DOUT): track 7.63 -> 7.03 mm
- net Net-(D7-DOUT): track 7.63 -> 7.03 mm
- net Net-(D6-DOUT): track 7.63 -> 7.03 mm
- net Net-(D5-DOUT): track 7.63 -> 7.03 mm
- net Net-(D49-DOUT): track 7.63 -> 7.03 mm
- net Net-(D48-DOUT): track 7.63 -> 7.03 mm
- net Net-(D47-DOUT): track 7.63 -> 7.03 mm
- net Net-(D46-DOUT): track 7.63 -> 7.03 mm
- net Net-(D45-DOUT): track 7.63 -> 7.03 mm
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Other:
- outline, holes or cut-outs redrawn

Commit message: Comply with versioning scheme
Other:
- board text added: "Rev. 1p0"
